Commit message: OnRobot 2FG7 addition - Inclusion package 1

File: urdf/inc/rg_common.xacro (robot description, xacro)
@@ -1,5 +1,7 @@
 <?xml version="1.0"?>
 <robot xmlns:xacro="http://www.ros.org/wiki/xacro">
-  <xacro:macro name="onrobot_base_link" params="prefix">
+  <!-- Include common utilities -->
+  <xacro:include filename="$(find onrobot_description)/urdf/inc/common_utils.xacro" />
+  <xacro:macro name="onrobot_rg_base_link" params="prefix">
     <xacro:if value="${onrobot_type == 'rg2'}">
       <xacro:property name="mass" value="0.78" />
@@ -49,5 +51,5 @@
     </gazebo>
   </xacro:macro>
-  <xacro:macro name="outer_knuckle" params="prefix fingerprefix">
+  <xacro:macro name="onrobot_rg_outer_knuckle" params="prefix fingerprefix">
     <link name="${prefix}${fingerprefix}_outer_knuckle">
       <inertial>
@@ -79,5 +81,5 @@
     </gazebo>
   </xacro:macro>
-  <xacro:macro name="inner_knuckle" params="prefix fingerprefix">
+  <xacro:macro name="onrobot_rg_inner_knuckle" params="prefix fingerprefix">
     <link name="${prefix}${fingerprefix}_inner_knuckle">
       <inertial>
@@ -109,5 +111,5 @@
     </gazebo>
   </xacro:macro>
-  <xacro:macro name="inner_finger" params="prefix fingerprefix">
+  <xacro:macro name="onrobot_rg_inner_finger" params="prefix fingerprefix">
     <link name="${prefix}${fingerprefix}_inner_finger">
       <inertial>
@@ -143,33 +145,12 @@
     </gazebo>
   </xacro:macro>
-  <xacro:macro name="finger_joints" params="prefix fingerprefix reflect">
-    <xacro:inner_knuckle_joint prefix="${prefix}" fingerprefix="${fingerprefix}" reflect="${reflect}"/>
-    <xacro:inner_finger_joint prefix="${prefix}" fingerprefix="${fingerprefix}"/>
+  <xacro:macro name="onrobot_rg_finger_joints" params="prefix fingerprefix reflect">
+    <xacro:onrobot_rg_inner_knuckle_joint prefix="${prefix}" fingerprefix="${fingerprefix}" reflect="${reflect}"/>
+    <xacro:onrobot_rg_inner_finger_joint prefix="${prefix}" fingerprefix="${fingerprefix}"/>
   </xacro:macro>
-  <xacro:macro name="finger_links" params="prefix fingerprefix">
-    <xacro:outer_knuckle prefix="${prefix}" fingerprefix="${fingerprefix}"/>
-    <xacro:inner_knuckle prefix="${prefix}" fingerprefix="${fingerprefix}"/>
-    <xacro:inner_finger prefix="${prefix}" fingerprefix="${fingerprefix}"/>
-  </xacro:macro>
-  <!-- Gazebo plugin macro (for ros2_control simulation) -->
-  <xacro:macro name="gazebo_plugin" params="prefix">
-    <gazebo>
-      <plugin filename="libgazebo_ros2_control.so" name="gazebo_ros2_control">
-        <!-- Add additional parameters as needed -->
-      </plugin>
-    </gazebo>
-  </xacro:macro>
-  <!-- Simple transmission macro for a joint -->
-  <xacro:macro name="transmission_macro" params="prefix joint_name">
-    <transmission name="${prefix}${joint_name}_trans">
-      <type>transmission_interface/SimpleTransmission</type>
-      <joint name="${prefix}${joint_name}">
-        <hardwareInterface>hardware_interface/PositionJointInterface</hardwareInterface>
-      </joint>
-      <actuator name="${prefix}${joint_name}_motor">
-        <hardwareInterface>hardware_interface/PositionJointInterface</hardwareInterface>
-        <mechanicalReduction>1</mechanicalReduction>
-      </actuator>
-    </transmission>
+  <xacro:macro name="onrobot_rg_finger_links" params="prefix fingerprefix">
+    <xacro:onrobot_rg_outer_knuckle prefix="${prefix}" fingerprefix="${fingerprefix}"/>
+    <xacro:onrobot_rg_inner_knuckle prefix="${prefix}" fingerprefix="${fingerprefix}"/>
+    <xacro:onrobot_rg_inner_finger prefix="${prefix}" fingerprefix="${fingerprefix}"/>
   </xacro:macro>
 </robot>

File: urdf/onrobot_macro.xacro (robot description, xacro)
@@ -8,8 +8,9 @@
         sim_gazebo:=false
         use_fake_hardware:=false
-        connection_type:=serial
+        connection_type:=tcp
         device:=/tmp/ttyUR
         ip_address:=192.168.1.1
         port:=502
+        device_address:=65
         ">
         <xacro:if value="${onrobot_type == 'rg2'}">
@@ -21,8 +22,15 @@
             <xacro:onrobot_rg6 prefix="${prefix}"/>
         </xacro:if>
+        <!-- 2FG7 and 2FG14 Support -->
+        <xacro:if value="${onrobot_type == '2fg7' or onrobot_type == '2fg14'}">
+            <xacro:include filename="$(find onrobot_description)/urdf/2fg7_macro.xacro"/>
+            <xacro:onrobot_2fg7 prefix="${prefix}" onrobot_type="${onrobot_type}"/>
+        </xacro:if>
         <!-- Enable the gazebo plugin for simulation -->
         <xacro:if value="${sim_gazebo}">
             <gazebo>
-                <plugin filename="libgazebo_ros2_control.so" name="gazebo_ros2_control"/>
+                <plugin filename="libgazebo_ros2_control.so" name="gazebo_ros2_control">
+                    <parameters>$(find onrobot_description)/config/onrobot_controllers.yaml</parameters>
+                </plugin>
             </gazebo>
         </xacro:if>
@@ -32,10 +40,18 @@
                 <xacro:if value="${sim_gazebo}">
                     <plugin>gazebo_ros2_control/GazeboSystem</plugin>
+                    <param name="use_sim_time">true</param>
                 </xacro:if>
                 <xacro:if value="${use_fake_hardware}">
-                    <plugin>test_hardware_components/TestSingleJointActuator</plugin>
+                    <plugin>fake_components/GenericSystem</plugin>
+                    <param name="state_following_offset">0.0</param>
                 </xacro:if>
                 <xacro:unless value="${sim_gazebo or use_fake_hardware}">
-                    <plugin>onrobot_driver/RGHardwareInterface</plugin>
+                    <!-- Select appropriate hardware interface based on gripper type -->
+                    <xacro:if value="${onrobot_type == '2fg7' or onrobot_type == '2fg14'}">
+                        <plugin>onrobot_driver/FGHardwareInterface</plugin>
+                    </xacro:if>
+                    <xacro:if value="${onrobot_type == 'rg2' or onrobot_type == 'rg6'}">
+                        <plugin>onrobot_driver/RGHardwareInterface</plugin>
+                    </xacro:if>
                     <param name="onrobot_type">${onrobot_type}</param>
                     <param name="prefix">${prefix}</param>
@@ -44,4 +60,7 @@
                     <param name="ip_address">${ip_address}</param>
                     <param name="port">${port}</param>
+                    <xacro:if value="${onrobot_type == '2fg7' or onrobot_type == '2fg14'}">
+                        <param name="device_address">${device_address}</param>
+                    </xacro:if>
                 </xacro:unless>
             </hardware>
@@ -49,4 +68,5 @@
                 <command_interface name="position"/>
                 <state_interface name="position"/>
+                <state_interface name="velocity"/>
             </joint>
         </ros2_control>
