Commit message: materials file refactoring

File: urdf/inc/common_materials.xacro (robot description, xacro)
@@ -8,3 +8,6 @@
     <color rgba="0.700 0.700 0.700 1.000"/>
   </material>
+  <material name="onrobot_black">
+    <color rgba="0.1 0.1 0.1 1" />
+  </material>
 </robot>

File: urdf/inc/rg_common.xacro (robot description, xacro)
@@ -3,4 +3,5 @@
   <!-- Include common utilities -->
   <xacro:include filename="$(find onrobot_description)/urdf/inc/common_utils.xacro" />
+  <xacro:include filename="$(find onrobot_description)/urdf/inc/common_materials.xacro" />
   <xacro:macro name="onrobot_rg_base_link" params="prefix">
     <xacro:if value="${onrobot_type == 'rg2'}">
@@ -33,7 +34,5 @@
           <mesh filename="package://onrobot_description/meshes/${onrobot_type}/visual/base_link.stl" />
         </geometry>
-        <material name="">
-          <color rgba="0.8 0.8 0.8 1" />
-        </material>
+        <material name="onrobot_silver"/>
       </visual>
       <collision>
@@ -63,7 +62,5 @@
           <mesh filename="package://onrobot_description/meshes/${onrobot_type}/visual/outer_knuckle.stl" />
         </geometry>
-        <material name="">
-          <color rgba="0.8 0.8 0.8 1" />
-        </material>
+        <material name="onrobot_silver"/>
       </visual>
       <collision>
@@ -93,7 +90,5 @@
           <mesh filename="package://onrobot_description/meshes/${onrobot_type}/visual/inner_knuckle.stl" />
         </geometry>
-        <material name="">
-          <color rgba="0.8 0.8 0.8 1" />
-        </material>
+        <material name="onrobot_silver"/>
       </visual>
       <collision>
@@ -123,7 +118,5 @@
           <mesh filename="package://onrobot_description/meshes/${onrobot_type}/visual/inner_finger.stl" />
         </geometry>
-        <material name="">
-          <color rgba="0.1 0.1 0.1 1" />
-        </material>
+        <material name="onrobot_black"/>
       </visual>
       <collision>
@@ -136,5 +129,4 @@
     <gazebo reference="${prefix}${fingerprefix}_inner_finger">
       <kp>1000000.0</kp>
-      <kd>1.0</kd>
       <kd>1.0</kd>
       <mu1>1.0</mu1>

File: urdf/rg2_macro.xacro (robot description, xacro)
@@ -3,4 +3,5 @@
   <xacro:property name="onrobot_type" value="rg2" />
   <xacro:include filename="$(find onrobot_description)/urdf/inc/rg_common.xacro" />
+  <xacro:include filename="$(find onrobot_description)/urdf/inc/common_materials.xacro" />
   <!-- Define the missing macros that are referenced but not defined -->
   <xacro:macro name="onrobot_base_link" params="prefix">

File: urdf/rg6_macro.xacro (robot description, xacro)
@@ -3,4 +3,5 @@
   <xacro:property name="onrobot_type" value="rg6" />
   <xacro:include filename="$(find onrobot_description)/urdf/inc/rg_common.xacro" />
+  <xacro:include filename="$(find onrobot_description)/urdf/inc/common_materials.xacro" />
   <!-- Define the missing macros that are referenced but not defined -->
   <xacro:macro name="onrobot_base_link" params="prefix">
