Commit message: OnRobot 2FG7 addition - Inclusion package 1

File: urdf/onrobot_macro.xacro (robot description, xacro)
@@ -36,17 +36,8 @@
         </xacro:if>
         <!-- Define the OnRobot gripper hardware interface for ROS 2 control -->
-        <ros2_control name="OnRobotGripper" type="actuator">
-            <hardware>
-                <xacro:if value="${sim_gazebo}">
-                    <plugin>gazebo_ros2_control/GazeboSystem</plugin>
-                    <param name="use_sim_time">true</param>
-                </xacro:if>
-                <xacro:if value="${use_fake_hardware}">
-                    <!-- Use the correct fake hardware plugin for ROS 2 Humble -->
-                    <plugin>mock_components/GenericSystem</plugin>
-                    <param name="fake_sensor_commands">true</param>
-                    <param name="state_following_offset">0.0</param>
-                </xacro:if>
-                <xacro:unless value="${sim_gazebo or use_fake_hardware}">
+        <!-- For fake hardware, the UR macro handles everything, so we only define real hardware here -->
+        <xacro:unless value="${use_fake_hardware}">
+            <ros2_control name="OnRobotGripper" type="actuator">
+                <hardware>
                     <!-- Select appropriate hardware interface based on gripper type -->
                     <xacro:if value="${onrobot_type == '2fg7' or onrobot_type == '2fg14'}">
@@ -65,12 +56,12 @@
                         <param name="device_address">${device_address}</param>
                     </xacro:if>
-                </xacro:unless>
-            </hardware>
-            <joint name="${prefix}finger_width">
-                <command_interface name="position"/>
-                <state_interface name="position"/>
-                <state_interface name="velocity"/>
-            </joint>
-        </ros2_control>
+                </hardware>
+                <joint name="${prefix}finger_width">
+                    <command_interface name="position"/>
+                    <state_interface name="position"/>
+                    <state_interface name="velocity"/>
+                </joint>
+            </ros2_control>
+        </xacro:unless>
     </xacro:macro>
 </robot>

Commit message: 3fg15 inclusion

File: urdf/onrobot_macro.xacro (robot description, xacro)
@@ -1,73 +1,80 @@
 <?xml version="1.0"?>
 <robot xmlns:xacro="http://wiki.ros.org/xacro">
-    <!-- Include the macro file for the specific OnRobot model -->
-    <xacro:macro name="onrobot"
-        params="
-        onrobot_type
-        prefix:=''
-        sim_gazebo:=false
-        use_fake_hardware:=false
-        connection_type:=tcp
-        device:=/tmp/ttyUR
-        ip_address:=192.168.1.1
-        port:=502
-        device_address:=65
-        ">
-        <xacro:if value="${onrobot_type == 'rg2'}">
-            <xacro:include filename="$(find onrobot_description)/urdf/rg2_macro.xacro"/>
-            <xacro:onrobot_rg2 prefix="${prefix}"/>
-        </xacro:if>
-        <xacro:if value="${onrobot_type == 'rg6'}">
-            <xacro:include filename="$(find onrobot_description)/urdf/rg6_macro.xacro"/>
-            <xacro:onrobot_rg6 prefix="${prefix}"/>
-        </xacro:if>
-        <!-- 2FG7 and 2FG14 Support -->
-        <xacro:if value="${onrobot_type == '2fg7' or onrobot_type == '2fg14'}">
-            <xacro:include filename="$(find onrobot_description)/urdf/2fg7_macro.xacro"/>
-            <xacro:onrobot_2fg7 prefix="${prefix}" onrobot_type="${onrobot_type}"/>
-        </xacro:if>
-        <!-- Enable the gazebo plugin for simulation -->
-        <xacro:if value="${sim_gazebo}">
-            <gazebo>
-                <plugin filename="libgazebo_ros2_control.so" name="gazebo_ros2_control">
-                    <parameters>$(find onrobot_description)/config/onrobot_controllers.yaml</parameters>
-                </plugin>
-            </gazebo>
-        </xacro:if>
-        <!-- Define the OnRobot gripper hardware interface for ROS 2 control -->
-        <!-- For fake hardware, the UR macro handles everything, so we only define real hardware here -->
-        <xacro:unless value="${use_fake_hardware}">
-            <ros2_control name="OnRobotGripper" type="actuator">
-                <hardware>
-                    <!-- Select appropriate hardware interface based on gripper type -->
-                    <xacro:if value="${onrobot_type == '2fg7' or onrobot_type == '2fg14'}">
-                        <plugin>onrobot_driver::FGHardwareInterface</plugin>
-                        <param name="onrobot_type">${onrobot_type}</param>
-                        <param name="prefix">${prefix}</param>
-                        <param name="connection_type">${connection_type}</param>
-                        <param name="device">${device}</param>
-                        <param name="ip_address">${ip_address}</param>
-                        <param name="port">${port}</param>
-                        <param name="device_address">${device_address}</param>
-                        <param name="use_fake_hardware">false</param>
-                    </xacro:if>
-                    <xacro:if value="${onrobot_type == 'rg2' or onrobot_type == 'rg6'}">
-                        <plugin>onrobot_driver/RGHardwareInterface</plugin>
-                        <param name="onrobot_type">${onrobot_type}</param>
-                        <param name="prefix">${prefix}</param>
-                        <param name="connection_type">${connection_type}</param>
-                        <param name="device">${device}</param>
-                        <param name="ip_address">${ip_address}</param>
-                        <param name="port">${port}</param>
-                        <param name="use_fake_hardware">false</param>
-                    </xacro:if>
-                </hardware>
-                <joint name="${prefix}finger_width">
-                    <command_interface name="position"/>
-                    <state_interface name="position"/>
-                    <state_interface name="velocity"/>
-                </joint>
-            </ros2_control>
-        </xacro:unless>
-    </xacro:macro>
+  <!-- Macro principal para todos los grippers OnRobot -->
+  <xacro:macro name="onrobot"
+    params="
+      onrobot_type
+      prefix:=''
+      sim_gazebo:=false
+      use_fake_hardware:=false
+      connection_type:=tcp
+      device:=/tmp/ttyUR
+      ip_address:=192.168.1.1
+      port:=502
+      device_address:=65
+    ">
+    <!-- ====================== RG2 ====================== -->
+    <xacro:if value="${onrobot_type == 'rg2'}">
+      <xacro:include filename="$(find onrobot_description)/urdf/rg2_macro.xacro"/>
+      <xacro:onrobot_rg2 prefix="${prefix}"/>
+    </xacro:if>
+    <!-- ====================== RG6 ====================== -->
+    <xacro:if value="${onrobot_type == 'rg6'}">
+      <xacro:include filename="$(find onrobot_description)/urdf/rg6_macro.xacro"/>
+      <xacro:onrobot_rg6 prefix="${prefix}"/>
+    </xacro:if>
+    <!-- ====================== 2FG7 / 2FG14 ====================== -->
+    <xacro:if value="${onrobot_type == '2fg7' or onrobot_type == '2fg14'}">
+      <xacro:include filename="$(find onrobot_description)/urdf/2fg7_macro.xacro"/>
+      <xacro:onrobot_2fg7 prefix="${prefix}" onrobot_type="${onrobot_type}"/>
+    </xacro:if>
+    <!-- ====================== 3FG15 (NUEVO) ====================== -->
+    <xacro:if value="${onrobot_type == '3fg15'}">
+      <xacro:include filename="$(find onrobot_description)/urdf/3fg15_macro.xacro"/>
+      <xacro:onrobot_3fg15 prefix="${prefix}"/>
+    </xacro:if>
+    <!-- ====================== Gazebo Simulation ====================== -->
+    <xacro:if value="${sim_gazebo}">
+      <gazebo>
+        <plugin filename="libgazebo_ros2_control.so" name="gazebo_ros2_control">
+          <parameters>$(find onrobot_description)/config/onrobot_controllers.yaml</parameters>
+        </plugin>
+      </gazebo>
+    </xacro:if>
+    <!-- ====================== ROS2 Control ====================== -->
+    <xacro:unless value="${use_fake_hardware}">
+      <ros2_control name="OnRobotGripper" type="actuator">
+        <hardware>
+          <!-- 2FG7, 2FG14 y 3FG15 usan el mismo driver -->
+          <xacro:if value="${onrobot_type == '2fg7' or onrobot_type == '2fg14' or onrobot_type == '3fg15'}">
+            <plugin>onrobot_driver::FGHardwareInterface</plugin>
+            <param name="onrobot_type">${onrobot_type}</param>
+            <param name="prefix">${prefix}</param>
+            <param name="connection_type">${connection_type}</param>
+            <param name="device">${device}</param>
+            <param name="ip_address">${ip_address}</param>
+            <param name="port">${port}</param>
+            <param name="device_address">${device_address}</param>
+            <param name="use_fake_hardware">false</param>
+          </xacro:if>
+          <!-- RG2 / RG6 -->
+          <xacro:if value="${onrobot_type == 'rg2' or onrobot_type == 'rg6'}">
+            <plugin>onrobot_driver/RGHardwareInterface</plugin>
+            <param name="onrobot_type">${onrobot_type}</param>
+            <param name="prefix">${prefix}</param>
+            <param name="connection_type">${connection_type}</param>
+            <param name="device">${device}</param>
+            <param name="ip_address">${ip_address}</param>
+            <param name="port">${port}</param>
+            <param name="use_fake_hardware">false</param>
+          </xacro:if>
+        </hardware>
+        <joint name="${prefix}finger_width">
+          <command_interface name="position"/>
+          <state_interface name="position"/>
+          <state_interface name="velocity"/>
+        </joint>
+      </ros2_control>
+    </xacro:unless>
+  </xacro:macro>
 </robot>

Commit message: vgc10 gripper inclusion

File: urdf/onrobot_macro.xacro (robot description, xacro)
@@ -1,87 +1,113 @@
 <?xml version="1.0"?>
 <robot xmlns:xacro="http://wiki.ros.org/xacro">
-  <!-- Macro principal para todos los grippers OnRobot -->
-  <xacro:macro name="onrobot"
-    params="
-      onrobot_type
-      prefix:=''
-      sim_gazebo:=false
-      use_fake_hardware:=false
-      connection_type:=tcp
-      device:=/tmp/ttyUR
-      ip_address:=192.168.1.1
-      port:=502
-      device_address:=65
-    ">
-    <!-- ====================== RG2 ====================== -->
-    <xacro:if value="${onrobot_type == 'rg2'}">
-      <xacro:include filename="$(find onrobot_description)/urdf/rg2_macro.xacro"/>
-      <xacro:onrobot_rg2 prefix="${prefix}"/>
-    </xacro:if>
-    <!-- ====================== RG6 ====================== -->
-    <xacro:if value="${onrobot_type == 'rg6'}">
-      <xacro:include filename="$(find onrobot_description)/urdf/rg6_macro.xacro"/>
-      <xacro:onrobot_rg6 prefix="${prefix}"/>
-    </xacro:if>
-    <!-- ====================== 2FG7 / 2FG14 ====================== -->
-    <xacro:if value="${onrobot_type == '2fg7' or onrobot_type == '2fg14'}">
-      <xacro:include filename="$(find onrobot_description)/urdf/2fg7_macro.xacro"/>
-      <xacro:onrobot_2fg7 prefix="${prefix}" onrobot_type="${onrobot_type}"/>
-    </xacro:if>
-    <!-- ====================== 3FG15 ====================== -->
-    <xacro:if value="${onrobot_type == '3fg15'}">
-      <xacro:include filename="$(find onrobot_description)/urdf/3fg15_macro.xacro"/>
-      <xacro:onrobot_3fg15 prefix="${prefix}"/>
-    </xacro:if>
-    <!-- ====================== Gazebo Simulation ====================== -->
-    <xacro:if value="${sim_gazebo}">
-      <gazebo>
-        <plugin filename="libgazebo_ros2_control.so" name="gazebo_ros2_control">
-          <parameters>$(find onrobot_description)/config/onrobot_controllers.yaml</parameters>
-        </plugin>
-      </gazebo>
-      <!-- Include Gazebo-specific plugins for each gripper type -->
-      <xacro:if value="${onrobot_type == '3fg15'}">
-        <xacro:include filename="$(find onrobot_description)/urdf/inc/3fg15_gazebo.xacro"/>
-        <xacro:onrobot_3fg15_grasp_plugin prefix="${prefix}"/>
-        <xacro:onrobot_3fg15_mimic_plugin prefix="${prefix}"/>
-        <xacro:onrobot_3fg15_gazebo_properties prefix="${prefix}"/>
-      </xacro:if>
-    </xacro:if>
-    <!-- ====================== ROS2 Control ====================== -->
-    <xacro:unless value="${use_fake_hardware}">
-      <ros2_control name="OnRobotGripper" type="actuator">
-        <hardware>
-          <!-- 2FG7, 2FG14 y 3FG15 usan el mismo driver -->
-          <xacro:if value="${onrobot_type == '2fg7' or onrobot_type == '2fg14' or onrobot_type == '3fg15'}">
-            <plugin>onrobot_driver::FGHardwareInterface</plugin>
-            <param name="onrobot_type">${onrobot_type}</param>
-            <param name="prefix">${prefix}</param>
-            <param name="connection_type">${connection_type}</param>
-            <param name="device">${device}</param>
-            <param name="ip_address">${ip_address}</param>
-            <param name="port">${port}</param>
-            <param name="device_address">${device_address}</param>
-            <param name="use_fake_hardware">false</param>
-          </xacro:if>
-          <!-- RG2 / RG6 -->
-          <xacro:if value="${onrobot_type == 'rg2' or onrobot_type == 'rg6'}">
-            <plugin>onrobot_driver/RGHardwareInterface</plugin>
-            <param name="onrobot_type">${onrobot_type}</param>
-            <param name="prefix">${prefix}</param>
-            <param name="connection_type">${connection_type}</param>
-            <param name="device">${device}</param>
-            <param name="ip_address">${ip_address}</param>
-            <param name="port">${port}</param>
-            <param name="use_fake_hardware">false</param>
-          </xacro:if>
-        </hardware>
-        <joint name="${prefix}finger_width">
-          <command_interface name="position"/>
-          <state_interface name="position"/>
-          <state_interface name="velocity"/>
-        </joint>
-      </ros2_control>
-    </xacro:unless>
-  </xacro:macro>
+    <!-- Include the macro file for the specific OnRobot model -->
+    <xacro:macro name="onrobot"
+        params="
+        onrobot_type
+        prefix:=''
+        sim_gazebo:=false
+        use_fake_hardware:=false
+        connection_type:=tcp
+        device:=/tmp/ttyUR
+        ip_address:=192.168.1.1
+        port:=502
+        device_address:=65
+        ">
+        <xacro:if value="${onrobot_type == 'rg2'}">
+            <xacro:include filename="$(find onrobot_description)/urdf/rg2_macro.xacro"/>
+            <xacro:onrobot_rg2 prefix="${prefix}"/>
+        </xacro:if>
+        <xacro:if value="${onrobot_type == 'rg6'}">
+            <xacro:include filename="$(find onrobot_description)/urdf/rg6_macro.xacro"/>
+            <xacro:onrobot_rg6 prefix="${prefix}"/>
+        </xacro:if>
+        <!-- 2FG7 and 2FG14 Support -->
+        <xacro:if value="${onrobot_type == '2fg7' or onrobot_type == '2fg14'}">
+            <xacro:include filename="$(find onrobot_description)/urdf/2fg7_macro.xacro"/>
+            <xacro:onrobot_2fg7 prefix="${prefix}" onrobot_type="${onrobot_type}"/>
+        </xacro:if>
+        <!-- 3FG15 and 3FG25 Support -->
+        <xacro:if value="${onrobot_type == '3fg15' or onrobot_type == '3fg25'}">
+            <xacro:include filename="$(find onrobot_description)/urdf/3fg15_macro.xacro"/>
+            <xacro:onrobot_3fg15 prefix="${prefix}"/>
+        </xacro:if>
+        <!-- VG10 and VGC10 Support -->
+        <xacro:if value="${onrobot_type == 'vg10' or onrobot_type == 'vgc10'}">
+            <xacro:include filename="$(find onrobot_description)/urdf/vg_macro.xacro"/>
+            <xacro:onrobot_vg prefix="${prefix}" onrobot_type="${onrobot_type}"/>
+        </xacro:if>
+        <!-- Enable the gazebo plugin for simulation -->
+        <xacro:if value="${sim_gazebo}">
+            <gazebo>
+                <plugin filename="libgazebo_ros2_control.so" name="gazebo_ros2_control">
+                    <parameters>$(find onrobot_description)/config/onrobot_controllers.yaml</parameters>
+                </plugin>
+            </gazebo>
+        </xacro:if>
+        <!-- Define the OnRobot gripper hardware interface for ROS 2 control -->
+        <!-- For fake hardware, the UR macro handles everything, so we only define real hardware here -->
+        <xacro:unless value="${use_fake_hardware}">
+            <ros2_control name="OnRobotGripper" type="actuator">
+                <hardware>
+                    <!-- Select appropriate hardware interface based on gripper type -->
+                    <xacro:if value="${onrobot_type == '2fg7' or onrobot_type == '2fg14'}">
+                        <plugin>onrobot_driver/TwoFGHardwareInterface</plugin>
+                        <param name="onrobot_type">${onrobot_type}</param>
+                        <param name="prefix">${prefix}</param>
+                        <param name="connection_type">${connection_type}</param>
+                        <param name="device">${device}</param>
+                        <param name="ip_address">${ip_address}</param>
+                        <param name="port">${port}</param>
+                        <param name="device_address">${device_address}</param>
+                        <param name="use_fake_hardware">false</param>
+                    </xacro:if>
+                    <xacro:if value="${onrobot_type == '3fg15' or onrobot_type == '3fg25'}">
+                        <plugin>onrobot_driver/ThreeFGHardwareInterface</plugin>
+                        <param name="onrobot_type">${onrobot_type}</param>
+                        <param name="prefix">${prefix}</param>
+                        <param name="connection_type">${connection_type}</param>
+                        <param name="device">${device}</param>
+                        <param name="ip_address">${ip_address}</param>
+                        <param name="port">${port}</param>
+                        <param name="device_address">${device_address}</param>
+                        <param name="use_fake_hardware">false</param>
+                    </xacro:if>
+                    <xacro:if value="${onrobot_type == 'vg10' or onrobot_type == 'vgc10'}">
+                        <plugin>onrobot_driver/VGHardwareInterface</plugin>
+                        <param name="onrobot_type">${onrobot_type}</param>
+                        <param name="prefix">${prefix}</param>
+                        <param name="connection_type">${connection_type}</param>
+                        <param name="device">${device}</param>
+                        <param name="ip_address">${ip_address}</param>
+                        <param name="port">${port}</param>
+                        <param name="device_address">${device_address}</param>
+                        <param name="use_fake_hardware">false</param>
+                    </xacro:if>
+                    <xacro:if value="${onrobot_type == 'rg2' or onrobot_type == 'rg6'}">
+                        <plugin>onrobot_driver/RGHardwareInterface</plugin>
+                        <param name="onrobot_type">${onrobot_type}</param>
+                        <param name="prefix">${prefix}</param>
+                        <param name="connection_type">${connection_type}</param>
+                        <param name="device">${device}</param>
+                        <param name="ip_address">${ip_address}</param>
+                        <param name="port">${port}</param>
+                        <param name="use_fake_hardware">false</param>
+                    </xacro:if>
+                </hardware>
+                <xacro:if value="${onrobot_type.startswith('vg')}">
+                    <joint name="${prefix}gripper">
+                        <command_interface name="position"/>
+                        <state_interface name="position"/>
+                    </joint>
+                </xacro:if>
+                <xacro:unless value="${onrobot_type.startswith('vg')}">
+                    <joint name="${prefix}finger_width">
+                        <command_interface name="position"/>
+                        <state_interface name="position"/>
+                        <state_interface name="velocity"/>
+                    </joint>
+                </xacro:unless>
+            </ros2_control>
+        </xacro:unless>
+    </xacro:macro>
 </robot>
