Commit message: VGC10 inclusion

File: urdf/onrobot_macro.xacro (robot description, xacro)
@@ -1,5 +1,5 @@
 <?xml version="1.0"?>
 <robot xmlns:xacro="http://wiki.ros.org/xacro">
-  <!-- Macro principal para todos los grippers OnRobot -->
+  <!-- ====================== MACRO PRINCIPAL ONROBOT ====================== -->
   <xacro:macro name="onrobot"
     params="
@@ -13,5 +13,8 @@
       port:=502
       device_address:=65
+      num_cups:=4
     ">
+    <!-- ====================== INCLUSIONES COMUNES ====================== -->
+    <xacro:include filename="$(find onrobot_description)/urdf/inc/common_materials.xacro"/>
     <!-- ====================== RG2 ====================== -->
     <xacro:if value="${onrobot_type == 'rg2'}">
@@ -29,32 +32,43 @@
       <xacro:onrobot_2fg7 prefix="${prefix}" onrobot_type="${onrobot_type}"/>
     </xacro:if>
-    <!-- ====================== 3FG15 (NUEVO) ====================== -->
+    <!-- ====================== 3FG15 ====================== -->
     <xacro:if value="${onrobot_type == '3fg15'}">
       <xacro:include filename="$(find onrobot_description)/urdf/3fg15_macro.xacro"/>
       <xacro:onrobot_3fg15 prefix="${prefix}"/>
     </xacro:if>
-    <!-- ====================== Gazebo Simulation ====================== -->
+    <!-- ====================== VG10 (legacy) ====================== -->
+    <xacro:if value="${onrobot_type == 'vg10'}">
+      <xacro:include filename="$(find onrobot_description)/urdf/vg_macro.xacro"/>
+      <xacro:onrobot_vg prefix="${prefix}" onrobot_type="vg10" num_cups="${num_cups}"/>
+    </xacro:if>
+    <!-- ====================== VGC10 ====================== -->
+    <xacro:if value="${onrobot_type == 'vgc10'}">
+      <xacro:include filename="$(find onrobot_description)/urdf/vg_macro.xacro"/>
+      <xacro:include filename="$(find onrobot_description)/urdf/vgc10_gazebo.xacro"/>
+      <xacro:onrobot_vg prefix="${prefix}" onrobot_type="vgc10" num_cups="${num_cups}"/>
+    </xacro:if>
+    <!-- ====================== GAZEBO: Plugins y Propiedades ====================== -->
     <xacro:if value="${sim_gazebo}">
-      <gazebo>
-        <plugin filename="libgazebo_ros2_control.so" name="gazebo_ros2_control">
-          <parameters>$(find onrobot_description)/config/onrobot_controllers.yaml</parameters>
-        </plugin>
-      </gazebo>
+      <!-- Solo para 2FG7 (pinzas) -->
+      <xacro:if value="${onrobot_type == '2fg7' or onrobot_type == '2fg14'}">
+        <xacro:include filename="$(find onrobot_description)/urdf/2fg7_gazebo.xacro"/>
+        <xacro:onrobot_2fg7_grasp_plugin prefix="${prefix}"/>
+        <xacro:onrobot_2fg7_mimic_plugin prefix="${prefix}"/>
+        <xacro:onrobot_2fg7_gazebo_properties prefix="${prefix}"/>
+      </xacro:if>
+      <!-- Solo para VGC10 (vacío) -->
+      <xacro:if value="${onrobot_type == 'vgc10'}">
+        <xacro:onrobot_vgc10_vacuum_plugin prefix="${prefix}" num_cups="${num_cups}"/>
+        <xacro:onrobot_vgc10_gazebo_properties prefix="${prefix}"/>
+      </xacro:if>
     </xacro:if>
-    <!-- ====================== ROS2 Control ====================== -->
+    <!-- ====================== ROS2 CONTROL (REAL) ====================== -->
     <xacro:unless value="${use_fake_hardware}">
       <ros2_control name="OnRobotGripper" type="actuator">
         <hardware>
-          <!-- 2FG7 y 2FG14 y usan el mismo driver -->
+          <!-- 2FG7 / 2FG14 -->
           <xacro:if value="${onrobot_type == '2fg7' or onrobot_type == '2fg14'}">
             <plugin>onrobot_driver::TwoFGHardwareInterface</plugin>
             <param name="onrobot_type">${onrobot_type}</param>
-            <param name="prefix">${prefix}</param>
-            <param name="connection_type">${connection_type}</param>
-            <param name="device">${device}</param>
-            <param name="ip_address">${ip_address}</param>
-            <param name="port">${port}</param>
-            <param name="device_address">${device_address}</param>
-            <param name="use_fake_hardware">false</param>
           </xacro:if>
           <!-- 3FG15 -->
@@ -62,11 +76,4 @@
             <plugin>onrobot_driver::ThreeFGHardwareInterface</plugin>
             <param name="onrobot_type">${onrobot_type}</param>
-            <param name="prefix">${prefix}</param>
-            <param name="connection_type">${connection_type}</param>
-            <param name="device">${device}</param>
-            <param name="ip_address">${ip_address}</param>
-            <param name="port">${port}</param>
-            <param name="device_address">${device_address}</param>
-            <param name="use_fake_hardware">false</param>
           </xacro:if>
           <!-- RG2 / RG6 -->
@@ -74,13 +81,21 @@
             <plugin>onrobot_driver::RGHardwareInterface</plugin>
             <param name="onrobot_type">${onrobot_type}</param>
-            <param name="prefix">${prefix}</param>
-            <param name="connection_type">${connection_type}</param>
-            <param name="device">${device}</param>
-            <param name="ip_address">${ip_address}</param>
-            <param name="port">${port}</param>
-            <param name="use_fake_hardware">false</param>
           </xacro:if>
+          <!-- VGC10 -->
+          <xacro:if value="${onrobot_type == 'vgc10'}">
+            <plugin>onrobot_driver::VGCHardwareInterface</plugin>
+            <param name="onrobot_type">vgc10</param>
+          </xacro:if>
+          <!-- Parámetros comunes -->
+          <param name="prefix">${prefix}</param>
+          <param name="connection_type">${connection_type}</param>
+          <param name="device">${device}</param>
+          <param name="ip_address">${ip_address}</param>
+          <param name="port">${port}</param>
+          <param name="device_address">${device_address}</param>
+          <param name="use_fake_hardware">false</param>
         </hardware>
-        <joint name="${prefix}finger_width">
+        <!-- Joint de control (mismo nombre en todos los macros) -->
+        <joint name="${prefix}gripper">
           <command_interface name="position"/>
           <state_interface name="position"/>

File: urdf/vg_macro.xacro (robot description, xacro)
@@ -1,16 +1,36 @@
 <?xml version="1.0"?>
 <robot xmlns:xacro="http://ros.org/wiki/xacro">
-  <xacro:macro name="onrobot_vg" params="prefix onrobot_type:='vg10'">
-    <!-- Base Link -->
+  <!-- =================================================================== -->
+  <!-- Macro: OnRobot VGC10 / VG10 Vacuum Gripper                          -->
+  <!-- =================================================================== -->
+  <xacro:macro name="onrobot_vg" params="
+      prefix
+      onrobot_type:='vgc10'
+      num_cups:=4
+    ">
+    <!-- =============================================================== -->
+    <!-- Determinar carpeta de mallas según tipo                         -->
+    <!-- =============================================================== -->
+    <xacro:property name="mesh_dir" value="${
+        'vg10' if onrobot_type == 'vg10' else 'vgc10'
+      }"/>
+    <!-- Sufijo para 1 o 4 ventosas -->
+    <xacro:property name="cup_suffix" value="_${num_cups}cups"/>
+    <xacro:property name="cup_suffix" value="" if="${num_cups == 4}"/>
+    <!-- =============================================================== -->
+    <!-- Base Link                                                       -->
+    <!-- =============================================================== -->
     <link name="${prefix}onrobot_base_link">
       <inertial>
         <origin xyz="0 0 0" rpy="0 0 0"/>
-        <mass value="0.5"/>
-        <inertia ixx="0.001" ixy="0.0" ixz="0.0" iyy="0.001" iyz="0.0" izz="0.001"/>
+        <mass value="0.65"/>
+        <inertia ixx="0.0025" ixy="0.0" ixz="0.0"
+                 iyy="0.0025" iyz="0.0" izz="0.0018"/>
       </inertial>
       <visual>
         <origin xyz="0 0 0" rpy="0 0 0"/>
         <geometry>
-          <mesh filename="package://onrobot_description/meshes/${onrobot_type}/visual/base_link.stl" scale="0.001 0.001 0.001"/>
+          <mesh filename="package://onrobot_description/meshes/${mesh_dir}/visual/base_link${cup_suffix}.stl"
+                scale="0.001 0.001 0.001"/>
         </geometry>
         <material name="onrobot_silver"/>
@@ -19,19 +39,24 @@
         <origin xyz="0 0 0" rpy="0 0 0"/>
         <geometry>
-          <mesh filename="package://onrobot_description/meshes/${onrobot_type}/collision/base_link.stl" scale="0.001 0.001 0.001"/>
+          <mesh filename="package://onrobot_description/meshes/${mesh_dir}/collision/base_link${cup_suffix}.stl"
+                scale="0.001 0.001 0.001"/>
         </geometry>
       </collision>
     </link>
-    <!-- Suction Cups -->
+    <!-- =============================================================== -->
+    <!-- Suction Cups Link                                               -->
+    <!-- =============================================================== -->
     <link name="${prefix}suction_cups">
       <inertial>
-        <origin xyz="0 0 0" rpy="0 0 0"/>
-        <mass value="0.1"/>
-        <inertia ixx="0.0001" ixy="0.0" ixz="0.0" iyy="0.0001" iyz="0.0" izz="0.0001"/>
+        <origin xyz="0 0 -0.01" rpy="0 0 0"/>
+        <mass value="0.12"/>
+        <inertia ixx="0.0003" ixy="0.0" ixz="0.0"
+                 iyy="0.0003" iyz="0.0" izz="0.00015"/>
       </inertial>
       <visual>
         <origin xyz="0 0 0" rpy="0 0 0"/>
         <geometry>
-          <mesh filename="package://onrobot_description/meshes/${onrobot_type}/visual/suction_cups.stl" scale="0.001 0.001 0.001"/>
+          <mesh filename="package://onrobot_description/meshes/${mesh_dir}/visual/suction_cup${cup_suffix}.stl"
+                scale="0.001 0.001 0.001"/>
         </geometry>
         <material name="onrobot_silver"/>
@@ -40,9 +65,12 @@
         <origin xyz="0 0 0" rpy="0 0 0"/>
         <geometry>
-          <mesh filename="package://onrobot_description/meshes/${onrobot_type}/collision/suction_cups.stl" scale="0.001 0.001 0.001"/>
+          <mesh filename="package://onrobot_description/meshes/${mesh_dir}/collision/suction_cup${cup_suffix}.stl"
+                scale="0.001 0.001 0.001"/>
         </geometry>
       </collision>
     </link>
-    <!-- Suction Cups Joint -->
+    <!-- =============================================================== -->
+    <!-- Joint: Suction Cups                                             -->
+    <!-- =============================================================== -->
     <joint name="${prefix}suction_cups_joint" type="fixed">
       <origin xyz="0 0 0.02" rpy="0 0 0"/>
@@ -50,5 +78,7 @@
       <child link="${prefix}suction_cups"/>
     </joint>
-    <!-- TCP Link -->
+    <!-- =============================================================== -->
+    <!-- TCP Link (Tool Center Point)                                    -->
+    <!-- =============================================================== -->
     <link name="${prefix}gripper_tcp"/>
     <joint name="${prefix}tcp_joint" type="fixed">
@@ -57,5 +87,7 @@
       <child link="${prefix}gripper_tcp"/>
     </joint>
-    <!-- Dummy joint for ROS Control (simulates gripper state) -->
+    <!-- =============================================================== -->
+    <!-- Dummy Prismatic Joint (para control y visualización)           -->
+    <!-- =============================================================== -->
     <link name="${prefix}gripper_mock_link"/>
     <joint name="${prefix}gripper" type="prismatic">
@@ -64,7 +96,10 @@
       <child link="${prefix}gripper_mock_link"/>
       <axis xyz="0 0 1"/>
-      <limit lower="0.0" upper="1.0" velocity="1.0" effort="10"/>
+      <limit lower="0.0" upper="1.0" velocity="0.5" effort="100.0"/>
+      <dynamics damping="0.7" friction="0.0"/>
     </joint>
-    <!-- Transmission for ROS Control -->
+    <!-- =============================================================== -->
+    <!-- Transmission (para simulación y control)                        -->
+    <!-- =============================================================== -->
     <transmission name="${prefix}gripper_trans">
       <type>transmission_interface/SimpleTransmission</type>
@@ -72,7 +107,6 @@
         <hardwareInterface>hardware_interface/PositionJointInterface</hardwareInterface>
       </joint>
-      <actuator name="${prefix}gripper_motor">
-        <hardwareInterface>hardware_interface/PositionJointInterface</hardwareInterface>
-        <mechanicalReduction>1</mechanicalReduction>
+      <actuator name="${prefix}gripper_actuator">
+        <mechanicalReduction>1.0</mechanicalReduction>
       </actuator>
     </transmission>

Commit message: driver refactorization update

File: urdf/onrobot_macro.xacro (robot description, xacro)
@@ -29,5 +29,5 @@
       <xacro:onrobot_2fg7 prefix="${prefix}" onrobot_type="${onrobot_type}"/>
     </xacro:if>
-    <!-- ====================== 3FG15 (NUEVO) ====================== -->
+    <!-- ====================== 3FG15 ====================== -->
     <xacro:if value="${onrobot_type == '3fg15'}">
       <xacro:include filename="$(find onrobot_description)/urdf/3fg15_macro.xacro"/>
@@ -46,7 +46,7 @@
       <ros2_control name="OnRobotGripper" type="actuator">
         <hardware>
-          <!-- 2FG7, 2FG14 y 3FG15 usan el mismo driver -->
-          <xacro:if value="${onrobot_type == '2fg7' or onrobot_type == '2fg14' or onrobot_type == '3fg15'}">
-            <plugin>onrobot_driver::FGHardwareInterface</plugin>
+          <!-- 2FG7 / 2FG14 - TwoFG Hardware Interface -->
+          <xacro:if value="${onrobot_type == '2fg7' or onrobot_type == '2fg14'}">
+            <plugin>onrobot_driver::TwoFGHardwareInterface</plugin>
             <param name="onrobot_type">${onrobot_type}</param>
             <param name="prefix">${prefix}</param>
@@ -58,5 +58,17 @@
             <param name="use_fake_hardware">false</param>
           </xacro:if>
-          <!-- RG2 / RG6 -->
+          <!-- 3FG15 - ThreeFG Hardware Interface -->
+          <xacro:if value="${onrobot_type == '3fg15'}">
+            <plugin>onrobot_driver::ThreeFGHardwareInterface</plugin>
+            <param name="onrobot_type">${onrobot_type}</param>
+            <param name="prefix">${prefix}</param>
+            <param name="connection_type">${connection_type}</param>
+            <param name="device">${device}</param>
+            <param name="ip_address">${ip_address}</param>
+            <param name="port">${port}</param>
+            <param name="device_address">${device_address}</param>
+            <param name="use_fake_hardware">false</param>
+          </xacro:if>
+          <!-- RG2 / RG6 - RG Hardware Interface -->
           <xacro:if value="${onrobot_type == 'rg2' or onrobot_type == 'rg6'}">
             <plugin>onrobot_driver::RGHardwareInterface</plugin>
@@ -67,14 +79,83 @@
             <param name="ip_address">${ip_address}</param>
             <param name="port">${port}</param>
+            <param name="device_address">${device_address}</param>
             <param name="use_fake_hardware">false</param>
           </xacro:if>
         </hardware>
-        <joint name="${prefix}finger_width">
-          <command_interface name="position"/>
-          <state_interface name="position"/>
-          <state_interface name="velocity"/>
-        </joint>
+        <!-- Joint configuration for all gripper types -->
+        <xacro:if value="${onrobot_type == '2fg7' or onrobot_type == '2fg14' or onrobot_type == '3fg15'}">
+          <joint name="${prefix}finger_width">
+            <command_interface name="position"/>
+            <state_interface name="position"/>
+            <state_interface name="velocity"/>
+          </joint>
+        </xacro:if>
+        <xacro:if value="${onrobot_type == 'rg2' or onrobot_type == 'rg6'}">
+          <joint name="${prefix}gripper_finger_joint">
+            <command_interface name="position"/>
+            <state_interface name="position"/>
+            <state_interface name="velocity"/>
+          </joint>
+        </xacro:if>
       </ros2_control>
     </xacro:unless>
+    <!-- ====================== Fake Hardware (for testing) ====================== -->
+    <xacro:if value="${use_fake_hardware}">
+      <ros2_control name="OnRobotGripper" type="actuator">
+        <hardware>
+          <!-- 2FG7 / 2FG14 - TwoFG Hardware Interface with fake hardware -->
+          <xacro:if value="${onrobot_type == '2fg7' or onrobot_type == '2fg14'}">
+            <plugin>onrobot_driver::TwoFGHardwareInterface</plugin>
+            <param name="onrobot_type">${onrobot_type}</param>
+            <param name="prefix">${prefix}</param>
+            <param name="connection_type">${connection_type}</param>
+            <param name="device">${device}</param>
+            <param name="ip_address">${ip_address}</param>
+            <param name="port">${port}</param>
+            <param name="device_address">${device_address}</param>
+            <param name="use_fake_hardware">true</param>
+          </xacro:if>
+          <!-- 3FG15 - ThreeFG Hardware Interface with fake hardware -->
+          <xacro:if value="${onrobot_type == '3fg15'}">
+            <plugin>onrobot_driver::ThreeFGHardwareInterface</plugin>
+            <param name="onrobot_type">${onrobot_type}</param>
+            <param name="prefix">${prefix}</param>
+            <param name="connection_type">${connection_type}</param>
+            <param name="device">${device}</param>
+            <param name="ip_address">${ip_address}</param>
+            <param name="port">${port}</param>
+            <param name="device_address">${device_address}</param>
+            <param name="use_fake_hardware">true</param>
+          </xacro:if>
+          <!-- RG2 / RG6 - RG Hardware Interface with fake hardware -->
+          <xacro:if value="${onrobot_type == 'rg2' or onrobot_type == 'rg6'}">
+            <plugin>onrobot_driver::RGHardwareInterface</plugin>
+            <param name="onrobot_type">${onrobot_type}</param>
+            <param name="prefix">${prefix}</param>
+            <param name="connection_type">${connection_type}</param>
+            <param name="device">${device}</param>
+            <param name="ip_address">${ip_address}</param>
+            <param name="port">${port}</param>
+            <param name="device_address">${device_address}</param>
+            <param name="use_fake_hardware">true</param>
+          </xacro:if>
+        </hardware>
+        <!-- Joint configuration for all gripper types -->
+        <xacro:if value="${onrobot_type == '2fg7' or onrobot_type == '2fg14' or onrobot_type == '3fg15'}">
+          <joint name="${prefix}finger_width">
+            <command_interface name="position"/>
+            <state_interface name="position"/>
+            <state_interface name="velocity"/>
+          </joint>
+        </xacro:if>
+        <xacro:if value="${onrobot_type == 'rg2' or onrobot_type == 'rg6'}">
+          <joint name="${prefix}gripper_finger_joint">
+            <command_interface name="position"/>
+            <state_interface name="position"/>
+            <state_interface name="velocity"/>
+          </joint>
+        </xacro:if>
+      </ros2_control>
+    </xacro:if>
   </xacro:macro>
 </robot>
