Commit message: Add VGC10 vacuum gripper support with dual vacuum channels in URDF/XACRO files

File: urdf/onrobot_macro.xacro (robot description, xacro)
@@ -71,4 +71,36 @@
       </ros2_control>
     </xacro:if>
+    <!-- VGC10 Vacuum Gripper -->
+    <xacro:if value="${onrobot_type == 'vgc10'}">
+      <ros2_control name="OnRobotGripper" type="actuator">
+        <hardware>
+          <xacro:if value="${use_mock_hardware}">
+            <plugin>mock_components/GenericSystem</plugin>
+          </xacro:if>
+          <xacro:unless value="${use_mock_hardware}">
+            <plugin>onrobot_driver::VGC10HardwareInterface</plugin>
+            <param name="onrobot_type">${onrobot_type}</param>
+            <param name="prefix">${prefix}</param>
+            <param name="connection_type">${connection_type}</param>
+            <param name="device">${device}</param>
+            <param name="ip_address">${ip_address}</param>
+            <param name="port">${port}</param>
+            <param name="device_address">${device_address}</param>
+            <param name="use_fake_hardware">${use_fake_hardware}</param>
+          </xacro:unless>
+        </hardware>
+        <!-- Independent Dual Vacuum Channels -->
+        <joint name="${prefix}vacuum_channel_a">
+          <command_interface name="position"/>
+          <state_interface name="position"/>
+          <state_interface name="effort"/>
+        </joint>
+        <joint name="${prefix}vacuum_channel_b">
+          <command_interface name="position"/>
+          <state_interface name="position"/>
+          <state_interface name="effort"/>
+        </joint>
+      </ros2_control>
+    </xacro:if>
   </xacro:macro>
 </robot>

File: urdf/vgc10_macro.xacro (robot description, xacro)
@@ -44,4 +44,31 @@
       <child link="${prefix}gripper_tcp"/>
     </joint>
+    <!-- Virtual links and joints for dual vacuum channels (Channel A and Channel B) -->
+    <link name="${prefix}vacuum_channel_a_mock_link">
+      <inertial>
+        <mass value="1e-9"/>
+        <inertia ixx="1e-9" ixy="0" ixz="0" iyy="1e-9" iyz="0" izz="1e-9"/>
+      </inertial>
+    </link>
+    <joint name="${prefix}vacuum_channel_a" type="prismatic">
+      <origin xyz="0 0 0" rpy="0 0 0"/>
+      <parent link="${prefix}onrobot_base_link"/>
+      <child link="${prefix}vacuum_channel_a_mock_link"/>
+      <axis xyz="0 0 1"/>
+      <limit lower="0.0" upper="1.0" velocity="1.0" effort="100.0"/>
+    </joint>
+    <link name="${prefix}vacuum_channel_b_mock_link">
+      <inertial>
+        <mass value="1e-9"/>
+        <inertia ixx="1e-9" ixy="0" ixz="0" iyy="1e-9" iyz="0" izz="1e-9"/>
+      </inertial>
+    </link>
+    <joint name="${prefix}vacuum_channel_b" type="prismatic">
+      <origin xyz="0 0 0" rpy="0 0 0"/>
+      <parent link="${prefix}onrobot_base_link"/>
+      <child link="${prefix}vacuum_channel_b_mock_link"/>
+      <axis xyz="0 0 1"/>
+      <limit lower="0.0" upper="1.0" velocity="1.0" effort="100.0"/>
+    </joint>
   </xacro:macro>
 </robot>
