Commit message: Working with decomposed stl files

File: urdf/3fg15_macro.xacro (robot description, xacro)
@@ -3,48 +3,45 @@
   <xacro:include filename="$(find onrobot_description)/urdf/inc/common_utils.xacro" />
   <xacro:include filename="$(find onrobot_description)/urdf/inc/2fg7_materials.xacro" />
-  <!-- ============================================= -->
-  <!-- MACRO: OnRobot 3FG15 (estructura IGUAL a 2FG7) -->
-  <!-- STL COMPLETO → solo base_link con visual     -->
-  <!-- ============================================= -->
+  <!-- Macro for OnRobot 3FG15 gripper -->
   <xacro:macro name="onrobot_3fg15" params="prefix onrobot_type:='3fg15'">
-    <!-- ====================== Base Link (STL COMPLETO del 3FG15) ====================== -->
+    <!-- Base Link -->
     <link name="${prefix}onrobot_base_link">
       <inertial>
-        <origin xyz="0 0 0.05" rpy="${-pi/2} 0 0"/>
+        <origin xyz="0 0 0.05" rpy="0 0 0"/>
         <mass value="1.2"/>
         <inertia ixx="0.012" ixy="0.0" ixz="0.0" iyy="0.012" iyz="0.0" izz="0.008"/>
       </inertial>
       <visual>
-        <origin xyz="0 0 0.05" rpy="${-pi/2} 0 0"/>
+        <origin xyz="0 0 0" rpy="0 0 0"/>
         <geometry>
-          <mesh filename="package://onrobot_description/meshes/3fg15/visual/3fg15.stl" scale="0.001 0.001 0.001"/>
+          <mesh filename="package://onrobot_description/meshes/3fg15/visual/base.stl" scale="0.001 0.001 0.001"/>
         </geometry>
         <material name="onrobot_silver"/>
       </visual>
       <collision>
-        <origin xyz="0 0 0.05" rpy="${-pi/2} 0 0"/>
+        <origin xyz="0 0 0" rpy="0 0 0"/>
         <geometry>
-          <mesh filename="package://onrobot_description/meshes/3fg15/collision/3fg15.stl" scale="0.001 0.001 0.001"/>
+          <mesh filename="package://onrobot_description/meshes/3fg15/collision/base.stl" scale="0.001 0.001 0.001"/>
         </geometry>
       </collision>
     </link>
-    <!-- ====================== Dummy Links para simular movimiento (solo para joint) ====================== -->
-    <!-- No tienen STL → solo para el joint principal (finger_width) -->
+    <!-- Finger Links with proper STL files -->
     <link name="${prefix}left_finger_link">
       <inertial>
         <origin xyz="0 0 0" rpy="0 0 0"/>
-        <mass value="0.01"/>
-        <inertia ixx="0.00001" ixy="0.0" ixz="0.0" iyy="0.00001" iyz="0.0" izz="0.00001"/>
+        <mass value="0.1"/>
+        <inertia ixx="0.0001" ixy="0.0" ixz="0.0" iyy="0.0001" iyz="0.0" izz="0.0001"/>
       </inertial>
       <visual>
         <origin xyz="0 0 0" rpy="0 0 0"/>
         <geometry>
-          <box size="0.001 0.001 0.001"/> <!-- invisible -->
+          <mesh filename="package://onrobot_description/meshes/3fg15/visual/left_finger.stl" scale="0.001 0.001 0.001"/>
         </geometry>
+        <material name="onrobot_silver"/>
       </visual>
       <collision>
         <origin xyz="0 0 0" rpy="0 0 0"/>
         <geometry>
-          <box size="0.001 0.001 0.001"/>
+          <mesh filename="package://onrobot_description/meshes/3fg15/collision/left_finger.stl" scale="0.001 0.001 0.001"/>
         </geometry>
       </collision>
@@ -53,23 +50,45 @@
       <inertial>
         <origin xyz="0 0 0" rpy="0 0 0"/>
-        <mass value="0.01"/>
-        <inertia ixx="0.00001" ixy="0.0" ixz="0.0" iyy="0.00001" iyz="0.0" izz="0.00001"/>
+        <mass value="0.1"/>
+        <inertia ixx="0.0001" ixy="0.0" ixz="0.0" iyy="0.0001" iyz="0.0" izz="0.0001"/>
       </inertial>
       <visual>
         <origin xyz="0 0 0" rpy="0 0 0"/>
         <geometry>
-          <box size="0.001 0.001 0.001"/> <!-- invisible -->
+          <mesh filename="package://onrobot_description/meshes/3fg15/visual/right_finger.stl" scale="0.001 0.001 0.001"/>
         </geometry>
+        <material name="onrobot_silver"/>
       </visual>
       <collision>
         <origin xyz="0 0 0" rpy="0 0 0"/>
         <geometry>
-          <box size="0.001 0.001 0.001"/>
+          <mesh filename="package://onrobot_description/meshes/3fg15/collision/right_finger.stl" scale="0.001 0.001 0.001"/>
         </geometry>
       </collision>
     </link>
-    <!-- ====================== Dummy link for the main control joint ====================== -->
+    <!-- Middle Finger Link -->
+    <link name="${prefix}middle_finger_link">
+      <inertial>
+        <origin xyz="0 0 0" rpy="0 0 0"/>
+        <mass value="0.05"/>
+        <inertia ixx="0.00005" ixy="0.0" ixz="0.0" iyy="0.00005" iyz="0.0" izz="0.00005"/>
+      </inertial>
+      <visual>
+        <origin xyz="0 0 0" rpy="0 0 0"/>
+        <geometry>
+          <mesh filename="package://onrobot_description/meshes/3fg15/visual/middle_finger.stl" scale="0.001 0.001 0.001"/>
+        </geometry>
+        <material name="onrobot_silver"/>
+      </visual>
+      <collision>
+        <origin xyz="0 0 0" rpy="0 0 0"/>
+        <geometry>
+          <mesh filename="package://onrobot_description/meshes/3fg15/collision/middle_finger.stl" scale="0.001 0.001 0.001"/>
+        </geometry>
+      </collision>
+    </link>
+    <!-- Dummy link for the main control joint -->
     <link name="${prefix}finger_width_mock_link"/>
-    <!-- ====================== Main control joint (finger_width) ====================== -->
+    <!-- Main control joint (finger_width) -->
     <joint name="${prefix}finger_width" type="prismatic">
       <origin xyz="0 0 0" rpy="0 0 0"/>
@@ -79,5 +98,5 @@
       <limit lower="0.0" upper="0.15" velocity="0.25" effort="200"/>
     </joint>
-    <!-- ====================== Left Finger Joint (mimic) ====================== -->
+    <!-- Left Finger Joint -->
     <joint name="${prefix}left_finger_joint" type="prismatic">
       <origin xyz="-0.075 0 0" rpy="0 0 0"/>
@@ -88,5 +107,5 @@
       <mimic joint="${prefix}finger_width" multiplier="0.5" offset="0"/>
     </joint>
-    <!-- ====================== Right Finger Joint (mimic) ====================== -->
+    <!-- Right Finger Joint -->
     <joint name="${prefix}right_finger_joint" type="prismatic">
       <origin xyz="0.075 0 0" rpy="0 0 0"/>
@@ -94,8 +113,14 @@
       <child link="${prefix}right_finger_link"/>
       <axis xyz="-1 0 0"/>
-      <limit lower="-0.075" upper="0." effort="200" velocity="0.25"/>
+      <limit lower="-0.075" upper="0.0" effort="200" velocity="0.25"/>
       <mimic joint="${prefix}finger_width" multiplier="0.5" offset="0"/>
     </joint>
-    <!-- ====================== TCP Link ====================== -->
+    <!-- Middle Finger Joint (fixed for now, can be made movable if needed) -->
+    <joint name="${prefix}middle_finger_joint" type="fixed">
+      <origin xyz="0 0 0" rpy="0 0 0"/>
+      <parent link="${prefix}onrobot_base_link"/>
+      <child link="${prefix}middle_finger_link"/>
+    </joint>
+    <!-- TCP Link -->
     <link name="${prefix}gripper_tcp"/>
     <joint name="${prefix}tcp_joint" type="fixed">
@@ -104,5 +129,5 @@
       <child link="${prefix}gripper_tcp"/>
     </joint>
-    <!-- ====================== Transmission for ROS Control (IGUAL QUE 2FG7) ====================== -->
+    <!-- Transmission for ROS Control -->
     <xacro:transmission_macro prefix="${prefix}" joint_name="finger_width"/>
   </xacro:macro>

File: urdf/onrobot_macro.xacro (robot description, xacro)
@@ -29,5 +29,5 @@
       <xacro:onrobot_2fg7 prefix="${prefix}" onrobot_type="${onrobot_type}"/>
     </xacro:if>
-    <!-- ====================== 3FG15 (NUEVO) ====================== -->
+    <!-- ====================== 3FG15 ====================== -->
     <xacro:if value="${onrobot_type == '3fg15'}">
       <xacro:include filename="$(find onrobot_description)/urdf/3fg15_macro.xacro"/>
@@ -41,4 +41,11 @@
         </plugin>
       </gazebo>
+      <!-- Include Gazebo-specific plugins for each gripper type -->
+      <xacro:if value="${onrobot_type == '3fg15'}">
+        <xacro:include filename="$(find onrobot_description)/urdf/inc/3fg15_gazebo.xacro"/>
+        <xacro:onrobot_3fg15_grasp_plugin prefix="${prefix}"/>
+        <xacro:onrobot_3fg15_mimic_plugin prefix="${prefix}"/>
+        <xacro:onrobot_3fg15_gazebo_properties prefix="${prefix}"/>
+      </xacro:if>
     </xacro:if>
     <!-- ====================== ROS2 Control ====================== -->

Commit message: Working with decomposed stl files

File: urdf/3fg15_macro.xacro (robot description, xacro)
@@ -100,5 +100,5 @@
     <!-- Left Finger Joint -->
     <joint name="${prefix}left_finger_joint" type="prismatic">
-      <origin xyz="-0.075 0 0" rpy="0 0 0"/>
+      <origin xyz="0 0 0" rpy="0 0 0"/>
       <parent link="${prefix}onrobot_base_link"/>
       <child link="${prefix}left_finger_link"/>
@@ -109,5 +109,5 @@
     <!-- Right Finger Joint -->
     <joint name="${prefix}right_finger_joint" type="prismatic">
-      <origin xyz="0.075 0 0" rpy="0 0 0"/>
+      <origin xyz="0 0 0" rpy="0 0 0"/>
       <parent link="${prefix}onrobot_base_link"/>
       <child link="${prefix}right_finger_link"/>

Commit message: Revoluting fingers 3fg15

File: urdf/3fg15_macro.xacro (robot description, xacro)
@@ -3,10 +3,14 @@
   <xacro:include filename="$(find onrobot_description)/urdf/inc/common_utils.xacro" />
   <xacro:include filename="$(find onrobot_description)/urdf/inc/2fg7_materials.xacro" />
-  <!-- Macro for OnRobot 3FG15 gripper -->
+  <!-- Macro for OnRobot 3FG15 three-finger revolutionary gripper -->
   <xacro:macro name="onrobot_3fg15" params="prefix onrobot_type:='3fg15'">
+    <!-- Constants for 3FG15 -->
+    <xacro:property name="max_aperture" value="0.1175" /> <!-- 117.5mm in meters -->
+    <xacro:property name="min_aperture" value="0.0088" /> <!-- 8.8mm in meters -->
+    <xacro:property name="finger_radius" value="0.05875" /> <!-- Radius from center to finger tip -->
     <!-- Base Link -->
     <link name="${prefix}onrobot_base_link">
       <inertial>
-        <origin xyz="0 0 0.05" rpy="0 0 0"/>
+        <origin xyz="0 0 0" rpy="0 0 0"/>
         <mass value="1.2"/>
         <inertia ixx="0.012" ixy="0.0" ixz="0.0" iyy="0.012" iyz="0.0" izz="0.008"/>
@@ -26,10 +30,10 @@
       </collision>
     </link>
-    <!-- Finger Links with proper STL files -->
+    <!-- Left Finger Link -->
     <link name="${prefix}left_finger_link">
       <inertial>
         <origin xyz="0 0 0" rpy="0 0 0"/>
-        <mass value="0.1"/>
-        <inertia ixx="0.0001" ixy="0.0" ixz="0.0" iyy="0.0001" iyz="0.0" izz="0.0001"/>
+        <mass value="0.08"/>
+        <inertia ixx="0.00008" ixy="0.0" ixz="0.0" iyy="0.00008" iyz="0.0" izz="0.00008"/>
       </inertial>
       <visual>
@@ -47,9 +51,10 @@
       </collision>
     </link>
+    <!-- Right Finger Link -->
     <link name="${prefix}right_finger_link">
       <inertial>
         <origin xyz="0 0 0" rpy="0 0 0"/>
-        <mass value="0.1"/>
-        <inertia ixx="0.0001" ixy="0.0" ixz="0.0" iyy="0.0001" iyz="0.0" izz="0.0001"/>
+        <mass value="0.08"/>
+        <inertia ixx="0.00008" ixy="0.0" ixz="0.0" iyy="0.00008" iyz="0.0" izz="0.00008"/>
       </inertial>
       <visual>
@@ -71,6 +76,6 @@
       <inertial>
         <origin xyz="0 0 0" rpy="0 0 0"/>
-        <mass value="0.05"/>
-        <inertia ixx="0.00005" ixy="0.0" ixz="0.0" iyy="0.00005" iyz="0.0" izz="0.00005"/>
+        <mass value="0.08"/>
+        <inertia ixx="0.00008" ixy="0.0" ixz="0.0" iyy="0.00008" iyz="0.0" izz="0.00008"/>
       </inertial>
       <visual>
@@ -90,5 +95,5 @@
     <!-- Dummy link for the main control joint -->
     <link name="${prefix}finger_width_mock_link"/>
-    <!-- Main control joint (finger_width) -->
+    <!-- Main control joint (finger_width) - represents aperture diameter -->
     <joint name="${prefix}finger_width" type="prismatic">
       <origin xyz="0 0 0" rpy="0 0 0"/>
@@ -96,29 +101,32 @@
       <child link="${prefix}finger_width_mock_link"/>
       <axis xyz="0 0 1"/>
-      <limit lower="0.0" upper="0.15" velocity="0.25" effort="200"/>
+      <limit lower="${min_aperture}" upper="${max_aperture}" velocity="0.25" effort="200"/>
     </joint>
-    <!-- Left Finger Joint -->
-    <joint name="${prefix}left_finger_joint" type="prismatic">
+    <!-- Left Finger Joint (Revolute) -->
+    <joint name="${prefix}left_finger_joint" type="revolute">
       <origin xyz="0 0 0" rpy="0 0 0"/>
       <parent link="${prefix}onrobot_base_link"/>
       <child link="${prefix}left_finger_link"/>
-      <axis xyz="1 0 0"/>
-      <limit lower="0.0" upper="0.075" effort="200" velocity="0.25"/>
-      <mimic joint="${prefix}finger_width" multiplier="0.5" offset="0"/>
+      <axis xyz="0 0 1"/>
+      <limit lower="${-pi/3}" upper="${pi/3}" effort="200" velocity="0.25"/>
+      <mimic joint="${prefix}finger_width" multiplier="${(2*pi/3)/(max_aperture - min_aperture)}" offset="${-pi/3 - (2*pi/3)/(max_aperture - min_aperture) * min_aperture}"/>
     </joint>
-    <!-- Right Finger Joint -->
-    <joint name="${prefix}right_finger_joint" type="prismatic">
+    <!-- Right Finger Joint (Revolute) -->
+    <joint name="${prefix}right_finger_joint" type="revolute">
       <origin xyz="0 0 0" rpy="0 0 0"/>
       <parent link="${prefix}onrobot_base_link"/>
       <child link="${prefix}right_finger_link"/>
-      <axis xyz="-1 0 0"/>
-      <limit lower="-0.075" upper="0.0" effort="200" velocity="0.25"/>
-      <mimic joint="${prefix}finger_width" multiplier="0.5" offset="0"/>
+      <axis xyz="0 0 1"/>
+      <limit lower="${-pi/3}" upper="${pi/3}" effort="200" velocity="0.25"/>
+      <mimic joint="${prefix}finger_width" multiplier="${(2*pi/3)/(max_aperture - min_aperture)}" offset="${-pi/3 - (2*pi/3)/(max_aperture - min_aperture) * min_aperture}"/>
     </joint>
-    <!-- Middle Finger Joint (fixed for now, can be made movable if needed) -->
-    <joint name="${prefix}middle_finger_joint" type="fixed">
+    <!-- Middle Finger Joint (Revolute) -->
+    <joint name="${prefix}middle_finger_joint" type="revolute">
       <origin xyz="0 0 0" rpy="0 0 0"/>
       <parent link="${prefix}onrobot_base_link"/>
       <child link="${prefix}middle_finger_link"/>
+      <axis xyz="0 0 1"/>
+      <limit lower="${-pi/3}" upper="${pi/3}" effort="200" velocity="0.25"/>
+      <mimic joint="${prefix}finger_width" multiplier="${(2*pi/3)/(max_aperture - min_aperture)}" offset="${-pi/3 - (2*pi/3)/(max_aperture - min_aperture) * min_aperture}"/>
     </joint>
     <!-- TCP Link -->

File: urdf/inc/3fg15_gazebo.xacro (robot description, xacro)
@@ -12,22 +12,41 @@
           <gripper_link>${prefix}middle_finger_link</gripper_link>
         </arm>
-        <forces_angle_tolerance>80</forces_angle_tolerance>
-        <update_rate>10</update_rate>
-        <grip_count_threshold>1</grip_count_threshold>
-        <max_grip_count>3</max_grip_count>
-        <release_tolerance>0.01</release_tolerance>
-        <disable_collisions_on_attach>false</disable_collisions_on_attach>
+        <forces_angle_tolerance>100</forces_angle_tolerance>
+        <update_rate>15</update_rate>
+        <grip_count_threshold>2</grip_count_threshold>
+        <max_grip_count>4</max_grip_count>
+        <release_tolerance>0.005</release_tolerance>
+        <disable_collisions_on_attach>true</disable_collisions_on_attach>
         <contact_topic>__default_topic__</contact_topic>
       </plugin>
     </gazebo>
   </xacro:macro>
-  <!-- Mimic joint plugin for Gazebo -->
+  <!-- Mimic joint plugins for Gazebo for all three fingers -->
   <xacro:macro name="onrobot_3fg15_mimic_plugin" params="prefix">
+    <!-- Left finger mimic -->
     <gazebo>
-      <plugin filename="libroboticsgroup_upatras_gazebo_mimic_joint_plugin.so" name="mimic_3FG15">
-        <joint>${prefix}left_finger_joint</joint>
+      <plugin filename="libroboticsgroup_upatras_gazebo_mimic_joint_plugin.so" name="mimic_3fg15_left">
+        <joint>${prefix}finger_width</joint>
+        <mimicJoint>${prefix}left_finger_joint</mimicJoint>
+        <multiplier>${(2*pi/3)/(0.1175 - 0.0088)}</multiplier>
+        <offset>${-pi/3 - (2*pi/3)/(0.1175 - 0.0088) * 0.0088}</offset>
+      </plugin>
+    </gazebo>
+    <!-- Right finger mimic -->
+    <gazebo>
+      <plugin filename="libroboticsgroup_upatras_gazebo_mimic_joint_plugin.so" name="mimic_3fg15_right">
+        <joint>${prefix}finger_width</joint>
         <mimicJoint>${prefix}right_finger_joint</mimicJoint>
-        <multiplier>1.0</multiplier>
-        <offset>0.0</offset>
+        <multiplier>${(2*pi/3)/(0.1175 - 0.0088)}</multiplier>
+        <offset>${-pi/3 - (2*pi/3)/(0.1175 - 0.0088) * 0.0088}</offset>
+      </plugin>
+    </gazebo>
+    <!-- Middle finger mimic -->
+    <gazebo>
+      <plugin filename="libroboticsgroup_upatras_gazebo_mimic_joint_plugin.so" name="mimic_3fg15_middle">
+        <joint>${prefix}finger_width</joint>
+        <mimicJoint>${prefix}middle_finger_joint</mimicJoint>
+        <multiplier>${(2*pi/3)/(0.1175 - 0.0088)}</multiplier>
+        <offset>${-pi/3 - (2*pi/3)/(0.1175 - 0.0088) * 0.0088}</offset>
       </plugin>
     </gazebo>
@@ -36,30 +55,34 @@
   <xacro:macro name="onrobot_3fg15_gazebo_properties" params="prefix">
     <gazebo reference="${prefix}onrobot_base_link">
+      <material>Gazebo/DarkGrey</material>
+      <mu1>0.3</mu1>
+      <mu2>0.3</mu2>
+      <kp>100000000.0</kp>
+      <kd>1.5</kd>
+      <selfCollide>false</selfCollide>
+    </gazebo>
+    <gazebo reference="${prefix}left_finger_link">
       <material>Gazebo/Grey</material>
-      <mu1>0.2</mu1>
-      <mu2>0.2</mu2>
-      <kp>100000000.0</kp>
+      <mu1>0.4</mu1>
+      <mu2>0.4</mu2>
+      <kp>50000000.0</kp>
       <kd>1.0</kd>
+      <selfCollide>false</selfCollide>
     </gazebo>
     <gazebo reference="${prefix}right_finger_link">
       <material>Gazebo/Grey</material>
-      <mu1>0.2</mu1>
-      <mu2>0.2</mu2>
-      <kp>100000000.0</kp>
+      <mu1>0.4</mu1>
+      <mu2>0.4</mu2>
+      <kp>50000000.0</kp>
       <kd>1.0</kd>
-    </gazebo>
-    <gazebo reference="${prefix}left_finger_link">
-      <material>Gazebo/Grey</material>
-      <mu1>0.2</mu1>
-      <mu2>0.2</mu2>
-      <kp>100000000.0</kp>
-      <kd>1.0</kd>
+      <selfCollide>false</selfCollide>
     </gazebo>
     <gazebo reference="${prefix}middle_finger_link">
       <material>Gazebo/Grey</material>
-      <mu1>0.2</mu1>
-      <mu2>0.2</mu2>
-      <kp>100000000.0</kp>
+      <mu1>0.4</mu1>
+      <mu2>0.4</mu2>
+      <kp>50000000.0</kp>
       <kd>1.0</kd>
+      <selfCollide>false</selfCollide>
     </gazebo>
   </xacro:macro>
