Commit message: Revoluting fingers 3fg15 - fix 1

File: urdf/3fg15_macro.xacro (robot description, xacro)
@@ -3,11 +3,9 @@
   <xacro:include filename="$(find onrobot_description)/urdf/inc/common_utils.xacro" />
   <xacro:include filename="$(find onrobot_description)/urdf/inc/2fg7_materials.xacro" />
-  <!-- Macro for OnRobot 3FG15 three-finger revolutionary gripper -->
-  <xacro:macro name="onrobot_3fg15" params="prefix onrobot_type:='3fg15'">
-    <!-- Constants for 3FG15 -->
-    <xacro:property name="max_aperture" value="0.1175" /> <!-- 117.5mm in meters -->
-    <xacro:property name="min_aperture" value="0.0088" /> <!-- 8.8mm in meters -->
-    <xacro:property name="finger_radius" value="0.05875" /> <!-- Radius from center to finger tip -->
-    <!-- Base Link -->
+  <!-- Macro for OnRobot 3FG15 with rotation around RZ only -->
+  <xacro:macro name="onrobot_3fg15_rotatable" params="prefix">
+    <!-- Constants -->
+    <xacro:property name="finger_radius" value="0.05875" />
+    <!-- Base Link (fixed to robot) -->
     <link name="${prefix}onrobot_base_link">
       <inertial>
@@ -30,5 +28,14 @@
       </collision>
     </link>
-    <!-- Left Finger Link -->
+    <!-- Rotating frame: all fingers rotate together around Z -->
+    <link name="${prefix}rotating_frame"/>
+    <joint name="${prefix}gripper_rotation" type="revolute">
+      <parent link="${prefix}onrobot_base_link"/>
+      <child link="${prefix}rotating_frame"/>
+      <origin xyz="0 0 0" rpy="0 0 0"/>
+      <axis xyz="0 0 1"/>
+      <limit lower="-3.1416" upper="3.1416" effort="200" velocity="1.0"/>
+    </joint>
+    <!-- Left Finger (fixed pose, rotates with frame) -->
     <link name="${prefix}left_finger_link">
       <inertial>
@@ -51,5 +58,10 @@
       </collision>
     </link>
-    <!-- Right Finger Link -->
+    <joint name="${prefix}left_finger_fixed" type="fixed">
+      <parent link="${prefix}rotating_frame"/>
+      <child link="${prefix}left_finger_link"/>
+      <origin xyz="0 0 0" rpy="0 0 0"/>
+    </joint>
+    <!-- Right Finger -->
     <link name="${prefix}right_finger_link">
       <inertial>
@@ -72,5 +84,10 @@
       </collision>
     </link>
-    <!-- Middle Finger Link -->
+    <joint name="${prefix}right_finger_fixed" type="fixed">
+      <parent link="${prefix}rotating_frame"/>
+      <child link="${prefix}right_finger_link"/>
+      <origin xyz="0 0 0" rpy="0 0 0"/>
+    </joint>
+    <!-- Middle Finger -->
     <link name="${prefix}middle_finger_link">
       <inertial>
@@ -93,50 +110,18 @@
       </collision>
     </link>
-    <!-- Dummy link for the main control joint -->
-    <link name="${prefix}finger_width_mock_link"/>
-    <!-- Main control joint (finger_width) - represents aperture diameter -->
-    <joint name="${prefix}finger_width" type="prismatic">
+    <joint name="${prefix}middle_finger_fixed" type="fixed">
+      <parent link="${prefix}rotating_frame"/>
+      <child link="${prefix}middle_finger_link"/>
       <origin xyz="0 0 0" rpy="0 0 0"/>
-      <parent link="${prefix}onrobot_base_link"/>
-      <child link="${prefix}finger_width_mock_link"/>
-      <axis xyz="0 0 1"/>
-      <limit lower="${min_aperture}" upper="${max_aperture}" velocity="0.25" effort="200"/>
     </joint>
-    <!-- Left Finger Joint (Revolute) -->
-    <joint name="${prefix}left_finger_joint" type="revolute">
-      <origin xyz="0 0 0" rpy="0 0 0"/>
-      <parent link="${prefix}onrobot_base_link"/>
-      <child link="${prefix}left_finger_link"/>
-      <axis xyz="0 0 1"/>
-      <limit lower="${-pi/3}" upper="${pi/3}" effort="200" velocity="0.25"/>
-      <mimic joint="${prefix}finger_width" multiplier="${(2*pi/3)/(max_aperture - min_aperture)}" offset="${-pi/3 - (2*pi/3)/(max_aperture - min_aperture) * min_aperture}"/>
-    </joint>
-    <!-- Right Finger Joint (Revolute) -->
-    <joint name="${prefix}right_finger_joint" type="revolute">
-      <origin xyz="0 0 0" rpy="0 0 0"/>
-      <parent link="${prefix}onrobot_base_link"/>
-      <child link="${prefix}right_finger_link"/>
-      <axis xyz="0 0 1"/>
-      <limit lower="${-pi/3}" upper="${pi/3}" effort="200" velocity="0.25"/>
-      <mimic joint="${prefix}finger_width" multiplier="${(2*pi/3)/(max_aperture - min_aperture)}" offset="${-pi/3 - (2*pi/3)/(max_aperture - min_aperture) * min_aperture}"/>
-    </joint>
-    <!-- Middle Finger Joint (Revolute) -->
-    <joint name="${prefix}middle_finger_joint" type="revolute">
-      <origin xyz="0 0 0" rpy="0 0 0"/>
-      <parent link="${prefix}onrobot_base_link"/>
-      <child link="${prefix}middle_finger_link"/>
-      <axis xyz="0 0 1"/>
-      <limit lower="${-pi/3}" upper="${pi/3}" effort="200" velocity="0.25"/>
-      <mimic joint="${prefix}finger_width" multiplier="${(2*pi/3)/(max_aperture - min_aperture)}" offset="${-pi/3 - (2*pi/3)/(max_aperture - min_aperture) * min_aperture}"/>
-    </joint>
-    <!-- TCP Link -->
+    <!-- TCP Link (opcional, fijo al rotating_frame) -->
     <link name="${prefix}gripper_tcp"/>
     <joint name="${prefix}tcp_joint" type="fixed">
+      <parent link="${prefix}rotating_frame"/>
+      <child link="${prefix}gripper_tcp"/>
       <origin xyz="0 0 0.08" rpy="0 0 0"/>
-      <parent link="${prefix}onrobot_base_link"/>
-      <child link="${prefix}gripper_tcp"/>
     </joint>
-    <!-- Transmission for ROS Control -->
-    <xacro:transmission_macro prefix="${prefix}" joint_name="finger_width"/>
+    <!-- Transmission for rotation control -->
+    <xacro:transmission_macro prefix="${prefix}" joint_name="gripper_rotation"/>
   </xacro:macro>
 </robot>

Commit message: Revoluting fingers 3fg15 - fix 1 - ros2 humble

File: urdf/3fg15_macro.xacro (robot description, xacro)
@@ -3,9 +3,12 @@
   <xacro:include filename="$(find onrobot_description)/urdf/inc/common_utils.xacro" />
   <xacro:include filename="$(find onrobot_description)/urdf/inc/2fg7_materials.xacro" />
-  <!-- Macro for OnRobot 3FG15 with rotation around RZ only -->
-  <xacro:macro name="onrobot_3fg15_rotatable" params="prefix">
-    <!-- Constants -->
-    <xacro:property name="finger_radius" value="0.05875" />
-    <!-- Base Link (fixed to robot) -->
+  <!--
+    3FG15: Máxima apertura (117.5 mm), solo rota en RZ
+    100% compatible con ROS 2 Humble (sin cos/sin)
+  -->
+  <xacro:macro name="onrobot_3fg15_max_open_rotatable" params="prefix">
+    <!-- Posiciones precalculadas (máxima apertura) -->
+    <xacro:property name="finger_radius" value="0.05875" /> <!-- 117.5 / 2 -->
+    <!-- Base Link -->
     <link name="${prefix}onrobot_base_link">
       <inertial>
@@ -28,5 +31,5 @@
       </collision>
     </link>
-    <!-- Rotating frame: all fingers rotate together around Z -->
+    <!-- Marco rotativo -->
     <link name="${prefix}rotating_frame"/>
     <joint name="${prefix}gripper_rotation" type="revolute">
@@ -37,5 +40,5 @@
       <limit lower="-3.1416" upper="3.1416" effort="200" velocity="1.0"/>
     </joint>
-    <!-- Left Finger (fixed pose, rotates with frame) -->
+    <!-- === DEDO IZQUIERDO === -->
     <link name="${prefix}left_finger_link">
       <inertial>
@@ -61,7 +64,7 @@
       <parent link="${prefix}rotating_frame"/>
       <child link="${prefix}left_finger_link"/>
-      <origin xyz="0 0 0" rpy="0 0 0"/>
+      <origin xyz="0.05875 0.0 0" rpy="0 0 1.5708"/> <!-- 90° -->
     </joint>
-    <!-- Right Finger -->
+    <!-- === DEDO DERECHO === -->
     <link name="${prefix}right_finger_link">
       <inertial>
@@ -87,7 +90,7 @@
       <parent link="${prefix}rotating_frame"/>
       <child link="${prefix}right_finger_link"/>
-      <origin xyz="0 0 0" rpy="0 0 0"/>
+      <origin xyz="-0.029375 -0.050832 0" rpy="0 0 5.23599"/> <!-- 300° -->
     </joint>
-    <!-- Middle Finger -->
+    <!-- === DEDO MEDIO === -->
     <link name="${prefix}middle_finger_link">
       <inertial>
@@ -113,7 +116,7 @@
       <parent link="${prefix}rotating_frame"/>
       <child link="${prefix}middle_finger_link"/>
-      <origin xyz="0 0 0" rpy="0 0 0"/>
+      <origin xyz="-0.029375 0.050832 0" rpy="0 0 1.0472"/> <!-- 60° -->
     </joint>
-    <!-- TCP Link (opcional, fijo al rotating_frame) -->
+    <!-- TCP -->
     <link name="${prefix}gripper_tcp"/>
     <joint name="${prefix}tcp_joint" type="fixed">
@@ -122,5 +125,5 @@
       <origin xyz="0 0 0.08" rpy="0 0 0"/>
     </joint>
-    <!-- Transmission for rotation control -->
+    <!-- Transmisión -->
     <xacro:transmission_macro prefix="${prefix}" joint_name="gripper_rotation"/>
   </xacro:macro>

Commit message: Revoluting fingers 3fg15 - fix 2

File: urdf/3fg15_macro.xacro (robot description, xacro)
@@ -1,14 +1,11 @@
 <?xml version="1.0"?>
 <robot xmlns:xacro="http://ros.org/wiki/xacro">
-  <xacro:include filename="$(find onrobot_description)/urdf/inc/common_utils.xacro" />
-  <xacro:include filename="$(find onrobot_description)/urdf/inc/2fg7_materials.xacro" />
-  <!--
-    3FG15: Máxima apertura (117.5 mm), solo rota en RZ
-    100% compatible con ROS 2 Humble (sin cos/sin)
-  -->
-  <xacro:macro name="onrobot_3fg15_max_open_rotatable" params="prefix">
-    <!-- Posiciones precalculadas (máxima apertura) -->
-    <xacro:property name="finger_radius" value="0.05875" /> <!-- 117.5 / 2 -->
-    <!-- Base Link -->
+  <!-- ================================================================= -->
+  <!--  ONROBOT 3FG15 – VERSIÓN FIJA EN MÁXIMA APERTURA + SOLO ROTA EN RZ  -->
+  <!--  100% compatible con ROS 2 Humble (sin cos/sin/eval)               -->
+  <!--  Diámetro máximo fijo: 117.5 mm                                    -->
+  <!-- ================================================================= -->
+  <xacro:macro name="onrobot_3fg15" params="prefix">
+    <!-- ====================== BASE ====================== -->
     <link name="${prefix}onrobot_base_link">
       <inertial>
@@ -31,5 +28,5 @@
       </collision>
     </link>
-    <!-- Marco rotativo -->
+    <!-- =============== MARCO QUE ROTA (solo eje Z) =============== -->
     <link name="${prefix}rotating_frame"/>
     <joint name="${prefix}gripper_rotation" type="revolute">
@@ -38,7 +35,8 @@
       <origin xyz="0 0 0" rpy="0 0 0"/>
       <axis xyz="0 0 1"/>
-      <limit lower="-3.1416" upper="3.1416" effort="200" velocity="1.0"/>
+      <limit lower="-3.1416" upper="3.1416" effort="200" velocity="2.0"/>
+      <dynamics damping="0.7"/>
     </joint>
-    <!-- === DEDO IZQUIERDO === -->
+    <!-- ====================== DEDO IZQUIERDO ====================== -->
     <link name="${prefix}left_finger_link">
       <inertial>
@@ -64,7 +62,8 @@
       <parent link="${prefix}rotating_frame"/>
       <child link="${prefix}left_finger_link"/>
-      <origin xyz="0.05875 0.0 0" rpy="0 0 1.5708"/> <!-- 90° -->
+      <!-- Máxima apertura: radio = 58.75 mm, ángulo 90° -->
+      <origin xyz="0.05875 0 0" rpy="0 0 1.5708"/>
     </joint>
-    <!-- === DEDO DERECHO === -->
+    <!-- ====================== DEDO DERECHO ====================== -->
     <link name="${prefix}right_finger_link">
       <inertial>
@@ -90,7 +89,8 @@
       <parent link="${prefix}rotating_frame"/>
       <child link="${prefix}right_finger_link"/>
-      <origin xyz="-0.029375 -0.050832 0" rpy="0 0 5.23599"/> <!-- 300° -->
+      <!-- 210° → X = -0.029375, Y = -0.050832, rz total = 300° = 5.23599 rad -->
+      <origin xyz="-0.029375 -0.050832 0" rpy="0 0 5.23599"/>
     </joint>
-    <!-- === DEDO MEDIO === -->
+    <!-- ====================== DEDO MEDIO ====================== -->
     <link name="${prefix}middle_finger_link">
       <inertial>
@@ -116,7 +116,8 @@
       <parent link="${prefix}rotating_frame"/>
       <child link="${prefix}middle_finger_link"/>
-      <origin xyz="-0.029375 0.050832 0" rpy="0 0 1.0472"/> <!-- 60° -->
+      <!-- 330° → X = -0.029375, Y = +0.050832, rz total = 60° = 1.0472 rad -->
+      <origin xyz="-0.029375 0.050832 0" rpy="0 0 1.0472"/>
     </joint>
-    <!-- TCP -->
+    <!-- ====================== TCP ====================== -->
     <link name="${prefix}gripper_tcp"/>
     <joint name="${prefix}tcp_joint" type="fixed">
@@ -125,6 +126,14 @@
       <origin xyz="0 0 0.08" rpy="0 0 0"/>
     </joint>
-    <!-- Transmisión -->
-    <xacro:transmission_macro prefix="${prefix}" joint_name="gripper_rotation"/>
+    <!-- ====================== TRANSMISIÓN (para ROS Control) ====================== -->
+    <transmission name="${prefix}gripper_rotation_trans">
+      <type>transmission_interface/SimpleTransmission</type>
+      <joint name="${prefix}gripper_rotation">
+        <hardwareInterface>hardware_interface/EffortJointInterface</hardwareInterface>
+      </joint>
+      <actuator name="${prefix}gripper_rotation_motor">
+        <mechanicalReduction>1</mechanicalReduction>
+      </actuator>
+    </transmission>
   </xacro:macro>
 </robot>

Commit message: fixing materials error

File: urdf/3fg15_macro.xacro (robot description, xacro)
@@ -1,11 +1,13 @@
 <?xml version="1.0"?>
 <robot xmlns:xacro="http://ros.org/wiki/xacro">
-  <!-- ================================================================= -->
-  <!--  ONROBOT 3FG15 – VERSIÓN FIJA EN MÁXIMA APERTURA + SOLO ROTA EN RZ  -->
-  <!--  100% compatible con ROS 2 Humble (sin cos/sin/eval)               -->
-  <!--  Diámetro máximo fijo: 117.5 mm                                    -->
-  <!-- ================================================================= -->
-  <xacro:macro name="onrobot_3fg15" params="prefix">
-    <!-- ====================== BASE ====================== -->
+  <xacro:include filename="$(find onrobot_description)/urdf/inc/common_utils.xacro" />
+  <xacro:include filename="$(find onrobot_description)/urdf/inc/common_materials.xacro" />
+  <!-- Macro for OnRobot 3FG15 three-finger revolutionary gripper -->
+  <xacro:macro name="onrobot_3fg15" params="prefix onrobot_type:='3fg15'">
+    <!-- Constants for 3FG15 -->
+    <xacro:property name="max_aperture" value="0.1175" /> <!-- 117.5mm in meters -->
+    <xacro:property name="min_aperture" value="0.0088" /> <!-- 8.8mm in meters -->
+    <xacro:property name="finger_radius" value="0.05875" /> <!-- Radius from center to finger tip -->
+    <!-- Base Link -->
     <link name="${prefix}onrobot_base_link">
       <inertial>
@@ -28,15 +30,5 @@
       </collision>
     </link>
-    <!-- =============== MARCO QUE ROTA (solo eje Z) =============== -->
-    <link name="${prefix}rotating_frame"/>
-    <joint name="${prefix}gripper_rotation" type="revolute">
-      <parent link="${prefix}onrobot_base_link"/>
-      <child link="${prefix}rotating_frame"/>
-      <origin xyz="0 0 0" rpy="0 0 0"/>
-      <axis xyz="0 0 1"/>
-      <limit lower="-3.1416" upper="3.1416" effort="200" velocity="2.0"/>
-      <dynamics damping="0.7"/>
-    </joint>
-    <!-- ====================== DEDO IZQUIERDO ====================== -->
+    <!-- Left Finger Link -->
     <link name="${prefix}left_finger_link">
       <inertial>
@@ -59,11 +51,5 @@
       </collision>
     </link>
-    <joint name="${prefix}left_finger_fixed" type="fixed">
-      <parent link="${prefix}rotating_frame"/>
-      <child link="${prefix}left_finger_link"/>
-      <!-- Máxima apertura: radio = 58.75 mm, ángulo 90° -->
-      <origin xyz="0.05875 0 0" rpy="0 0 1.5708"/>
-    </joint>
-    <!-- ====================== DEDO DERECHO ====================== -->
+    <!-- Right Finger Link -->
     <link name="${prefix}right_finger_link">
       <inertial>
@@ -86,11 +72,5 @@
       </collision>
     </link>
-    <joint name="${prefix}right_finger_fixed" type="fixed">
-      <parent link="${prefix}rotating_frame"/>
-      <child link="${prefix}right_finger_link"/>
-      <!-- 210° → X = -0.029375, Y = -0.050832, rz total = 300° = 5.23599 rad -->
-      <origin xyz="-0.029375 -0.050832 0" rpy="0 0 5.23599"/>
-    </joint>
-    <!-- ====================== DEDO MEDIO ====================== -->
+    <!-- Middle Finger Link -->
     <link name="${prefix}middle_finger_link">
       <inertial>
@@ -113,27 +93,50 @@
       </collision>
     </link>
-    <joint name="${prefix}middle_finger_fixed" type="fixed">
-      <parent link="${prefix}rotating_frame"/>
+    <!-- Dummy link for the main control joint -->
+    <link name="${prefix}finger_width_mock_link"/>
+    <!-- Main control joint (finger_width) - represents aperture diameter -->
+    <joint name="${prefix}finger_width" type="prismatic">
+      <origin xyz="0 0 0" rpy="0 0 0"/>
+      <parent link="${prefix}onrobot_base_link"/>
+      <child link="${prefix}finger_width_mock_link"/>
+      <axis xyz="0 0 1"/>
+      <limit lower="${min_aperture}" upper="${max_aperture}" velocity="0.25" effort="200"/>
+    </joint>
+    <!-- Left Finger Joint (Revolute) -->
+    <joint name="${prefix}left_finger_joint" type="revolute">
+      <origin xyz="0 0 0" rpy="0 0 0"/>
+      <parent link="${prefix}onrobot_base_link"/>
+      <child link="${prefix}left_finger_link"/>
+      <axis xyz="0 0 1"/>
+      <limit lower="${-pi/3}" upper="${pi/3}" effort="200" velocity="0.25"/>
+      <mimic joint="${prefix}finger_width" multiplier="${(2*pi/3)/(max_aperture - min_aperture)}" offset="${-pi/3 - (2*pi/3)/(max_aperture - min_aperture) * min_aperture}"/>
+    </joint>
+    <!-- Right Finger Joint (Revolute) -->
+    <joint name="${prefix}right_finger_joint" type="revolute">
+      <origin xyz="0 0 0" rpy="0 0 0"/>
+      <parent link="${prefix}onrobot_base_link"/>
+      <child link="${prefix}right_finger_link"/>
+      <axis xyz="0 0 1"/>
+      <limit lower="${-pi/3}" upper="${pi/3}" effort="200" velocity="0.25"/>
+      <mimic joint="${prefix}finger_width" multiplier="${(2*pi/3)/(max_aperture - min_aperture)}" offset="${-pi/3 - (2*pi/3)/(max_aperture - min_aperture) * min_aperture}"/>
+    </joint>
+    <!-- Middle Finger Joint (Revolute) -->
+    <joint name="${prefix}middle_finger_joint" type="revolute">
+      <origin xyz="0 0 0" rpy="0 0 0"/>
+      <parent link="${prefix}onrobot_base_link"/>
       <child link="${prefix}middle_finger_link"/>
-      <!-- 330° → X = -0.029375, Y = +0.050832, rz total = 60° = 1.0472 rad -->
-      <origin xyz="-0.029375 0.050832 0" rpy="0 0 1.0472"/>
+      <axis xyz="0 0 1"/>
+      <limit lower="${-pi/3}" upper="${pi/3}" effort="200" velocity="0.25"/>
+      <mimic joint="${prefix}finger_width" multiplier="${(2*pi/3)/(max_aperture - min_aperture)}" offset="${-pi/3 - (2*pi/3)/(max_aperture - min_aperture) * min_aperture}"/>
     </joint>
-    <!-- ====================== TCP ====================== -->
+    <!-- TCP Link -->
     <link name="${prefix}gripper_tcp"/>
     <joint name="${prefix}tcp_joint" type="fixed">
-      <parent link="${prefix}rotating_frame"/>
+      <origin xyz="0 0 0.08" rpy="0 0 0"/>
+      <parent link="${prefix}onrobot_base_link"/>
       <child link="${prefix}gripper_tcp"/>
-      <origin xyz="0 0 0.08" rpy="0 0 0"/>
     </joint>
-    <!-- ====================== TRANSMISIÓN (para ROS Control) ====================== -->
-    <transmission name="${prefix}gripper_rotation_trans">
-      <type>transmission_interface/SimpleTransmission</type>
-      <joint name="${prefix}gripper_rotation">
-        <hardwareInterface>hardware_interface/EffortJointInterface</hardwareInterface>
-      </joint>
-      <actuator name="${prefix}gripper_rotation_motor">
-        <mechanicalReduction>1</mechanicalReduction>
-      </actuator>
-    </transmission>
+    <!-- Transmission for ROS Control -->
+    <xacro:transmission_macro prefix="${prefix}" joint_name="finger_width"/>
   </xacro:macro>
 </robot>

File: urdf/onrobot_macro.xacro (robot description, xacro)
@@ -13,4 +13,5 @@
         port:=502
         device_address:=65
+        auto_detect:=false
         ">
         <xacro:if value="${onrobot_type == 'rg2'}">
@@ -60,5 +61,6 @@
                         <param name="port">${port}</param>
                         <param name="device_address">${device_address}</param>
-                        <param name="use_fake_hardware">false</param>
+                        <param name="use_fake_hardware">${use_fake_hardware}</param>
+                        <param name="auto_detect">${auto_detect}</param>
                     </xacro:if>
                     <xacro:if value="${onrobot_type == '3fg15' or onrobot_type == '3fg25'}">
@@ -71,5 +73,6 @@
                         <param name="port">${port}</param>
                         <param name="device_address">${device_address}</param>
-                        <param name="use_fake_hardware">false</param>
+                        <param name="use_fake_hardware">${use_fake_hardware}</param>
+                        <param name="auto_detect">${auto_detect}</param>
                     </xacro:if>
                     <xacro:if value="${onrobot_type == 'vg10' or onrobot_type == 'vgc10'}">
@@ -82,5 +85,6 @@
                         <param name="port">${port}</param>
                         <param name="device_address">${device_address}</param>
-                        <param name="use_fake_hardware">false</param>
+                        <param name="use_fake_hardware">${use_fake_hardware}</param>
+                        <param name="auto_detect">${auto_detect}</param>
                     </xacro:if>
                     <xacro:if value="${onrobot_type == 'rg2' or onrobot_type == 'rg6'}">
@@ -92,5 +96,6 @@
                         <param name="ip_address">${ip_address}</param>
                         <param name="port">${port}</param>
-                        <param name="use_fake_hardware">false</param>
+                        <param name="use_fake_hardware">${use_fake_hardware}</param>
+                        <param name="auto_detect">${auto_detect}</param>
                     </xacro:if>
                 </hardware>

Commit message: 3fg15_macro update

File: urdf/3fg15_macro.xacro (robot description, xacro)
@@ -96,5 +96,5 @@
     <link name="${prefix}finger_width_mock_link"/>
     <!-- Main control joint (finger_width) - represents aperture diameter -->
-    <joint name="${prefix}finger_width" type="prismatic">
+    <joint name="${prefix}finger_width" type="revolute">
       <origin xyz="0 0 0" rpy="0 0 0"/>
       <parent link="${prefix}onrobot_base_link"/>
