Commit message: 3fg15_macro update

File: urdf/3fg15_macro.xacro (robot description, xacro)
@@ -2,14 +2,13 @@
 <robot xmlns:xacro="http://ros.org/wiki/xacro">
   <xacro:include filename="$(find onrobot_description)/urdf/inc/common_utils.xacro" />
-  <!-- Macro for OnRobot 3FG15 three-finger revolutionary gripper -->
+  <!-- Macro para OnRobot 3FG15 -->
   <xacro:macro name="onrobot_3fg15" params="prefix onrobot_type:='3fg15'">
-    <!-- Constants for 3FG15 -->
-    <xacro:property name="max_aperture" value="0.1175" /> <!-- 117.5mm in meters -->
-    <xacro:property name="min_aperture" value="0.0088" /> <!-- 8.8mm in meters -->
-    <xacro:property name="finger_radius" value="0.05875" /> <!-- Radius from center to finger tip -->
+    <!-- Constantes -->
+    <xacro:property name="min_diameter" value="0.000" />
+    <xacro:property name="max_diameter" value="0.150" />
     <!-- Base Link -->
     <link name="${prefix}onrobot_base_link">
       <inertial>
-        <origin xyz="0 0 0" rpy="0 0 0"/>
+        <origin xyz="0 0 0.04" rpy="0 0 0"/>
         <mass value="1.2"/>
         <inertia ixx="0.012" ixy="0.0" ixz="0.0" iyy="0.012" iyz="0.0" izz="0.008"/>
@@ -20,8 +19,7 @@
           <mesh filename="package://onrobot_description/meshes/3fg15/visual/base.stl" scale="0.001 0.001 0.001"/>
         </geometry>
-        <material name="onrobot_silver"/>
       </visual>
       <collision>
-        <origin xyz="0 0 0" rpy="0 0 0"/>
+        <origin xyz="0 0 0.04" rpy="0 0 0"/>
         <geometry>
           <mesh filename="package://onrobot_description/meshes/3fg15/collision/base.stl" scale="0.001 0.001 0.001"/>
@@ -29,5 +27,6 @@
       </collision>
     </link>
-    <!-- Left Finger Link -->
+    <!-- === DEDOS (con movimiento real via mimic) === -->
+    <!-- Left Finger -->
     <link name="${prefix}left_finger_link">
       <inertial>
@@ -41,5 +40,4 @@
           <mesh filename="package://onrobot_description/meshes/3fg15/visual/left_finger.stl" scale="0.001 0.001 0.001"/>
         </geometry>
-        <material name="onrobot_silver"/>
       </visual>
       <collision>
@@ -50,5 +48,5 @@
       </collision>
     </link>
-    <!-- Right Finger Link -->
+    <!-- Right Finger -->
     <link name="${prefix}right_finger_link">
       <inertial>
@@ -62,5 +60,4 @@
           <mesh filename="package://onrobot_description/meshes/3fg15/visual/right_finger.stl" scale="0.001 0.001 0.001"/>
         </geometry>
-        <material name="onrobot_silver"/>
       </visual>
       <collision>
@@ -71,5 +68,5 @@
       </collision>
     </link>
-    <!-- Middle Finger Link -->
+    <!-- Middle Finger -->
     <link name="${prefix}middle_finger_link">
       <inertial>
@@ -83,5 +80,4 @@
           <mesh filename="package://onrobot_description/meshes/3fg15/visual/middle_finger.stl" scale="0.001 0.001 0.001"/>
         </geometry>
-        <material name="onrobot_silver"/>
       </visual>
       <collision>
@@ -92,50 +88,54 @@
       </collision>
     </link>
-    <!-- Dummy link for the main control joint -->
+    <!-- Dummy link para control -->
     <link name="${prefix}finger_width_mock_link"/>
-    <!-- Main control joint (finger_width) - represents aperture diameter -->
-    <joint name="${prefix}finger_width" type="revolute">
-      <origin xyz="0 0 0" rpy="0 0 0"/>
+    <!-- JOINT PRINCIPAL (para el driver) -->
+    <joint name="${prefix}finger_diameter" type="prismatic">
       <parent link="${prefix}onrobot_base_link"/>
       <child link="${prefix}finger_width_mock_link"/>
-      <axis xyz="0 0 1"/>
-      <limit lower="${min_aperture}" upper="${max_aperture}" velocity="0.25" effort="200"/>
+      <origin xyz="0 0 0" rpy="0 0 0"/>
+      <axis xyz="0 1 0"/>
+      <limit lower="0.0" upper="0.150" effort="200" velocity="0.5"/>
     </joint>
-    <!-- Left Finger Joint (Revolute) -->
+    <!-- === DEDOS: REVOLUTE + MIMIC === -->
+    <xacro:property name="angle_per_meter" value="${(2*pi/3)/(0.150 - 0.0)}" />  <!-- 120° en 150mm -->
+    <xacro:property name="min_angle" value="${-pi/3}" />  <!-- -60° -->
+    <xacro:property name="offset" value="${min_angle - angle_per_meter * 0.0}" />
+    <!-- Left Finger -->
     <joint name="${prefix}left_finger_joint" type="revolute">
-      <origin xyz="0 0 0" rpy="0 0 0"/>
       <parent link="${prefix}onrobot_base_link"/>
       <child link="${prefix}left_finger_link"/>
+      <origin xyz="0 0 0" rpy="${pi}" />
       <axis xyz="0 0 1"/>
-      <limit lower="${-pi/3}" upper="${pi/3}" effort="200" velocity="0.25"/>
-      <mimic joint="${prefix}finger_width" multiplier="${(2*pi/3)/(max_aperture - min_aperture)}" offset="${-pi/3 - (2*pi/3)/(max_aperture - min_aperture) * min_aperture}"/>
+      <limit lower="${-pi/3}" upper="${pi/3}" effort="200" velocity="0.5"/>
+      <mimic joint="${prefix}finger_diameter" multiplier="${angle_per_meter}" offset="${offset}"/>
     </joint>
-    <!-- Right Finger Joint (Revolute) -->
+    <!-- Right Finger -->
     <joint name="${prefix}right_finger_joint" type="revolute">
-      <origin xyz="0 0 0" rpy="0 0 0"/>
       <parent link="${prefix}onrobot_base_link"/>
       <child link="${prefix}right_finger_link"/>
+      <origin xyz="0 0 0" rpy="0" />
       <axis xyz="0 0 1"/>
-      <limit lower="${-pi/3}" upper="${pi/3}" effort="200" velocity="0.25"/>
-      <mimic joint="${prefix}finger_width" multiplier="${(2*pi/3)/(max_aperture - min_aperture)}" offset="${-pi/3 - (2*pi/3)/(max_aperture - min_aperture) * min_aperture}"/>
+      <limit lower="${-pi/3}" upper="${pi/3}" effort="200" velocity="0.5"/>
+      <mimic joint="${prefix}finger_diameter" multiplier="${angle_per_meter}" offset="${offset}"/>
     </joint>
-    <!-- Middle Finger Joint (Revolute) -->
+    <!-- Middle Finger -->
     <joint name="${prefix}middle_finger_joint" type="revolute">
-      <origin xyz="0 0 0" rpy="0 0 0"/>
       <parent link="${prefix}onrobot_base_link"/>
       <child link="${prefix}middle_finger_link"/>
+      <origin xyz="0 0 0" rpy="${2*pi/3}" />
       <axis xyz="0 0 1"/>
-      <limit lower="${-pi/3}" upper="${pi/3}" effort="200" velocity="0.25"/>
-      <mimic joint="${prefix}finger_width" multiplier="${(2*pi/3)/(max_aperture - min_aperture)}" offset="${-pi/3 - (2*pi/3)/(max_aperture - min_aperture) * min_aperture}"/>
+      <limit lower="${-pi/3}" upper="${pi/3}" effort="200" velocity="0.5"/>
+      <mimic joint="${prefix}finger_diameter" multiplier="${angle_per_meter}" offset="${offset}"/>
     </joint>
-    <!-- TCP Link -->
+    <!-- TCP -->
     <link name="${prefix}gripper_tcp"/>
     <joint name="${prefix}tcp_joint" type="fixed">
-      <origin xyz="0 0 0.08" rpy="0 0 0"/>
       <parent link="${prefix}onrobot_base_link"/>
       <child link="${prefix}gripper_tcp"/>
+      <origin xyz="0 0 0.13" rpy="0 0 0"/>
     </joint>
-    <!-- Transmission for ROS Control -->
-    <xacro:transmission_macro prefix="${prefix}" joint_name="finger_width"/>
+    <!-- Transmission -->
+    <xacro:transmission_macro prefix="${prefix}" joint_name="finger_diameter"/>
   </xacro:macro>
 </robot>

File: urdf/onrobot_macro.xacro (robot description, xacro)
@@ -37,9 +37,4 @@
       <xacro:onrobot_3fg15 prefix="${prefix}"/>
     </xacro:if>
-    <!-- ====================== VG10 (legacy) ====================== -->
-    <xacro:if value="${onrobot_type == 'vg10'}">
-      <xacro:include filename="$(find onrobot_description)/urdf/vg_macro.xacro"/>
-      <xacro:onrobot_vg prefix="${prefix}" onrobot_type="vg10" num_cups="${num_cups}"/>
-    </xacro:if>
     <!-- ====================== VGC10 ====================== -->
     <xacro:if value="${onrobot_type == 'vgc10'}">
@@ -65,27 +60,24 @@
     <!-- ====================== ROS2 CONTROL (REAL) ====================== -->
     <xacro:unless value="${use_fake_hardware}">
-      <ros2_control name="OnRobotGripper" type="actuator">
+      <ros2_control name="OnRobotGripper" type="system">
         <hardware>
-          <!-- 2FG7 / 2FG14 -->
-          <xacro:if value="${onrobot_type == '2fg7' or onrobot_type == '2fg14'}">
-            <plugin>onrobot_driver::TwoFGHardwareInterface</plugin>
-            <param name="onrobot_type">${onrobot_type}</param>
-          </xacro:if>
-          <!-- 3FG15 -->
+          <!-- Selección del plugin según tipo -->
           <xacro:if value="${onrobot_type == '3fg15'}">
             <plugin>onrobot_driver::ThreeFGHardwareInterface</plugin>
-            <param name="onrobot_type">${onrobot_type}</param>
           </xacro:if>
-          <!-- RG2 / RG6 -->
-          <xacro:if value="${onrobot_type == 'rg2' or onrobot_type == 'rg6'}">
+          <xacro:elseif value="${onrobot_type == '2fg7' or onrobot_type == '2fg14'}">
+            <plugin>onrobot_driver::TwoFGHardwareInterface</plugin>
+          </xacro:elseif>
+          <xacro:elseif value="${onrobot_type == 'rg2' or onrobot_type == 'rg6'}">
             <plugin>onrobot_driver::RGHardwareInterface</plugin>
-            <param name="onrobot_type">${onrobot_type}</param>
-          </xacro:if>
-          <!-- VGC10 -->
-          <xacro:if value="${onrobot_type == 'vgc10'}">
+          </xacro:elseif>
+          <xacro:elseif value="${onrobot_type == 'vgc10'}">
             <plugin>onrobot_driver::VGCHardwareInterface</plugin>
-            <param name="onrobot_type">vgc10</param>
-          </xacro:if>
+          </xacro:elseif>
+          <xacro:else>
+            <plugin>onrobot_driver::TwoFGHardwareInterface</plugin> <!-- fallback -->
+          </xacro:else>
           <!-- Parámetros comunes -->
+          <param name="onrobot_type">${onrobot_type}</param>
           <param name="prefix">${prefix}</param>
           <param name="connection_type">${connection_type}</param>
@@ -96,10 +88,19 @@
           <param name="use_fake_hardware">false</param>
         </hardware>
-        <!-- Joint de control (mismo nombre en todos los macros) -->
-        <joint name="${prefix}gripper">
-          <command_interface name="position"/>
-          <state_interface name="position"/>
-          <state_interface name="velocity"/>
-        </joint>
+        <!-- JOINT DE CONTROL SEGÚN TIPO -->
+        <xacro:if value="${onrobot_type == '3fg15'}">
+          <joint name="${prefix}finger_diameter">
+            <command_interface name="position"/>
+            <state_interface name="position"/>
+            <state_interface name="velocity"/>
+          </joint>
+        </xacro:if>
+        <xacro:unless value="${onrobot_type == '3fg15'}">
+          <joint name="${prefix}finger_width">
+            <command_interface name="position"/>
+            <state_interface name="position"/>
+            <state_interface name="velocity"/>
+          </joint>
+        </xacro:unless>
       </ros2_control>
     </xacro:unless>

Commit message: Fix package 1 - angle fix

File: urdf/3fg15_macro.xacro (robot description, xacro)
@@ -1,11 +1,20 @@
 <?xml version="1.0"?>
 <robot xmlns:xacro="http://ros.org/wiki/xacro">
+  <!-- Incluir utilidades comunes y funciones matemáticas -->
   <xacro:include filename="$(find onrobot_description)/urdf/inc/common_utils.xacro" />
+  <xacro:include filename="$(find xacro)/xacro/math.xacro" /> <!-- Proporciona M_PI, sin(), cos(), etc. -->
   <!-- Macro para OnRobot 3FG15 -->
   <xacro:macro name="onrobot_3fg15" params="prefix onrobot_type:='3fg15'">
-    <!-- Constantes -->
-    <xacro:property name="min_diameter" value="0.000" />
-    <xacro:property name="max_diameter" value="0.150" />
-    <!-- Base Link -->
+    <!-- === CONSTANTES DEL GRIPPER === -->
+    <xacro:property name="min_diameter" value="0.000" />  <!-- m -->
+    <xacro:property name="max_diameter" value="0.150" />  <!-- m (150 mm) -->
+    <!-- Ángulo total por dedo: 120° = 2π/3 rad -->
+    <xacro:property name="total_angle" value="${2 * M_PI / 3}" />  <!-- 120° en radianes -->
+    <xacro:property name="angle_per_meter" value="${total_angle / (max_diameter - min_diameter)}" />
+    <xacro:property name="min_angle" value="${-M_PI / 3}" />      <!-- -60° -->
+    <xacro:property name="max_angle" value="${ M_PI / 3}" />      <!-- +60° -->
+    <!-- Offset para que en diámetro=0 → ángulo = -60° -->
+    <xacro:property name="mimic_offset" value="${min_angle}" />
+    <!-- === BASE LINK === -->
     <link name="${prefix}onrobot_base_link">
       <inertial>
@@ -27,5 +36,5 @@
       </collision>
     </link>
-    <!-- === DEDOS (con movimiento real via mimic) === -->
+    <!-- === DEDOS === -->
     <!-- Left Finger -->
     <link name="${prefix}left_finger_link">
@@ -88,7 +97,7 @@
       </collision>
     </link>
-    <!-- Dummy link para control -->
+    <!-- Dummy link para control de ancho -->
     <link name="${prefix}finger_width_mock_link"/>
-    <!-- JOINT PRINCIPAL (para el driver) -->
+    <!-- === JOINT PRINCIPAL (controlado por el driver) === -->
     <joint name="${prefix}finger_diameter" type="prismatic">
       <parent link="${prefix}onrobot_base_link"/>
@@ -96,45 +105,42 @@
       <origin xyz="0 0 0" rpy="0 0 0"/>
       <axis xyz="0 1 0"/>
-      <limit lower="0.0" upper="0.150" effort="200" velocity="0.5"/>
+      <limit lower="${min_diameter}" upper="${max_diameter}" effort="200" velocity="0.5"/>
     </joint>
     <!-- === DEDOS: REVOLUTE + MIMIC === -->
-    <xacro:property name="angle_per_meter" value="${(2*pi/3)/(0.150 - 0.0)}" />  <!-- 120° en 150mm -->
-    <xacro:property name="min_angle" value="${-pi/3}" />  <!-- -60° -->
-    <xacro:property name="offset" value="${min_angle - angle_per_meter * 0.0}" />
-    <!-- Left Finger -->
+    <!-- Left Finger (rotado 180°) -->
     <joint name="${prefix}left_finger_joint" type="revolute">
       <parent link="${prefix}onrobot_base_link"/>
       <child link="${prefix}left_finger_link"/>
-      <origin xyz="0 0 0" rpy="${pi}" />
+      <origin xyz="0 0 0" rpy="${M_PI} 0 0"/>   <!-- 180° -->
       <axis xyz="0 0 1"/>
-      <limit lower="${-pi/3}" upper="${pi/3}" effort="200" velocity="0.5"/>
-      <mimic joint="${prefix}finger_diameter" multiplier="${angle_per_meter}" offset="${offset}"/>
+      <limit lower="${min_angle}" upper="${max_angle}" effort="200" velocity="0.5"/>
+      <mimic joint="${prefix}finger_diameter" multiplier="${angle_per_meter}" offset="${mimic_offset}"/>
     </joint>
-    <!-- Right Finger -->
+    <!-- Right Finger (0°) -->
     <joint name="${prefix}right_finger_joint" type="revolute">
       <parent link="${prefix}onrobot_base_link"/>
       <child link="${prefix}right_finger_link"/>
-      <origin xyz="0 0 0" rpy="0" />
+      <origin xyz="0 0 0" rpy="0 0 0"/>
       <axis xyz="0 0 1"/>
-      <limit lower="${-pi/3}" upper="${pi/3}" effort="200" velocity="0.5"/>
-      <mimic joint="${prefix}finger_diameter" multiplier="${angle_per_meter}" offset="${offset}"/>
+      <limit lower="${min_angle}" upper="${max_angle}" effort="200" velocity="0.5"/>
+      <mimic joint="${prefix}finger_diameter" multiplier="${angle_per_meter}" offset="${mimic_offset}"/>
     </joint>
-    <!-- Middle Finger -->
+    <!-- Middle Finger (120°) -->
     <joint name="${prefix}middle_finger_joint" type="revolute">
       <parent link="${prefix}onrobot_base_link"/>
       <child link="${prefix}middle_finger_link"/>
-      <origin xyz="0 0 0" rpy="${2*pi/3}" />
+      <origin xyz="0 0 0" rpy="${2 * M_PI / 3} 0 0"/>  <!-- 120° -->
       <axis xyz="0 0 1"/>
-      <limit lower="${-pi/3}" upper="${pi/3}" effort="200" velocity="0.5"/>
-      <mimic joint="${prefix}finger_diameter" multiplier="${angle_per_meter}" offset="${offset}"/>
+      <limit lower="${min_angle}" upper="${max_angle}" effort="200" velocity="0.5"/>
+      <mimic joint="${prefix}finger_diameter" multiplier="${angle_per_meter}" offset="${mimic_offset}"/>
     </joint>
-    <!-- TCP -->
+    <!-- === TCP (Tool Center Point) === -->
     <link name="${prefix}gripper_tcp"/>
     <joint name="${prefix}tcp_joint" type="fixed">
       <parent link="${prefix}onrobot_base_link"/>
       <child link="${prefix}gripper_tcp"/>
-      <origin xyz="0 0 0.13" rpy="0 0 0"/>
+      <origin xyz="0 0 0.13" rpy="0 0 0"/>  <!-- 130 mm hacia adelante -->
     </joint>
-    <!-- Transmission -->
+    <!-- === TRANSMISSION (para ROS Control) === -->
     <xacro:transmission_macro prefix="${prefix}" joint_name="finger_diameter"/>
   </xacro:macro>
