Commit message: onrobot_driver_integration + 3fg15 diff approach

File: urdf/3fg15_macro.xacro (robot description, xacro)
@@ -1,16 +1,14 @@
 <?xml version="1.0"?>
 <robot xmlns:xacro="http://ros.org/wiki/xacro">
-  <!-- ================================================================= -->
-  <!--  ONROBOT 3FG15 – VERSIÓN FIJA EN MÁXIMA APERTURA + SOLO ROTA EN RZ  -->
-  <!--  100% compatible con ROS 2 Humble (sin cos/sin/eval)               -->
-  <!--  Diámetro máximo fijo: 117.5 mm                                    -->
-  <!-- ================================================================= -->
-  <xacro:macro name="onrobot_3fg15" params="prefix">
-    <!-- ====================== BASE ====================== -->
+  <xacro:include filename="$(find onrobot_description)/urdf/inc/common_utils.xacro" />
+  <xacro:include filename="$(find onrobot_description)/urdf/inc/common_materials.xacro" />
+  <!-- 3FG15 Macro - Proper 3-finger centripetal gripper with revolute joints -->
+  <xacro:macro name="onrobot_3fg15" params="prefix onrobot_type:='3fg15'">
+    <!-- Base Link -->
     <link name="${prefix}onrobot_base_link">
       <inertial>
         <origin xyz="0 0 0" rpy="0 0 0"/>
-        <mass value="1.2"/>
-        <inertia ixx="0.012" ixy="0.0" ixz="0.0" iyy="0.012" iyz="0.0" izz="0.008"/>
+        <mass value="1.8"/>
+        <inertia ixx="0.015" ixy="0.0" ixz="0.0" iyy="0.015" iyz="0.0" izz="0.010"/>
       </inertial>
       <visual>
@@ -28,20 +26,10 @@
       </collision>
     </link>
-    <!-- =============== MARCO QUE ROTA (solo eje Z) =============== -->
-    <link name="${prefix}rotating_frame"/>
-    <joint name="${prefix}gripper_rotation" type="revolute">
-      <parent link="${prefix}onrobot_base_link"/>
-      <child link="${prefix}rotating_frame"/>
-      <origin xyz="0 0 0" rpy="0 0 0"/>
-      <axis xyz="0 0 1"/>
-      <limit lower="-3.1416" upper="3.1416" effort="200" velocity="2.0"/>
-      <dynamics damping="0.7"/>
-    </joint>
-    <!-- ====================== DEDO IZQUIERDO ====================== -->
+    <!-- Finger Links -->
     <link name="${prefix}left_finger_link">
       <inertial>
         <origin xyz="0 0 0" rpy="0 0 0"/>
-        <mass value="0.08"/>
-        <inertia ixx="0.00008" ixy="0.0" ixz="0.0" iyy="0.00008" iyz="0.0" izz="0.00008"/>
+        <mass value="0.1"/>
+        <inertia ixx="0.0001" ixy="0.0" ixz="0.0" iyy="0.0001" iyz="0.0" izz="0.0001"/>
       </inertial>
       <visual>
@@ -55,20 +43,33 @@
         <origin xyz="0 0 0" rpy="0 0 0"/>
         <geometry>
-          <mesh filename="package://onrobot_description/meshes/3fg15/collision/left_finger.stl" scale="0.001 0.001 0.001"/>
+          <box size="0.01 0.02 0.06"/>
         </geometry>
       </collision>
     </link>
-    <joint name="${prefix}left_finger_fixed" type="fixed">
-      <parent link="${prefix}rotating_frame"/>
-      <child link="${prefix}left_finger_link"/>
-      <!-- Máxima apertura: radio = 58.75 mm, ángulo 90° -->
-      <origin xyz="0.05875 0 0" rpy="0 0 1.5708"/>
-    </joint>
-    <!-- ====================== DEDO DERECHO ====================== -->
+    <link name="${prefix}middle_finger_link">
+      <inertial>
+        <origin xyz="0 0 0" rpy="0 0 0"/>
+        <mass value="0.1"/>
+        <inertia ixx="0.0001" ixy="0.0" ixz="0.0" iyy="0.0001" iyz="0.0" izz="0.0001"/>
+      </inertial>
+      <visual>
+        <origin xyz="0 0 0" rpy="0 0 0"/>
+        <geometry>
+          <mesh filename="package://onrobot_description/meshes/3fg15/visual/middle_finger.stl" scale="0.001 0.001 0.001"/>
+        </geometry>
+        <material name="onrobot_silver"/>
+      </visual>
+      <collision>
+        <origin xyz="0 0 0" rpy="0 0 0"/>
+        <geometry>
+          <box size="0.01 0.02 0.06"/>
+        </geometry>
+      </collision>
+    </link>
     <link name="${prefix}right_finger_link">
       <inertial>
         <origin xyz="0 0 0" rpy="0 0 0"/>
-        <mass value="0.08"/>
-        <inertia ixx="0.00008" ixy="0.0" ixz="0.0" iyy="0.00008" iyz="0.0" izz="0.00008"/>
+        <mass value="0.1"/>
+        <inertia ixx="0.0001" ixy="0.0" ixz="0.0" iyy="0.0001" iyz="0.0" izz="0.0001"/>
       </inertial>
       <visual>
@@ -82,58 +83,59 @@
         <origin xyz="0 0 0" rpy="0 0 0"/>
         <geometry>
-          <mesh filename="package://onrobot_description/meshes/3fg15/collision/right_finger.stl" scale="0.001 0.001 0.001"/>
+          <box size="0.01 0.02 0.06"/>
         </geometry>
       </collision>
     </link>
-    <joint name="${prefix}right_finger_fixed" type="fixed">
-      <parent link="${prefix}rotating_frame"/>
+    <!-- Dummy link for the main control joint (diameter control) -->
+    <link name="${prefix}finger_width_mock_link"/>
+    <!-- Main control joint (finger_width) - represents target diameter -->
+    <joint name="${prefix}finger_width" type="prismatic">
+      <origin xyz="0 0 0" rpy="0 0 0"/>
+      <parent link="${prefix}onrobot_base_link"/>
+      <child link="${prefix}finger_width_mock_link"/>
+      <axis xyz="0 0 1"/>
+      <limit lower="0" upper="0.15" velocity="0.3" effort="240"/>
+    </joint>
+    <!-- Finger Joints - Revolute joints for centripetal movement -->
+    <!-- Each finger rotates around the Z-axis at its mounting point -->
+    <!-- Left Finger (120 degrees) -->
+    <joint name="${prefix}left_finger_joint" type="revolute">
+      <origin xyz="0 0 0" rpy="0 0 0"/> <!-- 120 degrees -->
+      <parent link="${prefix}onrobot_base_link"/>
+      <child link="${prefix}left_finger_link"/>
+      <axis xyz="0 0 1"/>
+      <limit lower="-0.5236" upper="0.5236" effort="80" velocity="0.3"/> <!-- ±30 degrees -->
+      <!-- Mimic relationship: as diameter decreases, fingers rotate inward -->
+      <mimic joint="${prefix}finger_width" multiplier="-3.0" offset="0.5236"/>
+    </joint>
+    <!-- Middle Finger (0 degrees) -->
+    <joint name="${prefix}middle_finger_joint" type="revolute">
+      <origin xyz="0 0 0" rpy="0 0 0"/> <!-- 0 degrees -->
+      <parent link="${prefix}onrobot_base_link"/>
+      <child link="${prefix}middle_finger_link"/>
+      <axis xyz="0 0 1"/>
+      <limit lower="-0.5236" upper="0.5236" effort="80" velocity="0.3"/> <!-- ±30 degrees -->
+      <!-- Mimic relationship: as diameter decreases, fingers rotate inward -->
+      <mimic joint="${prefix}finger_width" multiplier="-3.0" offset="0.5236"/>
+    </joint>
+    <!-- Right Finger (240 degrees) -->
+    <joint name="${prefix}right_finger_joint" type="revolute">
+      <origin xyz="0 0 0" rpy="0 0 0"/> <!-- 240 degrees -->
+      <parent link="${prefix}onrobot_base_link"/>
       <child link="${prefix}right_finger_link"/>
-      <!-- 210° → X = -0.029375, Y = -0.050832, rz total = 300° = 5.23599 rad -->
-      <origin xyz="-0.029375 -0.050832 0" rpy="0 0 5.23599"/>
+      <axis xyz="0 0 1"/>
+      <limit lower="-0.5236" upper="0.5236" effort="80" velocity="0.3"/> <!-- ±30 degrees -->
+      <!-- Mimic relationship: as diameter decreases, fingers rotate inward -->
+      <mimic joint="${prefix}finger_width" multiplier="-3.0" offset="0.5236"/>
     </joint>
-    <!-- ====================== DEDO MEDIO ====================== -->
-    <link name="${prefix}middle_finger_link">
-      <inertial>
-        <origin xyz="0 0 0" rpy="0 0 0"/>
-        <mass value="0.08"/>
-        <inertia ixx="0.00008" ixy="0.0" ixz="0.0" iyy="0.00008" iyz="0.0" izz="0.00008"/>
-      </inertial>
-      <visual>
-        <origin xyz="0 0 0" rpy="0 0 0"/>
-        <geometry>
-          <mesh filename="package://onrobot_description/meshes/3fg15/visual/middle_finger.stl" scale="0.001 0.001 0.001"/>
-        </geometry>
-        <material name="onrobot_silver"/>
-      </visual>
-      <collision>
-        <origin xyz="0 0 0" rpy="0 0 0"/>
-        <geometry>
-          <mesh filename="package://onrobot_description/meshes/3fg15/collision/middle_finger.stl" scale="0.001 0.001 0.001"/>
-        </geometry>
-      </collision>
-    </link>
-    <joint name="${prefix}middle_finger_fixed" type="fixed">
-      <parent link="${prefix}rotating_frame"/>
-      <child link="${prefix}middle_finger_link"/>
-      <!-- 330° → X = -0.029375, Y = +0.050832, rz total = 60° = 1.0472 rad -->
-      <origin xyz="-0.029375 0.050832 0" rpy="0 0 1.0472"/>
-    </joint>
-    <!-- ====================== TCP ====================== -->
+    <!-- TCP Link -->
     <link name="${prefix}gripper_tcp"/>
     <joint name="${prefix}tcp_joint" type="fixed">
-      <parent link="${prefix}rotating_frame"/>
+      <origin xyz="0 0 0.08" rpy="0 0 0"/>
+      <parent link="${prefix}onrobot_base_link"/>
       <child link="${prefix}gripper_tcp"/>
-      <origin xyz="0 0 0.08" rpy="0 0 0"/>
     </joint>
-    <!-- ====================== TRANSMISIÓN (para ROS Control) ====================== -->
-    <transmission name="${prefix}gripper_rotation_trans">
-      <type>transmission_interface/SimpleTransmission</type>
-      <joint name="${prefix}gripper_rotation">
-        <hardwareInterface>hardware_interface/EffortJointInterface</hardwareInterface>
-      </joint>
-      <actuator name="${prefix}gripper_rotation_motor">
-        <mechanicalReduction>1</mechanicalReduction>
-      </actuator>
-    </transmission>
+    <!-- Transmission for ROS Control -->
+    <xacro:transmission_macro prefix="${prefix}" joint_name="finger_width"/>
   </xacro:macro>
 </robot>

File: urdf/onrobot.urdf.xacro (robot description, xacro)
@@ -11,4 +11,5 @@
     <xacro:arg name="ip_address" default="192.168.1.1"/>
     <xacro:arg name="port" default="502"/>
+    <xacro:arg name="device_address" default="65"/>
     <!-- Import the OnRobot macro -->
     <xacro:include filename="$(find onrobot_description)/urdf/onrobot_macro.xacro"/>
@@ -23,4 +24,5 @@
         ip_address="$(arg ip_address)"
         port="$(arg port)"
+        device_address="$(arg device_address)"
     />
     <!-- Create link fixed to the world -->

File: urdf/onrobot_macro.xacro (robot description, xacro)
@@ -38,14 +38,6 @@
       <gazebo>
         <plugin filename="libgazebo_ros2_control.so" name="gazebo_ros2_control">
-          <parameters>$(find onrobot_description)/config/onrobot_controllers.yaml</parameters>
         </plugin>
       </gazebo>
-      <!-- Include Gazebo-specific plugins for each gripper type -->
-      <xacro:if value="${onrobot_type == '3fg15'}">
-        <xacro:include filename="$(find onrobot_description)/urdf/inc/3fg15_gazebo.xacro"/>
-        <xacro:onrobot_3fg15_grasp_plugin prefix="${prefix}"/>
-        <xacro:onrobot_3fg15_mimic_plugin prefix="${prefix}"/>
-        <xacro:onrobot_3fg15_gazebo_properties prefix="${prefix}"/>
-      </xacro:if>
     </xacro:if>
     <!-- ====================== ROS2 Control ====================== -->
@@ -53,7 +45,7 @@
       <ros2_control name="OnRobotGripper" type="actuator">
         <hardware>
-          <!-- 2FG7, 2FG14 y 3FG15 usan el mismo driver -->
-          <xacro:if value="${onrobot_type == '2fg7' or onrobot_type == '2fg14' or onrobot_type == '3fg15'}">
-            <plugin>onrobot_driver::FGHardwareInterface</plugin>
+          <!-- 2FG7 / 2FG14 use TwoFG hardware interface -->
+          <xacro:if value="${onrobot_type == '2fg7' or onrobot_type == '2fg14'}">
+            <plugin>onrobot_driver::TwoFGHardwareInterface</plugin>
             <param name="onrobot_type">${onrobot_type}</param>
             <param name="prefix">${prefix}</param>
@@ -65,7 +57,19 @@
             <param name="use_fake_hardware">false</param>
           </xacro:if>
-          <!-- RG2 / RG6 -->
+          <!-- 3FG15 uses ThreeFG hardware interface -->
+          <xacro:if value="${onrobot_type == '3fg15'}">
+            <plugin>onrobot_driver::ThreeFGHardwareInterface</plugin>
+            <param name="onrobot_type">${onrobot_type}</param>
+            <param name="prefix">${prefix}</param>
+            <param name="connection_type">${connection_type}</param>
+            <param name="device">${device}</param>
+            <param name="ip_address">${ip_address}</param>
+            <param name="port">${port}</param>
+            <param name="device_address">${device_address}</param>
+            <param name="use_fake_hardware">false</param>
+          </xacro:if>
+          <!-- RG2 / RG6 use RG hardware interface -->
           <xacro:if value="${onrobot_type == 'rg2' or onrobot_type == 'rg6'}">
-            <plugin>onrobot_driver/RGHardwareInterface</plugin>
+            <plugin>onrobot_driver::RGHardwareInterface</plugin>
             <param name="onrobot_type">${onrobot_type}</param>
             <param name="prefix">${prefix}</param>

Commit message: 3fg15 gripper parts splitted

File: urdf/3fg15_macro.xacro (robot description, xacro)
@@ -3,55 +3,132 @@
   <xacro:include filename="$(find onrobot_description)/urdf/inc/common_utils.xacro" />
   <xacro:include filename="$(find onrobot_description)/urdf/inc/common_materials.xacro" />
-  <!-- ============================================= -->
-  <!-- Usa joint: finger_width → topic: /finger_width_controller/commands -->
-  <!-- ============================================= -->
+  <!-- Macro for OnRobot 3FG15 three-finger revolutionary gripper -->
   <xacro:macro name="onrobot_3fg15" params="prefix onrobot_type:='3fg15'">
-    <!-- ====================== Base Link (STL COMPLETO) ====================== -->
+    <!-- Constants for 3FG15 -->
+    <xacro:property name="max_aperture" value="0.1175" /> <!-- 117.5mm in meters -->
+    <xacro:property name="min_aperture" value="0.0088" /> <!-- 8.8mm in meters -->
+    <xacro:property name="finger_radius" value="0.05875" /> <!-- Radius from center to finger tip -->
+    <!-- Base Link -->
     <link name="${prefix}onrobot_base_link">
       <inertial>
-        <origin xyz="0 0 0.05" rpy="${-pi/2} 0 0"/>
-        <mass value="1.8"/>
-        <inertia ixx="0.015" ixy="0.0" ixz="0.0" iyy="0.015" iyz="0.0" izz="0.010"/>
+        <origin xyz="0 0 0" rpy="0 0 0"/>
+        <mass value="1.2"/>
+        <inertia ixx="0.012" ixy="0.0" ixz="0.0" iyy="0.012" iyz="0.0" izz="0.008"/>
       </inertial>
       <visual>
-        <origin xyz="0 0 0.05" rpy="${-pi/2} 0 0"/>
+        <origin xyz="0 0 0" rpy="0 0 0"/>
         <geometry>
-          <mesh filename="package://onrobot_description/meshes/3fg15/visual/3fg15.stl" scale="0.001 0.001 0.001"/>
+          <mesh filename="package://onrobot_description/meshes/3fg15/visual/base.stl" scale="0.001 0.001 0.001"/>
         </geometry>
         <material name="onrobot_silver"/>
       </visual>
       <collision>
-        <origin xyz="0 0 0.05" rpy="${-pi/2} 0 0"/>
+        <origin xyz="0 0 0" rpy="0 0 0"/>
         <geometry>
-          <mesh filename="package://onrobot_description/meshes/3fg15/collision/3fg15.stl" scale="0.001 0.001 0.001"/>
+          <mesh filename="package://onrobot_description/meshes/3fg15/collision/base.stl" scale="0.001 0.001 0.001"/>
         </geometry>
       </collision>
     </link>
-    <!-- ====================== Mock Link (invisible, solo para joint) ====================== -->
-    <link name="${prefix}finger_width_mock_link">
+    <!-- Left Finger Link -->
+    <link name="${prefix}left_finger_link">
       <inertial>
         <origin xyz="0 0 0" rpy="0 0 0"/>
-        <mass value="0.001"/>
-        <inertia ixx="1e-6" ixy="0.0" ixz="0.0" iyy="1e-6" iyz="0.0" izz="1e-6"/>
+        <mass value="0.08"/>
+        <inertia ixx="0.00008" ixy="0.0" ixz="0.0" iyy="0.00008" iyz="0.0" izz="0.00008"/>
       </inertial>
       <visual>
         <origin xyz="0 0 0" rpy="0 0 0"/>
-        <geometry><box size="0.001 0.001 0.001"/></geometry>
+        <geometry>
+          <mesh filename="package://onrobot_description/meshes/3fg15/visual/left_finger.stl" scale="0.001 0.001 0.001"/>
+        </geometry>
+        <material name="onrobot_silver"/>
       </visual>
       <collision>
         <origin xyz="0 0 0" rpy="0 0 0"/>
-        <geometry><box size="0.001 0.001 0.001"/></geometry>
+        <geometry>
+          <mesh filename="package://onrobot_description/meshes/3fg15/collision/left_finger.stl" scale="0.001 0.001 0.001"/>
+        </geometry>
       </collision>
     </link>
-    <!-- ====================== Main Control Joint: finger_width (0 a 150 mm) ====================== -->
+    <!-- Right Finger Link -->
+    <link name="${prefix}right_finger_link">
+      <inertial>
+        <origin xyz="0 0 0" rpy="0 0 0"/>
+        <mass value="0.08"/>
+        <inertia ixx="0.00008" ixy="0.0" ixz="0.0" iyy="0.00008" iyz="0.0" izz="0.00008"/>
+      </inertial>
+      <visual>
+        <origin xyz="0 0 0" rpy="0 0 0"/>
+        <geometry>
+          <mesh filename="package://onrobot_description/meshes/3fg15/visual/right_finger.stl" scale="0.001 0.001 0.001"/>
+        </geometry>
+        <material name="onrobot_silver"/>
+      </visual>
+      <collision>
+        <origin xyz="0 0 0" rpy="0 0 0"/>
+        <geometry>
+          <mesh filename="package://onrobot_description/meshes/3fg15/collision/right_finger.stl" scale="0.001 0.001 0.001"/>
+        </geometry>
+      </collision>
+    </link>
+    <!-- Middle Finger Link -->
+    <link name="${prefix}middle_finger_link">
+      <inertial>
+        <origin xyz="0 0 0" rpy="0 0 0"/>
+        <mass value="0.08"/>
+        <inertia ixx="0.00008" ixy="0.0" ixz="0.0" iyy="0.00008" iyz="0.0" izz="0.00008"/>
+      </inertial>
+      <visual>
+        <origin xyz="0 0 0" rpy="0 0 0"/>
+        <geometry>
+          <mesh filename="package://onrobot_description/meshes/3fg15/visual/middle_finger.stl" scale="0.001 0.001 0.001"/>
+        </geometry>
+        <material name="onrobot_silver"/>
+      </visual>
+      <collision>
+        <origin xyz="0 0 0" rpy="0 0 0"/>
+        <geometry>
+          <mesh filename="package://onrobot_description/meshes/3fg15/collision/middle_finger.stl" scale="0.001 0.001 0.001"/>
+        </geometry>
+      </collision>
+    </link>
+    <!-- Dummy link for the main control joint -->
+    <link name="${prefix}finger_width_mock_link"/>
+    <!-- Main control joint (finger_width) - represents aperture diameter -->
     <joint name="${prefix}finger_width" type="prismatic">
+      <origin xyz="0 0 0" rpy="0 0 0"/>
       <parent link="${prefix}onrobot_base_link"/>
       <child link="${prefix}finger_width_mock_link"/>
-      <origin xyz="0 0 0.05" rpy="0 0 0"/>
       <axis xyz="0 0 1"/>
-      <limit lower="0.0" upper="0.150" effort="240" velocity="0.3"/>
-      <!-- 150 mm = 0.15 m (diámetro externo del 3FG15) -->
+      <limit lower="${min_aperture}" upper="${max_aperture}" velocity="0.25" effort="200"/>
     </joint>
-    <!-- ====================== TCP Link (punto de agarre) ====================== -->
+    <!-- Left Finger Joint (Revolute) -->
+    <joint name="${prefix}left_finger_joint" type="revolute">
+      <origin xyz="0 0 0" rpy="0 0 0"/>
+      <parent link="${prefix}onrobot_base_link"/>
+      <child link="${prefix}left_finger_link"/>
+      <axis xyz="0 0 1"/>
+      <limit lower="${-pi/3}" upper="${pi/3}" effort="200" velocity="0.25"/>
+      <mimic joint="${prefix}finger_width" multiplier="${(2*pi/3)/(max_aperture - min_aperture)}" offset="${-pi/3 - (2*pi/3)/(max_aperture - min_aperture) * min_aperture}"/>
+    </joint>
+    <!-- Right Finger Joint (Revolute) -->
+    <joint name="${prefix}right_finger_joint" type="revolute">
+      <origin xyz="0 0 0" rpy="0 0 0"/>
+      <parent link="${prefix}onrobot_base_link"/>
+      <child link="${prefix}right_finger_link"/>
+      <axis xyz="0 0 1"/>
+      <limit lower="${-pi/3}" upper="${pi/3}" effort="200" velocity="0.25"/>
+      <mimic joint="${prefix}finger_width" multiplier="${(2*pi/3)/(max_aperture - min_aperture)}" offset="${-pi/3 - (2*pi/3)/(max_aperture - min_aperture) * min_aperture}"/>
+    </joint>
+    <!-- Middle Finger Joint (Revolute) -->
+    <joint name="${prefix}middle_finger_joint" type="revolute">
+      <origin xyz="0 0 0" rpy="0 0 0"/>
+      <parent link="${prefix}onrobot_base_link"/>
+      <child link="${prefix}middle_finger_link"/>
+      <axis xyz="0 0 1"/>
+      <limit lower="${-pi/3}" upper="${pi/3}" effort="200" velocity="0.25"/>
+      <mimic joint="${prefix}finger_width" multiplier="${(2*pi/3)/(max_aperture - min_aperture)}" offset="${-pi/3 - (2*pi/3)/(max_aperture - min_aperture) * min_aperture}"/>
+    </joint>
+    <!-- TCP Link -->
     <link name="${prefix}gripper_tcp"/>
     <joint name="${prefix}tcp_joint" type="fixed">
@@ -60,5 +137,5 @@
       <child link="${prefix}gripper_tcp"/>
     </joint>
-    <!-- ====================== Transmission (genera /finger_width_controller) ====================== -->
+    <!-- Transmission for ROS Control -->
     <xacro:transmission_macro prefix="${prefix}" joint_name="finger_width"/>
   </xacro:macro>
