Commit message: 3fg15 updated

File: urdf/3fg15_macro.xacro (robot description, xacro)
@@ -3,19 +3,14 @@
   <xacro:include filename="$(find onrobot_description)/urdf/inc/common_utils.xacro" />
   <xacro:include filename="$(find onrobot_description)/urdf/inc/common_materials.xacro" />
-  <!-- Macro for OnRobot 3FG15 three-finger revolutionary gripper -->
   <xacro:macro name="onrobot_3fg15" params="prefix onrobot_type:='3fg15'">
-    <!-- Constants for 3FG15 -->
-    <xacro:property name="max_aperture" value="0.1175" /> <!-- 117.5mm in meters -->
-    <xacro:property name="min_aperture" value="0.0088" /> <!-- 8.8mm in meters -->
-    <xacro:property name="finger_radius" value="0.05875" /> <!-- Radius from center to finger tip -->
-    <!-- Base Link -->
+    <!-- ====================== Base Link ====================== -->
     <link name="${prefix}onrobot_base_link">
       <inertial>
-        <origin xyz="0 0 0" rpy="0 0 0"/>
-        <mass value="1.2"/>
-        <inertia ixx="0.012" ixy="0.0" ixz="0.0" iyy="0.012" iyz="0.0" izz="0.008"/>
+        <origin xyz="0 0 0.03" rpy="${-pi/2} 0 0"/>
+        <mass value="1.3"/>
+        <inertia ixx="0.015" ixy="0.0" ixz="0.0" iyy="0.015" iyz="0.0" izz="0.010"/>
       </inertial>
       <visual>
-        <origin xyz="0 0 0" rpy="0 0 0"/>
+        <origin xyz="0 0 0" rpy="${-pi/2} 0 0"/>
         <geometry>
           <mesh filename="package://onrobot_description/meshes/3fg15/visual/base.stl" scale="0.001 0.001 0.001"/>
@@ -24,5 +19,5 @@
       </visual>
       <collision>
-        <origin xyz="0 0 0" rpy="0 0 0"/>
+        <origin xyz="0 0 0" rpy="${-pi/2} 0 0"/>
         <geometry>
           <mesh filename="package://onrobot_description/meshes/3fg15/collision/base.stl" scale="0.001 0.001 0.001"/>
@@ -30,13 +25,14 @@
       </collision>
     </link>
-    <!-- Left Finger Link -->
+    <!-- ====================== Dedos individuales ====================== -->
+    <!-- Dedo izquierdo (120° a la izquierda) -->
     <link name="${prefix}left_finger_link">
       <inertial>
-        <origin xyz="0 0 0" rpy="0 0 0"/>
+        <origin xyz="0.026 -0.015 0" rpy="${-pi/2} 0 0"/>
         <mass value="0.08"/>
-        <inertia ixx="0.00008" ixy="0.0" ixz="0.0" iyy="0.00008" iyz="0.0" izz="0.00008"/>
+        <inertia ixx="0.0001" ixy="0.0" ixz="0.0" iyy="0.0001" iyz="0.0" izz="0.0001"/>
       </inertial>
       <visual>
-        <origin xyz="0 0 0" rpy="0 0 0"/>
+        <origin xyz="0.026 -0.015 0" rpy="${-pi/2} 0 0"/>
         <geometry>
           <mesh filename="package://onrobot_description/meshes/3fg15/visual/left_finger.stl" scale="0.001 0.001 0.001"/>
@@ -45,5 +41,5 @@
       </visual>
       <collision>
-        <origin xyz="0 0 0" rpy="0 0 0"/>
+        <origin xyz=" 0.026 -0.015 0 " rpy="${-pi/2} 0 0"/>
         <geometry>
           <mesh filename="package://onrobot_description/meshes/3fg15/collision/left_finger.stl" scale="0.001 0.001 0.001"/>
@@ -51,13 +47,13 @@
       </collision>
     </link>
-    <!-- Right Finger Link -->
+    <!-- Dedo derecho (120° a la derecha) -->
     <link name="${prefix}right_finger_link">
       <inertial>
-        <origin xyz="0 0 0" rpy="0 0 0"/>
+        <origin xyz="-0.026 -0.015 -0.15" rpy="${-pi/2} 0 0"/>
         <mass value="0.08"/>
-        <inertia ixx="0.00008" ixy="0.0" ixz="0.0" iyy="0.00008" iyz="0.0" izz="0.00008"/>
+        <inertia ixx="0.0001" ixy="0.0" ixz="0.0" iyy="0.0001" iyz="0.0" izz="0.0001"/>
       </inertial>
       <visual>
-        <origin xyz="0 0 0" rpy="0 0 0"/>
+        <origin xyz="-0.0260 -0.0150 -0.1500" rpy="${-pi/2} 0 0"/>
         <geometry>
           <mesh filename="package://onrobot_description/meshes/3fg15/visual/right_finger.stl" scale="0.001 0.001 0.001"/>
@@ -66,5 +62,5 @@
       </visual>
       <collision>
-        <origin xyz="0 0 0" rpy="0 0 0"/>
+        <origin xyz="-0.026 -0.015 -0.15" rpy="${-pi/2} 0 0"/>
         <geometry>
           <mesh filename="package://onrobot_description/meshes/3fg15/collision/right_finger.stl" scale="0.001 0.001 0.001"/>
@@ -72,13 +68,13 @@
       </collision>
     </link>
-    <!-- Middle Finger Link -->
-    <link name="${prefix}middle_finger_link">
+    <!-- Dedo central (hacia abajo) -->
+    <link name="${prefix}center_finger_link">
       <inertial>
-        <origin xyz="0 0 0" rpy="0 0 0"/>
+        <origin xyz="0 +0.03 0 " rpy="${-pi/2} 0 0"/>
         <mass value="0.08"/>
-        <inertia ixx="0.00008" ixy="0.0" ixz="0.0" iyy="0.00008" iyz="0.0" izz="0.00008"/>
+        <inertia ixx="0.0001" ixy="0.0" ixz="0.0" iyy="0.0001" iyz="0.0" izz="0.0001"/>
       </inertial>
       <visual>
-        <origin xyz="0 0 0" rpy="0 0 0"/>
+        <origin xyz="0 +0.03 0" rpy="${-pi/2} 0 0"/>
         <geometry>
           <mesh filename="package://onrobot_description/meshes/3fg15/visual/middle_finger.stl" scale="0.001 0.001 0.001"/>
@@ -87,5 +83,5 @@
       </visual>
       <collision>
-        <origin xyz="0 0 0" rpy="0 0 0"/>
+        <origin xyz="0 +0.03 0" rpy="${-pi/2} 0 0"/>
         <geometry>
           <mesh filename="package://onrobot_description/meshes/3fg15/collision/middle_finger.stl" scale="0.001 0.001 0.001"/>
@@ -93,49 +89,104 @@
       </collision>
     </link>
-    <!-- Dummy link for the main control joint -->
-    <link name="${prefix}finger_width_mock_link"/>
-    <!-- Main control joint (finger_width) - represents aperture diameter -->
-    <joint name="${prefix}finger_width" type="prismatic">
-      <origin xyz="0 0 0" rpy="0 0 0"/>
+    <!-- ====================== Mock link para el joint principal ====================== -->
+    <link name="${prefix}finger_width_mock_link">
+      <inertial>
+        <mass value="0.001"/>
+        <inertia ixx="1e-6" ixy="0" ixz="0" iyy="1e-6" iyz="0" izz="1e-6"/>
+      </inertial>
+    </link>
+    <!-- ====================== Joint principal de control (0 a 150 mm) ====================== -->
+    <joint name="${prefix}finger_width" type="revolute">
       <parent link="${prefix}onrobot_base_link"/>
       <child link="${prefix}finger_width_mock_link"/>
+      <origin xyz="0 0 0.0" rpy="0 0 0"/>
       <axis xyz="0 0 1"/>
-      <limit lower="${min_aperture}" upper="${max_aperture}" velocity="0.25" effort="200"/>
+      <limit lower="0.0" upper="2.9" effort="140" velocity="0.45"/>
     </joint>
-    <!-- Left Finger Joint (Revolute) -->
+    <!-- ====================== Eje Z visual (debug) ====================== -->
+    <!--
+    <link name="${prefix}z_axis_visual_link2">
+      <visual>
+        <origin xyz="0 0 0" rpy="0 0 0"/>
+        <geometry>
+          <cylinder radius="0.001" length="0.18"/>
+        </geometry>
+        <material name="">
+          <color rgba="0 0 1 1"/>
+        </material>
+      </visual>
+    </link>
+    <joint name="${prefix}z_axis_visual_joint2" type="fixed">
+      <parent link="${prefix}onrobot_base_link"/>
+      <child  link="${prefix}z_axis_visual_link2"/>
+      <origin xyz="0 -0.02783 0.000" rpy="0 0 0"/>
+    </joint>
+    <link name="${prefix}z_axis_visual_link3">
+      <visual>
+        <origin xyz="0 0 0" rpy="0 0 0"/>
+        <geometry>W
+          <cylinder radius="0.001" length="0.18"/>
+        </geometry>
+        <material name="">
+          <color rgba="0 0 1 1"/>
+        </material>
+      </visual>
+    </link>
+    <joint name="${prefix}z_axis_visual_joint3" type="fixed">
+      <parent link="${prefix}onrobot_base_link"/>
+      <child  link="${prefix}z_axis_visual_link3"/>
+      <origin xyz="-0.02492 0.01299 0" rpy="0 0 0"/>
+    </joint>
+    <link name="${prefix}z_axis_visual_link4">
+      <visual>
+        <origin xyz="0 0 0" rpy="0 0 0"/>
+        <geometry>
+          <cylinder radius="0.001" length="0.18"/>
+        </geometry>
+        <material name="">
+          <color rgba="0 0 1 1"/>
+        </material>
+      </visual>
+    </link>
+    <joint name="${prefix}z_axis_visual_joint4" type="fixed">
+      <parent link="${prefix}onrobot_base_link"/>
+      <child  link="${prefix}z_axis_visual_link4"/>
+      <origin xyz=" 0.02492 0.01299  0" rpy="0 0 0"/>
+    </joint>
+    -->
+    <!-- ====================== Joints de los dedos (mimic del principal) ====================== -->
+    <!-- Los tres dedos se mueven radialmente según el ancho (finger_width / 3 por dedo) -->
     <joint name="${prefix}left_finger_joint" type="revolute">
-      <origin xyz="0 0 0" rpy="0 0 0"/>
+      <origin xyz="-0.026 0.015 0" rpy = "0 0 0"/>
       <parent link="${prefix}onrobot_base_link"/>
       <child link="${prefix}left_finger_link"/>
       <axis xyz="0 0 1"/>
-      <limit lower="${-pi/3}" upper="${pi/3}" effort="200" velocity="0.25"/>
-      <mimic joint="${prefix}finger_width" multiplier="${(2*pi/3)/(max_aperture - min_aperture)}" offset="${-pi/3 - (2*pi/3)/(max_aperture - min_aperture) * min_aperture}"/>
+      <limit lower="0.0" upper="3.14" effort="140" velocity="0.45"/>
+      <mimic joint="${prefix}finger_width" offset="0"/>
     </joint>
-    <!-- Right Finger Joint (Revolute) -->
     <joint name="${prefix}right_finger_joint" type="revolute">
-      <origin xyz="0 0 0" rpy="0 0 0"/>
+      <origin xyz="0.026 0.015 0.15" rpy="0 0 0"/>
       <parent link="${prefix}onrobot_base_link"/>
       <child link="${prefix}right_finger_link"/>
       <axis xyz="0 0 1"/>
-      <limit lower="${-pi/3}" upper="${pi/3}" effort="200" velocity="0.25"/>
-      <mimic joint="${prefix}finger_width" multiplier="${(2*pi/3)/(max_aperture - min_aperture)}" offset="${-pi/3 - (2*pi/3)/(max_aperture - min_aperture) * min_aperture}"/>
+      <limit lower="0.0" upper="3.14" effort="140" velocity="0.45"/>
+      <mimic joint="${prefix}finger_width"  offset="0"/>
     </joint>
-    <!-- Middle Finger Joint (Revolute) -->
-    <joint name="${prefix}middle_finger_joint" type="revolute">
-      <origin xyz="0 0 0" rpy="0 0 0"/>
+    <joint name="${prefix}center_finger_joint" type="revolute">
+      <origin xyz="0 -0.03 0" rpy="0 0 0"/>
       <parent link="${prefix}onrobot_base_link"/>
-      <child link="${prefix}middle_finger_link"/>
+      <child link="${prefix}center_finger_link"/>
       <axis xyz="0 0 1"/>
-      <limit lower="${-pi/3}" upper="${pi/3}" effort="200" velocity="0.25"/>
-      <mimic joint="${prefix}finger_width" multiplier="${(2*pi/3)/(max_aperture - min_aperture)}" offset="${-pi/3 - (2*pi/3)/(max_aperture - min_aperture) * min_aperture}"/>
+      <limit lower="0.0" upper="3.14" effort="140" velocity="0.45"/>
+      <mimic joint="${prefix}finger_width"  offset="0"/>
     </joint>
-    <!-- TCP Link -->
+    <!-- ====================== TCP (punto de agarre) ====================== -->
     <link name="${prefix}gripper_tcp"/>
     <joint name="${prefix}tcp_joint" type="fixed">
-      <origin xyz="0 0 0.08" rpy="0 0 0"/>
+      <origin xyz="0 0 0" rpy="0 0 0"/>
       <parent link="${prefix}onrobot_base_link"/>
       <child link="${prefix}gripper_tcp"/>
     </joint>
-    <!-- Transmission for ROS Control -->
+    <!-- ====================== Transmission para ROS Control ====================== -->
     <xacro:transmission_macro prefix="${prefix}" joint_name="finger_width"/>
   </xacro:macro>

Commit message: 3fg15 updated - fix

File: urdf/3fg15_macro.xacro (robot description, xacro)
@@ -7,10 +7,10 @@
     <link name="${prefix}onrobot_base_link">
       <inertial>
-        <origin xyz="0 0 0.03" rpy="${-pi/2} 0 0"/>
+        <origin xyz="0 0 0.045" rpy="${-pi/2} 0 0"/>
         <mass value="1.3"/>
         <inertia ixx="0.015" ixy="0.0" ixz="0.0" iyy="0.015" iyz="0.0" izz="0.010"/>
       </inertial>
       <visual>
-        <origin xyz="0 0 0" rpy="${-pi/2} 0 0"/>
+        <origin xyz="0 0 0.045" rpy="${-pi/2} 0 0"/>
         <geometry>
           <mesh filename="package://onrobot_description/meshes/3fg15/visual/base.stl" scale="0.001 0.001 0.001"/>
@@ -19,5 +19,5 @@
       </visual>
       <collision>
-        <origin xyz="0 0 0" rpy="${-pi/2} 0 0"/>
+        <origin xyz="0 0 0.045" rpy="${-pi/2} 0 0"/>
         <geometry>
           <mesh filename="package://onrobot_description/meshes/3fg15/collision/base.stl" scale="0.001 0.001 0.001"/>
@@ -29,10 +29,10 @@
     <link name="${prefix}left_finger_link">
       <inertial>
-        <origin xyz="0.026 -0.015 0" rpy="${-pi/2} 0 0"/>
+        <origin xyz="0.026 -0.015 0.045" rpy="${-pi/2} 0 0"/>
         <mass value="0.08"/>
         <inertia ixx="0.0001" ixy="0.0" ixz="0.0" iyy="0.0001" iyz="0.0" izz="0.0001"/>
       </inertial>
       <visual>
-        <origin xyz="0.026 -0.015 0" rpy="${-pi/2} 0 0"/>
+        <origin xyz="0.026 -0.015 0.045" rpy="${-pi/2} 0 0"/>
         <geometry>
           <mesh filename="package://onrobot_description/meshes/3fg15/visual/left_finger.stl" scale="0.001 0.001 0.001"/>
@@ -41,5 +41,5 @@
       </visual>
       <collision>
-        <origin xyz=" 0.026 -0.015 0 " rpy="${-pi/2} 0 0"/>
+        <origin xyz=" 0.026 -0.015 0.045" rpy="${-pi/2} 0 0"/>
         <geometry>
           <mesh filename="package://onrobot_description/meshes/3fg15/collision/left_finger.stl" scale="0.001 0.001 0.001"/>
@@ -50,10 +50,10 @@
     <link name="${prefix}right_finger_link">
       <inertial>
-        <origin xyz="-0.026 -0.015 -0.15" rpy="${-pi/2} 0 0"/>
+        <origin xyz="-0.026 -0.015 -0.105" rpy="${-pi/2} 0 0"/>
         <mass value="0.08"/>
         <inertia ixx="0.0001" ixy="0.0" ixz="0.0" iyy="0.0001" iyz="0.0" izz="0.0001"/>
       </inertial>
       <visual>
-        <origin xyz="-0.0260 -0.0150 -0.1500" rpy="${-pi/2} 0 0"/>
+        <origin xyz="-0.0260 -0.0150 -0.105" rpy="${-pi/2} 0 0"/>
         <geometry>
           <mesh filename="package://onrobot_description/meshes/3fg15/visual/right_finger.stl" scale="0.001 0.001 0.001"/>
@@ -62,5 +62,5 @@
       </visual>
       <collision>
-        <origin xyz="-0.026 -0.015 -0.15" rpy="${-pi/2} 0 0"/>
+        <origin xyz="-0.026 -0.015 -0.105" rpy="${-pi/2} 0 0"/>
         <geometry>
           <mesh filename="package://onrobot_description/meshes/3fg15/collision/right_finger.stl" scale="0.001 0.001 0.001"/>
@@ -71,10 +71,10 @@
     <link name="${prefix}center_finger_link">
       <inertial>
-        <origin xyz="0 +0.03 0 " rpy="${-pi/2} 0 0"/>
+        <origin xyz="0 0.03 0.045" rpy="${-pi/2} 0 0"/>
         <mass value="0.08"/>
         <inertia ixx="0.0001" ixy="0.0" ixz="0.0" iyy="0.0001" iyz="0.0" izz="0.0001"/>
       </inertial>
       <visual>
-        <origin xyz="0 +0.03 0" rpy="${-pi/2} 0 0"/>
+        <origin xyz="0 0.03 0.045" rpy="${-pi/2} 0 0"/>
         <geometry>
           <mesh filename="package://onrobot_description/meshes/3fg15/visual/middle_finger.stl" scale="0.001 0.001 0.001"/>
@@ -83,5 +83,5 @@
       </visual>
       <collision>
-        <origin xyz="0 +0.03 0" rpy="${-pi/2} 0 0"/>
+        <origin xyz="0 0.03 0.045" rpy="${-pi/2} 0 0"/>
         <geometry>
           <mesh filename="package://onrobot_description/meshes/3fg15/collision/middle_finger.stl" scale="0.001 0.001 0.001"/>
@@ -100,5 +100,5 @@
       <parent link="${prefix}onrobot_base_link"/>
       <child link="${prefix}finger_width_mock_link"/>
-      <origin xyz="0 0 0.0" rpy="0 0 0"/>
+      <origin xyz="0 0 0" rpy="0 0 0"/>
       <axis xyz="0 0 1"/>
       <limit lower="0.0" upper="2.9" effort="140" velocity="0.45"/>
@@ -184,5 +184,5 @@
     <link name="${prefix}gripper_tcp"/>
     <joint name="${prefix}tcp_joint" type="fixed">
-      <origin xyz="0 0 0" rpy="0 0 0"/>
+      <origin xyz="0 0 0.05" rpy="0 0 0"/>
       <parent link="${prefix}onrobot_base_link"/>
       <child link="${prefix}gripper_tcp"/>
