Commit message: OnRobot 2FG7 addition - Inclusion package 2

File: urdf/2fg7_macro.xacro (robot description, xacro)
@@ -4,15 +4,15 @@
   <xacro:include filename="$(find onrobot_description)/urdf/inc/2fg7_materials.xacro" />
   <xacro:macro name="onrobot_2fg7" params="prefix onrobot_type:='2fg7'">
-    <!-- Base Link -->
+    <!-- Base Link - CORRECTED SCALING -->
     <link name="${prefix}onrobot_base_link">
       <inertial>
         <origin xyz="0 0 0" rpy="0 0 0"/>
-        <mass value="0.5"/>
-        <inertia ixx="0.001" ixy="0.0" ixz="0.0" iyy="0.001" iyz="0.0" izz="0.001"/>
+        <mass value="0.3"/>
+        <inertia ixx="0.0005" ixy="0.0" ixz="0.0" iyy="0.0005" iyz="0.0" izz="0.0005"/>
       </inertial>
       <visual>
         <origin xyz="0 0 0" rpy="0 0 0"/>
         <geometry>
-          <mesh filename="package://onrobot_description/meshes/2fg7/visual/base_link.stl"/>
+          <mesh filename="package://onrobot_description/meshes/2fg7/visual/base_link.stl" scale="0.001 0.001 0.001"/>
         </geometry>
         <material name="silver"/>
@@ -21,19 +21,19 @@
         <origin xyz="0 0 0" rpy="0 0 0"/>
         <geometry>
-          <box size="0.08 0.08 0.06"/>
+          <box size="0.045 0.045 0.04"/>
         </geometry>
       </collision>
     </link>
-    <!-- Finger Links (simplified for 2FG7) -->
+    <!-- Finger Links - CORRECTED SCALING -->
     <link name="${prefix}left_finger_link">
       <inertial>
         <origin xyz="0 0 0" rpy="0 0 0"/>
-        <mass value="0.1"/>
-        <inertia ixx="0.0001" ixy="0.0" ixz="0.0" iyy="0.0001" iyz="0.0" izz="0.0001"/>
+        <mass value="0.05"/>
+        <inertia ixx="0.00005" ixy="0.0" ixz="0.0" iyy="0.00005" iyz="0.0" izz="0.00005"/>
       </inertial>
       <visual>
         <origin xyz="0 0 0" rpy="0 0 0"/>
         <geometry>
-          <mesh filename="package://onrobot_description/meshes/2fg7/visual/left_finger_link.stl"/>
+          <mesh filename="package://onrobot_description/meshes/2fg7/visual/left_finger_link.stl" scale="0.001 0.001 0.001"/>
         </geometry>
         <material name="silver"/>
@@ -42,5 +42,5 @@
         <origin xyz="0 0 0" rpy="0 0 0"/>
         <geometry>
-          <box size="0.02 0.03 0.08"/>
+          <box size="0.008 0.025 0.06"/>
         </geometry>
       </collision>
@@ -49,11 +49,11 @@
       <inertial>
         <origin xyz="0 0 0" rpy="0 0 0"/>
-        <mass value="0.1"/>
-        <inertia ixx="0.0001" ixy="0.0" ixz="0.0" iyy="0.0001" iyz="0.0" izz="0.0001"/>
+        <mass value="0.05"/>
+        <inertia ixx="0.00005" ixy="0.0" ixz="0.0" iyy="0.00005" iyz="0.0" izz="0.00005"/>
       </inertial>
       <visual>
         <origin xyz="0 0 0" rpy="0 0 0"/>
         <geometry>
-          <mesh filename="package://onrobot_description/meshes/2fg7/visual/right_finger_link.stl"/>
+          <mesh filename="package://onrobot_description/meshes/2fg7/visual/right_finger_link.stl" scale="0.001 0.001 0.001"/>
         </geometry>
         <material name="silver"/>
@@ -62,5 +62,5 @@
         <origin xyz="0 0 0" rpy="0 0 0"/>
         <geometry>
-          <box size="0.02 0.03 0.08"/>
+          <box size="0.008 0.025 0.06"/>
         </geometry>
       </collision>
@@ -78,5 +78,5 @@
     <!-- Left Finger Joint -->
     <joint name="${prefix}left_finger_joint" type="prismatic">
-      <origin xyz="0.02 0 0.04" rpy="0 0 0"/>
+      <origin xyz="0.0225 0 0.05" rpy="0 0 0"/>
       <parent link="${prefix}onrobot_base_link"/>
       <child link="${prefix}left_finger_link"/>
@@ -87,5 +87,5 @@
     <!-- Right Finger Joint -->
     <joint name="${prefix}right_finger_joint" type="prismatic">
-      <origin xyz="-0.02 0 0.04" rpy="0 0 0"/>
+      <origin xyz="-0.0225 0 0.05" rpy="0 0 0"/>
       <parent link="${prefix}onrobot_base_link"/>
       <child link="${prefix}right_finger_link"/>
@@ -97,5 +97,5 @@
     <link name="${prefix}gripper_tcp"/>
     <joint name="${prefix}tcp_joint" type="fixed">
-      <origin xyz="0 0 0.12" rpy="0 0 0"/>
+      <origin xyz="0 0 0.08" rpy="0 0 0"/>
       <parent link="${prefix}onrobot_base_link"/>
       <child link="${prefix}gripper_tcp"/>

Commit message: OnRobot 2FG7 addition - Inclusion package 2.1

File: urdf/2fg7_macro.xacro (robot description, xacro)
@@ -4,5 +4,5 @@
   <xacro:include filename="$(find onrobot_description)/urdf/inc/2fg7_materials.xacro" />
   <xacro:macro name="onrobot_2fg7" params="prefix onrobot_type:='2fg7'">
-    <!-- Base Link - CORRECTED SCALING -->
+    <!-- Base Link -->
     <link name="${prefix}onrobot_base_link">
       <inertial>
@@ -25,5 +25,5 @@
       </collision>
     </link>
-    <!-- Finger Links - CORRECTED SCALING -->
+    <!-- Finger Links -->
     <link name="${prefix}left_finger_link">
       <inertial>
@@ -76,7 +76,7 @@
       <limit lower="0" upper="0.07" velocity="0.45" effort="140"/>
     </joint>
-    <!-- Left Finger Joint -->
+    <!-- Left Finger Joint - FIXED ORIGIN -->
     <joint name="${prefix}left_finger_joint" type="prismatic">
-      <origin xyz="0.0225 0 0.05" rpy="0 0 0"/>
+      <origin xyz="0.0225 0 0.02" rpy="0 0 0"/>
       <parent link="${prefix}onrobot_base_link"/>
       <child link="${prefix}left_finger_link"/>
@@ -85,7 +85,7 @@
       <mimic joint="${prefix}finger_width" multiplier="0.5" offset="0"/>
     </joint>
-    <!-- Right Finger Joint -->
+    <!-- Right Finger Joint - FIXED ORIGIN -->
     <joint name="${prefix}right_finger_joint" type="prismatic">
-      <origin xyz="-0.0225 0 0.05" rpy="0 0 0"/>
+      <origin xyz="-0.0225 0 0.02" rpy="0 0 0"/>
       <parent link="${prefix}onrobot_base_link"/>
       <child link="${prefix}right_finger_link"/>
@@ -97,5 +97,5 @@
     <link name="${prefix}gripper_tcp"/>
     <joint name="${prefix}tcp_joint" type="fixed">
-      <origin xyz="0 0 0.08" rpy="0 0 0"/>
+      <origin xyz="0 0 0.06" rpy="0 0 0"/>
       <parent link="${prefix}onrobot_base_link"/>
       <child link="${prefix}gripper_tcp"/>

Commit message: OnRobot 2FG7 addition - Inclusion package 2.2

File: urdf/2fg7_macro.xacro (robot description, xacro)
@@ -28,10 +28,10 @@
     <link name="${prefix}left_finger_link">
       <inertial>
-        <origin xyz="0 0 0" rpy="0 0 0"/>
+        <origin xyz="0 0 0.03" rpy="0 0 0"/>
         <mass value="0.05"/>
         <inertia ixx="0.00005" ixy="0.0" ixz="0.0" iyy="0.00005" iyz="0.0" izz="0.00005"/>
       </inertial>
       <visual>
-        <origin xyz="0 0 0" rpy="0 0 0"/>
+        <origin xyz="0 0 0.03" rpy="0 0 0"/>
         <geometry>
           <mesh filename="package://onrobot_description/meshes/2fg7/visual/left_finger_link.stl" scale="0.001 0.001 0.001"/>
@@ -40,5 +40,5 @@
       </visual>
       <collision>
-        <origin xyz="0 0 0" rpy="0 0 0"/>
+        <origin xyz="0 0 0.03" rpy="0 0 0"/>
         <geometry>
           <box size="0.008 0.025 0.06"/>
@@ -48,10 +48,10 @@
     <link name="${prefix}right_finger_link">
       <inertial>
-        <origin xyz="0 0 0" rpy="0 0 0"/>
+        <origin xyz="0 0 0.03" rpy="0 0 0"/>
         <mass value="0.05"/>
         <inertia ixx="0.00005" ixy="0.0" ixz="0.0" iyy="0.00005" iyz="0.0" izz="0.00005"/>
       </inertial>
       <visual>
-        <origin xyz="0 0 0" rpy="0 0 0"/>
+        <origin xyz="0 0 0.03" rpy="0 0 0"/>
         <geometry>
           <mesh filename="package://onrobot_description/meshes/2fg7/visual/right_finger_link.stl" scale="0.001 0.001 0.001"/>
@@ -60,5 +60,5 @@
       </visual>
       <collision>
-        <origin xyz="0 0 0" rpy="0 0 0"/>
+        <origin xyz="0 0 0.03" rpy="0 0 0"/>
         <geometry>
           <box size="0.008 0.025 0.06"/>
@@ -68,5 +68,5 @@
     <!-- Dummy link for the main control joint -->
     <link name="${prefix}finger_width_mock_link"/>
-    <!-- Main control joint (finger_width) -->
+    <!-- Main control joint (finger_width) - CORRECT RANGE: 0 to 0.07m (70mm) -->
     <joint name="${prefix}finger_width" type="prismatic">
       <origin xyz="0 0 0" rpy="0 0 0"/>
@@ -76,7 +76,7 @@
       <limit lower="0" upper="0.07" velocity="0.45" effort="140"/>
     </joint>
-    <!-- Left Finger Joint - FIXED ORIGIN -->
+    <!-- Left Finger Joint - FIXED: Proper origin and mimic -->
     <joint name="${prefix}left_finger_joint" type="prismatic">
-      <origin xyz="0.0225 0 0.02" rpy="0 0 0"/>
+      <origin xyz="0.0225 0 0.03" rpy="0 0 0"/>
       <parent link="${prefix}onrobot_base_link"/>
       <child link="${prefix}left_finger_link"/>
@@ -85,7 +85,7 @@
       <mimic joint="${prefix}finger_width" multiplier="0.5" offset="0"/>
     </joint>
-    <!-- Right Finger Joint - FIXED ORIGIN -->
+    <!-- Right Finger Joint - FIXED: Proper origin and mimic -->
     <joint name="${prefix}right_finger_joint" type="prismatic">
-      <origin xyz="-0.0225 0 0.02" rpy="0 0 0"/>
+      <origin xyz="-0.0225 0 0.03" rpy="0 0 0"/>
       <parent link="${prefix}onrobot_base_link"/>
       <child link="${prefix}right_finger_link"/>
@@ -97,5 +97,5 @@
     <link name="${prefix}gripper_tcp"/>
     <joint name="${prefix}tcp_joint" type="fixed">
-      <origin xyz="0 0 0.06" rpy="0 0 0"/>
+      <origin xyz="0 0 0.08" rpy="0 0 0"/>
       <parent link="${prefix}onrobot_base_link"/>
       <child link="${prefix}gripper_tcp"/>

Commit message: OnRobot 2FG7 addition - Inclusion package 2.2.1

File: urdf/2fg7_macro.xacro (robot description, xacro)
@@ -28,10 +28,10 @@
     <link name="${prefix}left_finger_link">
       <inertial>
-        <origin xyz="0 0 0.03" rpy="0 0 0"/>
+        <origin xyz="0 0 0" rpy="0 0 0"/>
         <mass value="0.05"/>
         <inertia ixx="0.00005" ixy="0.0" ixz="0.0" iyy="0.00005" iyz="0.0" izz="0.00005"/>
       </inertial>
       <visual>
-        <origin xyz="0 0 0.03" rpy="0 0 0"/>
+        <origin xyz="0 0 0" rpy="0 0 0"/>
         <geometry>
           <mesh filename="package://onrobot_description/meshes/2fg7/visual/left_finger_link.stl" scale="0.001 0.001 0.001"/>
@@ -40,5 +40,5 @@
       </visual>
       <collision>
-        <origin xyz="0 0 0.03" rpy="0 0 0"/>
+        <origin xyz="0 0 0" rpy="0 0 0"/>
         <geometry>
           <box size="0.008 0.025 0.06"/>
@@ -48,10 +48,10 @@
     <link name="${prefix}right_finger_link">
       <inertial>
-        <origin xyz="0 0 0.03" rpy="0 0 0"/>
+        <origin xyz="0 0 0" rpy="0 0 0"/>
         <mass value="0.05"/>
         <inertia ixx="0.00005" ixy="0.0" ixz="0.0" iyy="0.00005" iyz="0.0" izz="0.00005"/>
       </inertial>
       <visual>
-        <origin xyz="0 0 0.03" rpy="0 0 0"/>
+        <origin xyz="0 0 0" rpy="0 0 0"/>
         <geometry>
           <mesh filename="package://onrobot_description/meshes/2fg7/visual/right_finger_link.stl" scale="0.001 0.001 0.001"/>
@@ -60,5 +60,5 @@
       </visual>
       <collision>
-        <origin xyz="0 0 0.03" rpy="0 0 0"/>
+        <origin xyz="0 0 0" rpy="0 0 0"/>
         <geometry>
           <box size="0.008 0.025 0.06"/>
@@ -74,22 +74,22 @@
       <child link="${prefix}finger_width_mock_link"/>
       <axis xyz="0 0 1"/>
-      <limit lower="0" upper="0.07" velocity="0.45" effort="140"/>
+      <limit lower="0" upper="0.035" velocity="0.45" effort="140"/>
     </joint>
     <!-- Left Finger Joint - FIXED: Proper origin and mimic -->
     <joint name="${prefix}left_finger_joint" type="prismatic">
-      <origin xyz="0.0225 0 0.03" rpy="0 0 0"/>
+      <origin xyz="0 0 0" rpy="0 0 0"/>
       <parent link="${prefix}onrobot_base_link"/>
       <child link="${prefix}left_finger_link"/>
       <axis xyz="1 0 0"/>
-      <limit lower="0.0" upper="0.035" effort="140" velocity="0.45"/>
+      <limit lower="0.0" upper="0.0175" effort="140" velocity="0.45"/>
       <mimic joint="${prefix}finger_width" multiplier="0.5" offset="0"/>
     </joint>
     <!-- Right Finger Joint - FIXED: Proper origin and mimic -->
     <joint name="${prefix}right_finger_joint" type="prismatic">
-      <origin xyz="-0.0225 0 0.03" rpy="0 0 0"/>
+      <origin xyz="0 0 0" rpy="0 0 0"/>
       <parent link="${prefix}onrobot_base_link"/>
       <child link="${prefix}right_finger_link"/>
       <axis xyz="-1 0 0"/>
-      <limit lower="-0.035" upper="0.0" effort="140" velocity="0.45"/>
+      <limit lower="-0.0175" upper="0.0" effort="140" velocity="0.45"/>
       <mimic joint="${prefix}finger_width" multiplier="0.5" offset="0"/>
     </joint>

Commit message: OnRobot 2FG7 addition - Inclusion package 2.2.2

File: urdf/2fg7_macro.xacro (robot description, xacro)
@@ -76,7 +76,7 @@
       <limit lower="0" upper="0.035" velocity="0.45" effort="140"/>
     </joint>
-    <!-- Left Finger Joint - FIXED: Proper origin and mimic -->
+    <!-- Left Finger Joint - MODIFIED: Positioned to start close to center -->
     <joint name="${prefix}left_finger_joint" type="prismatic">
-      <origin xyz="0 0 0" rpy="0 0 0"/>
+      <origin xyz="-0.0175 0 0" rpy="0 0 0"/>
       <parent link="${prefix}onrobot_base_link"/>
       <child link="${prefix}left_finger_link"/>
@@ -85,7 +85,7 @@
       <mimic joint="${prefix}finger_width" multiplier="0.5" offset="0"/>
     </joint>
-    <!-- Right Finger Joint - FIXED: Proper origin and mimic -->
+    <!-- Right Finger Joint - MODIFIED: Positioned to start close to center -->
     <joint name="${prefix}right_finger_joint" type="prismatic">
-      <origin xyz="0 0 0" rpy="0 0 0"/>
+      <origin xyz="0.0175 0 0" rpy="0 0 0"/>
       <parent link="${prefix}onrobot_base_link"/>
       <child link="${prefix}right_finger_link"/>

Commit message: OnRobot 2FG7 addition - Inclusion package 2.2.2

File: urdf/2fg7_macro.xacro (robot description, xacro)
@@ -78,5 +78,5 @@
     <!-- Left Finger Joint - MODIFIED: Positioned to start close to center -->
     <joint name="${prefix}left_finger_joint" type="prismatic">
-      <origin xyz="-0.0175 0 0" rpy="0 0 0"/>
+      <origin xyz="-0.0225 0 0" rpy="0 0 0"/>
       <parent link="${prefix}onrobot_base_link"/>
       <child link="${prefix}left_finger_link"/>
@@ -87,5 +87,5 @@
     <!-- Right Finger Joint - MODIFIED: Positioned to start close to center -->
     <joint name="${prefix}right_finger_joint" type="prismatic">
-      <origin xyz="0.0175 0 0" rpy="0 0 0"/>
+      <origin xyz="0.0225 0 0" rpy="0 0 0"/>
       <parent link="${prefix}onrobot_base_link"/>
       <child link="${prefix}right_finger_link"/>

Commit message: OnRobot 2FG7 addition - Inclusion package 2.2.2 - Materials Fix

File: urdf/2fg7_macro.xacro (robot description, xacro)
@@ -16,5 +16,5 @@
           <mesh filename="package://onrobot_description/meshes/2fg7/visual/base_link.stl" scale="0.001 0.001 0.001"/>
         </geometry>
-        <material name="silver"/>
+        <material name="onrobot_silver"/>
       </visual>
       <collision>
@@ -37,5 +37,5 @@
           <mesh filename="package://onrobot_description/meshes/2fg7/visual/left_finger_link.stl" scale="0.001 0.001 0.001"/>
         </geometry>
-        <material name="silver"/>
+        <material name="onrobot_silver"/>
       </visual>
       <collision>
@@ -57,5 +57,5 @@
           <mesh filename="package://onrobot_description/meshes/2fg7/visual/right_finger_link.stl" scale="0.001 0.001 0.001"/>
         </geometry>
-        <material name="silver"/>
+        <material name="onrobot_silver"/>
       </visual>
       <collision>

File: urdf/inc/2fg7_materials.xacro (robot description, xacro)
@@ -1,6 +1,13 @@
 <?xml version="1.0"?>
 <robot xmlns:xacro="http://www.ros.org/wiki/xacro">
-  <material name="silver">
+  <!-- Use unique names for gripper materials to avoid conflicts -->
+  <material name="onrobot_silver">
     <color rgba="0.700 0.700 0.700 1.000"/>
   </material>
+  <material name="onrobot_gripper_gray">
+    <color rgba="0.700 0.700 0.700 1.000"/>
+  </material>
+  <material name="onrobot_aluminum">
+    <color rgba="0.800 0.800 0.800 1.000"/>
+  </material>
 </robot>

Commit message: OnRobot 2FG7 addition - Inclusion package 2.3 - Materials Fix

File: urdf/2fg7_macro.xacro (robot description, xacro)
@@ -68,5 +68,5 @@
     <!-- Dummy link for the main control joint -->
     <link name="${prefix}finger_width_mock_link"/>
-    <!-- Main control joint (finger_width) - CORRECT RANGE: 0 to 0.07m (70mm) -->
+    <!-- Main control joint (finger_width) -->
     <joint name="${prefix}finger_width" type="prismatic">
       <origin xyz="0 0 0" rpy="0 0 0"/>
@@ -76,5 +76,5 @@
       <limit lower="0" upper="0.035" velocity="0.45" effort="140"/>
     </joint>
-    <!-- Left Finger Joint - MODIFIED: Positioned to start close to center -->
+    <!-- Left Finger Joint -->
     <joint name="${prefix}left_finger_joint" type="prismatic">
       <origin xyz="-0.0225 0 0" rpy="0 0 0"/>
@@ -85,5 +85,5 @@
       <mimic joint="${prefix}finger_width" multiplier="0.5" offset="0"/>
     </joint>
-    <!-- Right Finger Joint - MODIFIED: Positioned to start close to center -->
+    <!-- Right Finger Joint -->
     <joint name="${prefix}right_finger_joint" type="prismatic">
       <origin xyz="0.0225 0 0" rpy="0 0 0"/>

File: urdf/inc/2fg7_materials.xacro (robot description, xacro)
@@ -8,6 +8,3 @@
     <color rgba="0.700 0.700 0.700 1.000"/>
   </material>
-  <material name="onrobot_aluminum">
-    <color rgba="0.800 0.800 0.800 1.000"/>
-  </material>
 </robot>

Commit message: OnRobot 2FG7 addition - Inclusion package 3

File: urdf/2fg7_macro.xacro (robot description, xacro)
@@ -78,5 +78,5 @@
     <!-- Left Finger Joint -->
     <joint name="${prefix}left_finger_joint" type="prismatic">
-      <origin xyz="-0.0225 0 0" rpy="0 0 0"/>
+      <origin xyz="-0.0175 0 0" rpy="0 0 0"/>
       <parent link="${prefix}onrobot_base_link"/>
       <child link="${prefix}left_finger_link"/>
@@ -87,5 +87,5 @@
     <!-- Right Finger Joint -->
     <joint name="${prefix}right_finger_joint" type="prismatic">
-      <origin xyz="0.0225 0 0" rpy="0 0 0"/>
+      <origin xyz="0.0175 0 0" rpy="0 0 0"/>
       <parent link="${prefix}onrobot_base_link"/>
       <child link="${prefix}right_finger_link"/>

Commit message: joint limits fix

File: urdf/2fg7_macro.xacro (robot description, xacro)
@@ -74,9 +74,9 @@
       <child link="${prefix}finger_width_mock_link"/>
       <axis xyz="0 0 1"/>
-      <limit lower="0" upper="0.035" velocity="0.45" effort="140"/>
+      <limit lower="0.035" upper="0.07" velocity="0.45" effort="140"/>
     </joint>
     <!-- Left Finger Joint -->
     <joint name="${prefix}left_finger_joint" type="prismatic">
-      <origin xyz="-0.0175 0 0" rpy="0 0 0"/>
+      <origin xyz="-0.035 0 0" rpy="0 0 0"/>
       <parent link="${prefix}onrobot_base_link"/>
       <child link="${prefix}left_finger_link"/>
@@ -87,5 +87,5 @@
     <!-- Right Finger Joint -->
     <joint name="${prefix}right_finger_joint" type="prismatic">
-      <origin xyz="0.0175 0 0" rpy="0 0 0"/>
+      <origin xyz="0.035 0 0" rpy="0 0 0"/>
       <parent link="${prefix}onrobot_base_link"/>
       <child link="${prefix}right_finger_link"/>
