Commit message: Fix package 1

File: urdf/2fg7_macro.xacro (robot description, xacro)
@@ -101,5 +101,14 @@
     </joint>
     <!-- Transmission for ROS Control -->
-    <xacro:transmission_macro prefix="${prefix}" joint_name="finger_width"/>
+    <transmission name="${prefix}finger_width_trans">
+      <type>transmission_interface/SimpleTransmission</type>
+      <joint name="${prefix}finger_width">
+        <hardwareInterface>hardware_interface/PositionJointInterface</hardwareInterface>
+      </joint>
+      <actuator name="${prefix}finger_width_motor">
+        <hardwareInterface>hardware_interface/PositionJointInterface</hardwareInterface>
+        <mechanicalReduction>1</mechanicalReduction>
+      </actuator>
+    </transmission>
   </xacro:macro>
 </robot>

File: urdf/inc/2fg7_gazebo.xacro (robot description, xacro)
@@ -27,5 +27,5 @@
         <joint>${prefix}left_finger_joint</joint>
         <mimicJoint>${prefix}right_finger_joint</mimicJoint>
-        <multiplier>1.0</multiplier>
+        <multiplier>-1.0</multiplier>
         <offset>0.0</offset>
       </plugin>

File: urdf/inc/3fg15_gazebo.xacro (robot description, xacro)
@@ -27,8 +27,8 @@
     <gazebo>
       <plugin filename="libroboticsgroup_upatras_gazebo_mimic_joint_plugin.so" name="mimic_3fg15_left">
-        <joint>${prefix}finger_width</joint>
-        <mimicJoint>${prefix}left_finger_joint</mimicJoint>
-        <multiplier>${(2*pi/3)/(0.1175 - 0.0088)}</multiplier>
-        <offset>${-pi/3 - (2*pi/3)/(0.1175 - 0.0088) * 0.0088}</offset>
+        <joint>${prefix}left_finger_joint</joint>
+        <mimicJoint>${prefix}finger_diameter</mimicJoint>
+        <multiplier>${(2*pi/3)/(0.150 - 0.0)}</multiplier>
+        <offset>${-pi/3}</offset>
       </plugin>
     </gazebo>
@@ -36,8 +36,8 @@
     <gazebo>
       <plugin filename="libroboticsgroup_upatras_gazebo_mimic_joint_plugin.so" name="mimic_3fg15_right">
-        <joint>${prefix}finger_width</joint>
-        <mimicJoint>${prefix}right_finger_joint</mimicJoint>
-        <multiplier>${(2*pi/3)/(0.1175 - 0.0088)}</multiplier>
-        <offset>${-pi/3 - (2*pi/3)/(0.1175 - 0.0088) * 0.0088}</offset>
+        <joint>${prefix}right_finger_joint</joint>
+        <mimicJoint>${prefix}finger_diameter</mimicJoint>
+        <multiplier>${(2*pi/3)/(0.150 - 0.0)}</multiplier>
+        <offset>${-pi/3}</offset>
       </plugin>
     </gazebo>
@@ -45,8 +45,8 @@
     <gazebo>
       <plugin filename="libroboticsgroup_upatras_gazebo_mimic_joint_plugin.so" name="mimic_3fg15_middle">
-        <joint>${prefix}finger_width</joint>
-        <mimicJoint>${prefix}middle_finger_joint</mimicJoint>
-        <multiplier>${(2*pi/3)/(0.1175 - 0.0088)}</multiplier>
-        <offset>${-pi/3 - (2*pi/3)/(0.1175 - 0.0088) * 0.0088}</offset>
+        <joint>${prefix}middle_finger_joint</joint>
+        <mimicJoint>${prefix}finger_diameter</mimicJoint>
+        <multiplier>${(2*pi/3)/(0.150 - 0.0)}</multiplier>
+        <offset>${-pi/3}</offset>
       </plugin>
     </gazebo>

File: urdf/onrobot_macro.xacro (robot description, xacro)
@@ -13,5 +13,4 @@
       port:=502
       device_address:=65
-      num_cups:=4
     ">
     <!-- ====================== INCLUSIONES COMUNES ====================== -->
@@ -27,6 +26,6 @@
       <xacro:onrobot_rg6 prefix="${prefix}"/>
     </xacro:if>
-    <!-- ====================== 2FG7 / 2FG14 ====================== -->
-    <xacro:if value="${onrobot_type == '2fg7' or onrobot_type == '2fg14'}">
+    <!-- ====================== 2FG7 ====================== -->
+    <xacro:if value="${onrobot_type == '2fg7'}">
       <xacro:include filename="$(find onrobot_description)/urdf/2fg7_macro.xacro"/>
       <xacro:onrobot_2fg7 prefix="${prefix}" onrobot_type="${onrobot_type}"/>
@@ -37,34 +36,35 @@
       <xacro:onrobot_3fg15 prefix="${prefix}"/>
     </xacro:if>
-    <!-- ====================== VGC10 ====================== -->
-    <xacro:if value="${onrobot_type == 'vgc10'}">
-      <xacro:include filename="$(find onrobot_description)/urdf/vg_macro.xacro"/>
-      <xacro:include filename="$(find onrobot_description)/urdf/vgc10_gazebo.xacro"/>
-      <xacro:onrobot_vg prefix="${prefix}" onrobot_type="vgc10" num_cups="${num_cups}"/>
-    </xacro:if>
     <!-- ====================== GAZEBO: Plugins y Propiedades ====================== -->
     <xacro:if value="${sim_gazebo}">
-      <!-- Solo para 2FG7 (pinzas) -->
-      <xacro:if value="${onrobot_type == '2fg7' or onrobot_type == '2fg14'}">
-        <xacro:include filename="$(find onrobot_description)/urdf/2fg7_gazebo.xacro"/>
+      <!-- Gazebo ROS Control Plugin -->
+      <gazebo>
+        <plugin filename="libgazebo_ros2_control.so" name="gazebo_ros2_control">
+          <parameters>$(find onrobot_description)/config/gazebo_controllers.yaml</parameters>
+        </plugin>
+      </gazebo>
+      <!-- Para 2FG7 -->
+      <xacro:if value="${onrobot_type == '2fg7'}">
+        <xacro:include filename="$(find onrobot_description)/urdf/inc/2fg7_gazebo.xacro"/>
         <xacro:onrobot_2fg7_grasp_plugin prefix="${prefix}"/>
         <xacro:onrobot_2fg7_mimic_plugin prefix="${prefix}"/>
         <xacro:onrobot_2fg7_gazebo_properties prefix="${prefix}"/>
       </xacro:if>
-      <!-- Solo para VGC10 (vacío) -->
-      <xacro:if value="${onrobot_type == 'vgc10'}">
-        <xacro:onrobot_vgc10_vacuum_plugin prefix="${prefix}" num_cups="${num_cups}"/>
-        <xacro:onrobot_vgc10_gazebo_properties prefix="${prefix}"/>
+      <!-- Para 3FG15 -->
+      <xacro:if value="${onrobot_type == '3fg15'}">
+        <xacro:include filename="$(find onrobot_description)/urdf/inc/3fg15_gazebo.xacro"/>
+        <xacro:onrobot_3fg15_grasp_plugin prefix="${prefix}"/>
+        <xacro:onrobot_3fg15_mimic_plugin prefix="${prefix}"/>
+        <xacro:onrobot_3fg15_gazebo_properties prefix="${prefix}"/>
       </xacro:if>
     </xacro:if>
-    <!-- ====================== ROS2 CONTROL (REAL) ====================== -->
-    <xacro:unless value="${use_fake_hardware}">
+    <!-- ====================== ROS2 CONTROL ====================== -->
+    <xacro:if value="${not use_fake_hardware}">
       <ros2_control name="OnRobotGripper" type="system">
         <hardware>
-          <!-- Selección del plugin según tipo -->
           <xacro:if value="${onrobot_type == '3fg15'}">
             <plugin>onrobot_driver::ThreeFGHardwareInterface</plugin>
           </xacro:if>
-          <xacro:elseif value="${onrobot_type == '2fg7' or onrobot_type == '2fg14'}">
+          <xacro:elseif value="${onrobot_type == '2fg7'}">
             <plugin>onrobot_driver::TwoFGHardwareInterface</plugin>
           </xacro:elseif>
@@ -72,11 +72,4 @@
             <plugin>onrobot_driver::RGHardwareInterface</plugin>
           </xacro:elseif>
-          <xacro:elseif value="${onrobot_type == 'vgc10'}">
-            <plugin>onrobot_driver::VGCHardwareInterface</plugin>
-          </xacro:elseif>
-          <xacro:else>
-            <plugin>onrobot_driver::TwoFGHardwareInterface</plugin> <!-- fallback -->
-          </xacro:else>
-          <!-- Parámetros comunes -->
           <param name="onrobot_type">${onrobot_type}</param>
           <param name="prefix">${prefix}</param>
@@ -86,7 +79,6 @@
           <param name="port">${port}</param>
           <param name="device_address">${device_address}</param>
-          <param name="use_fake_hardware">false</param>
         </hardware>
-        <!-- JOINT DE CONTROL SEGÚN TIPO -->
+        <!-- Joint definitions -->
         <xacro:if value="${onrobot_type == '3fg15'}">
           <joint name="${prefix}finger_diameter">
@@ -96,5 +88,5 @@
           </joint>
         </xacro:if>
-        <xacro:unless value="${onrobot_type == '3fg15'}">
+        <xacro:else>
           <joint name="${prefix}finger_width">
             <command_interface name="position"/>
@@ -102,7 +94,7 @@
             <state_interface name="velocity"/>
           </joint>
-        </xacro:unless>
+        </xacro:else>
       </ros2_control>
-    </xacro:unless>
+    </xacro:if>
   </xacro:macro>
 </robot>
