Commit message: 3fg15 gripper update

File: urdf/2fg7_macro.xacro (robot description, xacro)
@@ -2,4 +2,5 @@
 <robot xmlns:xacro="http://ros.org/wiki/xacro">
   <xacro:include filename="$(find onrobot_description)/urdf/inc/common_utils.xacro" />
+  <xacro:include filename="$(find onrobot_description)/urdf/inc/2fg7_materials.xacro" />
   <xacro:macro name="onrobot_2fg7" params="prefix onrobot_type:='2fg7'">
     <!-- Base Link -->
@@ -73,9 +74,9 @@
       <child link="${prefix}finger_width_mock_link"/>
       <axis xyz="0 0 1"/>
-      <limit lower="0.035" upper="0.07" velocity="0.45" effort="140"/>
+      <limit lower="0" upper="0.035" velocity="0.45" effort="140"/>
     </joint>
     <!-- Left Finger Joint -->
     <joint name="${prefix}left_finger_joint" type="prismatic">
-      <origin xyz="-0.035 0 0" rpy="0 0 0"/>
+      <origin xyz="-0.0175 0 0" rpy="0 0 0"/>
       <parent link="${prefix}onrobot_base_link"/>
       <child link="${prefix}left_finger_link"/>
@@ -86,5 +87,5 @@
     <!-- Right Finger Joint -->
     <joint name="${prefix}right_finger_joint" type="prismatic">
-      <origin xyz="0.035 0 0" rpy="0 0 0"/>
+      <origin xyz="0.0175 0 0" rpy="0 0 0"/>
       <parent link="${prefix}onrobot_base_link"/>
       <child link="${prefix}right_finger_link"/>

File: urdf/3fg15_macro.xacro (robot description, xacro)
@@ -2,140 +2,64 @@
 <robot xmlns:xacro="http://ros.org/wiki/xacro">
   <xacro:include filename="$(find onrobot_description)/urdf/inc/common_utils.xacro" />
-  <!-- Macro para OnRobot 3FG15 -->
+  <xacro:include filename="$(find onrobot_description)/urdf/inc/2fg7_materials.xacro" />
+  <!-- ============================================= -->
+  <!-- Usa joint: finger_width → topic: /finger_width_controller/commands -->
+  <!-- ============================================= -->
   <xacro:macro name="onrobot_3fg15" params="prefix onrobot_type:='3fg15'">
-    <!-- Constantes -->
-    <xacro:property name="min_diameter" value="0.000" />
-    <xacro:property name="max_diameter" value="0.150" />
-    <!-- Base Link -->
+    <!-- ====================== Base Link (STL COMPLETO) ====================== -->
     <link name="${prefix}onrobot_base_link">
       <inertial>
-        <origin xyz="0 0 0.04" rpy="0 0 0"/>
-        <mass value="1.2"/>
-        <inertia ixx="0.012" ixy="0.0" ixz="0.0" iyy="0.012" iyz="0.0" izz="0.008"/>
+        <origin xyz="0 0 0.05" rpy="${-pi/2} 0 0"/>
+        <mass value="1.8"/>
+        <inertia ixx="0.015" ixy="0.0" ixz="0.0" iyy="0.015" iyz="0.0" izz="0.010"/>
+      </inertial>
+      <visual>
+        <origin xyz="0 0 0.05" rpy="${-pi/2} 0 0"/>
+        <geometry>
+          <mesh filename="package://onrobot_description/meshes/3fg15/visual/3fg15.stl" scale="0.001 0.001 0.001"/>
+        </geometry>
+        <material name="onrobot_silver"/>
+      </visual>
+      <collision>
+        <origin xyz="0 0 0.05" rpy="${-pi/2} 0 0"/>
+        <geometry>
+          <mesh filename="package://onrobot_description/meshes/3fg15/collision/3fg15.stl" scale="0.001 0.001 0.001"/>
+        </geometry>
+      </collision>
+    </link>
+    <!-- ====================== Mock Link (invisible, solo para joint) ====================== -->
+    <link name="${prefix}finger_width_mock_link">
+      <inertial>
+        <origin xyz="0 0 0" rpy="0 0 0"/>
+        <mass value="0.001"/>
+        <inertia ixx="1e-6" ixy="0.0" ixz="0.0" iyy="1e-6" iyz="0.0" izz="1e-6"/>
       </inertial>
       <visual>
         <origin xyz="0 0 0" rpy="0 0 0"/>
-        <geometry>
-          <mesh filename="package://onrobot_description/meshes/3fg15/visual/base.stl" scale="0.001 0.001 0.001"/>
-        </geometry>
-      </visual>
-      <collision>
-        <origin xyz="0 0 0.04" rpy="0 0 0"/>
-        <geometry>
-          <mesh filename="package://onrobot_description/meshes/3fg15/collision/base.stl" scale="0.001 0.001 0.001"/>
-        </geometry>
-      </collision>
-    </link>
-    <!-- === DEDOS (con movimiento real via mimic) === -->
-    <!-- Left Finger -->
-    <link name="${prefix}left_finger_link">
-      <inertial>
-        <origin xyz="0 0 0" rpy="0 0 0"/>
-        <mass value="0.08"/>
-        <inertia ixx="0.00008" ixy="0.0" ixz="0.0" iyy="0.00008" iyz="0.0" izz="0.00008"/>
-      </inertial>
-      <visual>
-        <origin xyz="0 0 0" rpy="0 0 0"/>
-        <geometry>
-          <mesh filename="package://onrobot_description/meshes/3fg15/visual/left_finger.stl" scale="0.001 0.001 0.001"/>
-        </geometry>
+        <geometry><box size="0.001 0.001 0.001"/></geometry>
       </visual>
       <collision>
         <origin xyz="0 0 0" rpy="0 0 0"/>
-        <geometry>
-          <mesh filename="package://onrobot_description/meshes/3fg15/collision/left_finger.stl" scale="0.001 0.001 0.001"/>
-        </geometry>
+        <geometry><box size="0.001 0.001 0.001"/></geometry>
       </collision>
     </link>
-    <!-- Right Finger -->
-    <link name="${prefix}right_finger_link">
-      <inertial>
-        <origin xyz="0 0 0" rpy="0 0 0"/>
-        <mass value="0.08"/>
-        <inertia ixx="0.00008" ixy="0.0" ixz="0.0" iyy="0.00008" iyz="0.0" izz="0.00008"/>
-      </inertial>
-      <visual>
-        <origin xyz="0 0 0" rpy="0 0 0"/>
-        <geometry>
-          <mesh filename="package://onrobot_description/meshes/3fg15/visual/right_finger.stl" scale="0.001 0.001 0.001"/>
-        </geometry>
-      </visual>
-      <collision>
-        <origin xyz="0 0 0" rpy="0 0 0"/>
-        <geometry>
-          <mesh filename="package://onrobot_description/meshes/3fg15/collision/right_finger.stl" scale="0.001 0.001 0.001"/>
-        </geometry>
-      </collision>
-    </link>
-    <!-- Middle Finger -->
-    <link name="${prefix}middle_finger_link">
-      <inertial>
-        <origin xyz="0 0 0" rpy="0 0 0"/>
-        <mass value="0.08"/>
-        <inertia ixx="0.00008" ixy="0.0" ixz="0.0" iyy="0.00008" iyz="0.0" izz="0.00008"/>
-      </inertial>
-      <visual>
-        <origin xyz="0 0 0" rpy="0 0 0"/>
-        <geometry>
-          <mesh filename="package://onrobot_description/meshes/3fg15/visual/middle_finger.stl" scale="0.001 0.001 0.001"/>
-        </geometry>
-      </visual>
-      <collision>
-        <origin xyz="0 0 0" rpy="0 0 0"/>
-        <geometry>
-          <mesh filename="package://onrobot_description/meshes/3fg15/collision/middle_finger.stl" scale="0.001 0.001 0.001"/>
-        </geometry>
-      </collision>
-    </link>
-    <!-- Dummy link para control -->
-    <link name="${prefix}finger_width_mock_link"/>
-    <!-- JOINT PRINCIPAL (para el driver) -->
-    <joint name="${prefix}finger_diameter" type="prismatic">
+    <!-- ====================== Main Control Joint: finger_width (0 a 150 mm) ====================== -->
+    <joint name="${prefix}finger_width" type="prismatic">
       <parent link="${prefix}onrobot_base_link"/>
       <child link="${prefix}finger_width_mock_link"/>
-      <origin xyz="0 0 0" rpy="0 0 0"/>
-      <axis xyz="0 1 0"/>
-      <limit lower="0.0" upper="0.150" effort="200" velocity="0.5"/>
+      <origin xyz="0 0 0.05" rpy="0 0 0"/>
+      <axis xyz="0 0 1"/>
+      <limit lower="0.0" upper="0.150" effort="240" velocity="0.3"/>
+      <!-- 150 mm = 0.15 m (diámetro externo del 3FG15) -->
     </joint>
-    <!-- === DEDOS: REVOLUTE + MIMIC === -->
-    <xacro:property name="angle_per_meter" value="${(2*pi/3)/(0.150 - 0.0)}" />  <!-- 120° en 150mm -->
-    <xacro:property name="min_angle" value="${-pi/3}" />  <!-- -60° -->
-    <xacro:property name="offset" value="${min_angle - angle_per_meter * 0.0}" />
-    <!-- Left Finger -->
-    <joint name="${prefix}left_finger_joint" type="revolute">
-      <parent link="${prefix}onrobot_base_link"/>
-      <child link="${prefix}left_finger_link"/>
-      <origin xyz="0 0 0" rpy="${pi}" />
-      <axis xyz="0 0 1"/>
-      <limit lower="${-pi/3}" upper="${pi/3}" effort="200" velocity="0.5"/>
-      <mimic joint="${prefix}finger_diameter" multiplier="${angle_per_meter}" offset="${offset}"/>
-    </joint>
-    <!-- Right Finger -->
-    <joint name="${prefix}right_finger_joint" type="revolute">
-      <parent link="${prefix}onrobot_base_link"/>
-      <child link="${prefix}right_finger_link"/>
-      <origin xyz="0 0 0" rpy="0" />
-      <axis xyz="0 0 1"/>
-      <limit lower="${-pi/3}" upper="${pi/3}" effort="200" velocity="0.5"/>
-      <mimic joint="${prefix}finger_diameter" multiplier="${angle_per_meter}" offset="${offset}"/>
-    </joint>
-    <!-- Middle Finger -->
-    <joint name="${prefix}middle_finger_joint" type="revolute">
-      <parent link="${prefix}onrobot_base_link"/>
-      <child link="${prefix}middle_finger_link"/>
-      <origin xyz="0 0 0" rpy="${2*pi/3}" />
-      <axis xyz="0 0 1"/>
-      <limit lower="${-pi/3}" upper="${pi/3}" effort="200" velocity="0.5"/>
-      <mimic joint="${prefix}finger_diameter" multiplier="${angle_per_meter}" offset="${offset}"/>
-    </joint>
-    <!-- TCP -->
+    <!-- ====================== TCP Link (punto de agarre) ====================== -->
     <link name="${prefix}gripper_tcp"/>
     <joint name="${prefix}tcp_joint" type="fixed">
+      <origin xyz="0 0 0.08" rpy="0 0 0"/>
       <parent link="${prefix}onrobot_base_link"/>
       <child link="${prefix}gripper_tcp"/>
-      <origin xyz="0 0 0.13" rpy="0 0 0"/>
     </joint>
-    <!-- Transmission -->
-    <xacro:transmission_macro prefix="${prefix}" joint_name="finger_diameter"/>
+    <!-- ====================== Transmission (genera /finger_width_controller) ====================== -->
+    <xacro:transmission_macro prefix="${prefix}" joint_name="finger_width"/>
   </xacro:macro>
 </robot>

File: urdf/onrobot_macro.xacro (robot description, xacro)
@@ -1,5 +1,5 @@
 <?xml version="1.0"?>
 <robot xmlns:xacro="http://wiki.ros.org/xacro">
-  <!-- ====================== MACRO PRINCIPAL ONROBOT ====================== -->
+  <!-- Macro principal para todos los grippers OnRobot -->
   <xacro:macro name="onrobot"
     params="
@@ -13,8 +13,5 @@
       port:=502
       device_address:=65
-      num_cups:=4
     ">
-    <!-- ====================== INCLUSIONES COMUNES ====================== -->
-    <xacro:include filename="$(find onrobot_description)/urdf/inc/common_materials.xacro"/>
     <!-- ====================== RG2 ====================== -->
     <xacro:if value="${onrobot_type == 'rg2'}">
@@ -32,75 +29,50 @@
       <xacro:onrobot_2fg7 prefix="${prefix}" onrobot_type="${onrobot_type}"/>
     </xacro:if>
-    <!-- ====================== 3FG15 ====================== -->
+    <!-- ====================== 3FG15 (NUEVO) ====================== -->
     <xacro:if value="${onrobot_type == '3fg15'}">
       <xacro:include filename="$(find onrobot_description)/urdf/3fg15_macro.xacro"/>
       <xacro:onrobot_3fg15 prefix="${prefix}"/>
     </xacro:if>
-    <!-- ====================== VGC10 ====================== -->
-    <xacro:if value="${onrobot_type == 'vgc10'}">
-      <xacro:include filename="$(find onrobot_description)/urdf/vg_macro.xacro"/>
-      <xacro:include filename="$(find onrobot_description)/urdf/vgc10_gazebo.xacro"/>
-      <xacro:onrobot_vg prefix="${prefix}" onrobot_type="vgc10" num_cups="${num_cups}"/>
+    <!-- ====================== Gazebo Simulation ====================== -->
+    <xacro:if value="${sim_gazebo}">
+      <gazebo>
+        <plugin filename="libgazebo_ros2_control.so" name="gazebo_ros2_control">
+          <parameters>$(find onrobot_description)/config/onrobot_controllers.yaml</parameters>
+        </plugin>
+      </gazebo>
     </xacro:if>
-    <!-- ====================== GAZEBO: Plugins y Propiedades ====================== -->
-    <xacro:if value="${sim_gazebo}">
-      <!-- Solo para 2FG7 (pinzas) -->
-      <xacro:if value="${onrobot_type == '2fg7' or onrobot_type == '2fg14'}">
-        <xacro:include filename="$(find onrobot_description)/urdf/2fg7_gazebo.xacro"/>
-        <xacro:onrobot_2fg7_grasp_plugin prefix="${prefix}"/>
-        <xacro:onrobot_2fg7_mimic_plugin prefix="${prefix}"/>
-        <xacro:onrobot_2fg7_gazebo_properties prefix="${prefix}"/>
-      </xacro:if>
-      <!-- Solo para VGC10 (vacío) -->
-      <xacro:if value="${onrobot_type == 'vgc10'}">
-        <xacro:onrobot_vgc10_vacuum_plugin prefix="${prefix}" num_cups="${num_cups}"/>
-        <xacro:onrobot_vgc10_gazebo_properties prefix="${prefix}"/>
-      </xacro:if>
-    </xacro:if>
-    <!-- ====================== ROS2 CONTROL (REAL) ====================== -->
+    <!-- ====================== ROS2 Control ====================== -->
     <xacro:unless value="${use_fake_hardware}">
-      <ros2_control name="OnRobotGripper" type="system">
+      <ros2_control name="OnRobotGripper" type="actuator">
         <hardware>
-          <!-- Selección del plugin según tipo -->
-          <xacro:if value="${onrobot_type == '3fg15'}">
-            <plugin>onrobot_driver::ThreeFGHardwareInterface</plugin>
+          <!-- 2FG7, 2FG14 y 3FG15 usan el mismo driver -->
+          <xacro:if value="${onrobot_type == '2fg7' or onrobot_type == '2fg14' or onrobot_type == '3fg15'}">
+            <plugin>onrobot_driver::FGHardwareInterface</plugin>
+            <param name="onrobot_type">${onrobot_type}</param>
+            <param name="prefix">${prefix}</param>
+            <param name="connection_type">${connection_type}</param>
+            <param name="device">${device}</param>
+            <param name="ip_address">${ip_address}</param>
+            <param name="port">${port}</param>
+            <param name="device_address">${device_address}</param>
+            <param name="use_fake_hardware">false</param>
           </xacro:if>
-          <xacro:elseif value="${onrobot_type == '2fg7' or onrobot_type == '2fg14'}">
-            <plugin>onrobot_driver::TwoFGHardwareInterface</plugin>
-          </xacro:elseif>
-          <xacro:elseif value="${onrobot_type == 'rg2' or onrobot_type == 'rg6'}">
+          <!-- RG2 / RG6 -->
+          <xacro:if value="${onrobot_type == 'rg2' or onrobot_type == 'rg6'}">
             <plugin>onrobot_driver::RGHardwareInterface</plugin>
-          </xacro:elseif>
-          <xacro:elseif value="${onrobot_type == 'vgc10'}">
-            <plugin>onrobot_driver::VGCHardwareInterface</plugin>
-          </xacro:elseif>
-          <xacro:else>
-            <plugin>onrobot_driver::TwoFGHardwareInterface</plugin> <!-- fallback -->
-          </xacro:else>
-          <!-- Parámetros comunes -->
-          <param name="onrobot_type">${onrobot_type}</param>
-          <param name="prefix">${prefix}</param>
-          <param name="connection_type">${connection_type}</param>
-          <param name="device">${device}</param>
-          <param name="ip_address">${ip_address}</param>
-          <param name="port">${port}</param>
-          <param name="device_address">${device_address}</param>
-          <param name="use_fake_hardware">false</param>
+            <param name="onrobot_type">${onrobot_type}</param>
+            <param name="prefix">${prefix}</param>
+            <param name="connection_type">${connection_type}</param>
+            <param name="device">${device}</param>
+            <param name="ip_address">${ip_address}</param>
+            <param name="port">${port}</param>
+            <param name="use_fake_hardware">false</param>
+          </xacro:if>
         </hardware>
-        <!-- JOINT DE CONTROL SEGÚN TIPO -->
-        <xacro:if value="${onrobot_type == '3fg15'}">
-          <joint name="${prefix}finger_diameter">
-            <command_interface name="position"/>
-            <state_interface name="position"/>
-            <state_interface name="velocity"/>
-          </joint>
-        </xacro:if>
-        <xacro:unless value="${onrobot_type == '3fg15'}">
-          <joint name="${prefix}finger_width">
-            <command_interface name="position"/>
-            <state_interface name="position"/>
-            <state_interface name="velocity"/>
-          </joint>
-        </xacro:unless>
+        <joint name="${prefix}finger_width">
+          <command_interface name="position"/>
+          <state_interface name="position"/>
+          <state_interface name="velocity"/>
+        </joint>
       </ros2_control>
     </xacro:unless>

Commit message: 2FG7 - tcp update

File: urdf/2fg7_macro.xacro (robot description, xacro)
@@ -97,5 +97,5 @@
     <link name="${prefix}gripper_tcp"/>
     <joint name="${prefix}tcp_joint" type="fixed">
-      <origin xyz="0 0 0.08" rpy="0 0 0"/>
+      <origin xyz="0 0 0.1386" rpy="0 0 0"/> <!-- 138.6 mm respecto al tool0/base_link -->
       <parent link="${prefix}onrobot_base_link"/>
       <child link="${prefix}gripper_tcp"/>

Commit message: Update 2FG7 robot model: replace and add STL files, adjust URDF configurations
- Added new STL files for Quick Changer Robot side, official base, and fingers.
- Removed outdated STL files for base link and finger links.
- Updated URDF to reference new STL files and adjusted visual/collision origins and geometries.
- Modified joint limits for left and right fingers to correct range.

File: urdf/2fg7_macro.xacro (robot description, xacro)
@@ -12,14 +12,27 @@
       </inertial>
       <visual>
-        <origin xyz="0 0 0" rpy="0 0 0"/>
+        <origin xyz="0 0 0" rpy="-1.570796 0 -1.570796"/>
         <geometry>
-          <mesh filename="package://onrobot_description/meshes/2fg7/visual/base_link.stl" scale="0.001 0.001 0.001"/>
+          <mesh filename="package://onrobot_description/meshes/2fg7/visual/Quick_Changer_Robot_side_1.stl" scale="0.001 0.001 0.001"/>
+        </geometry>
+        <material name="onrobot_silver"/>
+      </visual>
+      <visual>
+        <origin xyz="-0.05539 -0.14017 -0.28046" rpy="1.570796 0 0"/>
+        <geometry>
+          <mesh filename="package://onrobot_description/meshes/2fg7/visual/official_base_onrobot.stl" scale="0.001 0.001 0.001"/>
         </geometry>
         <material name="onrobot_silver"/>
       </visual>
       <collision>
-        <origin xyz="0 0 0" rpy="0 0 0"/>
+        <origin xyz="0 0 0" rpy="-1.570796 0 -1.570796"/>
         <geometry>
-          <box size="0.045 0.045 0.04"/>
+          <mesh filename="package://onrobot_description/meshes/2fg7/collision/Quick_Changer_Robot_side_1.stl" scale="0.001 0.001 0.001"/>
+        </geometry>
+      </collision>
+      <collision>
+        <origin xyz="-0.05539 -0.14017 -0.28046" rpy="1.570796 0 0"/>
+        <geometry>
+          <mesh filename="package://onrobot_description/meshes/2fg7/collision/official_base_onrobot.stl" scale="0.001 0.001 0.001"/>
         </geometry>
       </collision>
@@ -33,14 +46,14 @@
       </inertial>
       <visual>
-        <origin xyz="0 0 0" rpy="0 0 0"/>
+        <origin xyz="-0.05539 -0.14017 -0.28046" rpy="1.570796 0 0"/>
         <geometry>
-          <mesh filename="package://onrobot_description/meshes/2fg7/visual/left_finger_link.stl" scale="0.001 0.001 0.001"/>
+          <mesh filename="package://onrobot_description/meshes/2fg7/visual/official_left_finger.stl" scale="0.001 0.001 0.001"/>
         </geometry>
         <material name="onrobot_silver"/>
       </visual>
       <collision>
-        <origin xyz="0 0 0" rpy="0 0 0"/>
+        <origin xyz="-0.05539 -0.14017 -0.28046" rpy="1.570796 0 0"/>
         <geometry>
-          <box size="0.008 0.025 0.06"/>
+          <mesh filename="package://onrobot_description/meshes/2fg7/collision/official_left_finger.stl" scale="0.001 0.001 0.001"/>
         </geometry>
       </collision>
@@ -53,14 +66,14 @@
       </inertial>
       <visual>
-        <origin xyz="0 0 0" rpy="0 0 0"/>
+        <origin xyz="-0.05539 -0.14017 -0.28046" rpy="1.570796 0 0"/>
         <geometry>
-          <mesh filename="package://onrobot_description/meshes/2fg7/visual/right_finger_link.stl" scale="0.001 0.001 0.001"/>
+          <mesh filename="package://onrobot_description/meshes/2fg7/visual/official_right_finger.stl" scale="0.001 0.001 0.001"/>
         </geometry>
         <material name="onrobot_silver"/>
       </visual>
       <collision>
-        <origin xyz="0 0 0" rpy="0 0 0"/>
+        <origin xyz="-0.05539 -0.14017 -0.28046" rpy="1.570796 0 0"/>
         <geometry>
-          <box size="0.008 0.025 0.06"/>
+          <mesh filename="package://onrobot_description/meshes/2fg7/collision/official_right_finger.stl" scale="0.001 0.001 0.001"/>
         </geometry>
       </collision>
@@ -78,14 +91,14 @@
     <!-- Left Finger Joint -->
     <joint name="${prefix}left_finger_joint" type="prismatic">
-      <origin xyz="-0.035 0 0" rpy="0 0 0"/>
+      <origin xyz="-0.0302 0 0" rpy="0 0 0"/>
       <parent link="${prefix}onrobot_base_link"/>
       <child link="${prefix}left_finger_link"/>
       <axis xyz="1 0 0"/>
-      <limit lower="0.0" upper="0.0175" effort="140" velocity="0.45"/>
+      <limit lower="-0.0175" upper="0.0" effort="140" velocity="0.45"/>
       <mimic joint="${prefix}finger_width" multiplier="0.5" offset="0"/>
     </joint>
     <!-- Right Finger Joint -->
     <joint name="${prefix}right_finger_joint" type="prismatic">
-      <origin xyz="0.035 0 0" rpy="0 0 0"/>
+      <origin xyz="0.0302 0 0" rpy="0 0 0"/>
       <parent link="${prefix}onrobot_base_link"/>
       <child link="${prefix}right_finger_link"/>
