Commit message: english translation - comments and prints

File: urdf/2fg7_macro.xacro (robot description, xacro)
@@ -110,5 +110,5 @@
     <link name="${prefix}gripper_tcp"/>
     <joint name="${prefix}tcp_joint" type="fixed">
-      <origin xyz="0 0 0.1386" rpy="0 0 0"/> <!-- 138.6 mm respecto al tool0/base_link -->
+      <origin xyz="0 0 0.1386" rpy="0 0 0"/> <!-- 138.6 mm relative to tool0/base_link -->
       <parent link="${prefix}onrobot_base_link"/>
       <child link="${prefix}gripper_tcp"/>

File: urdf/3fg15_macro.xacro (robot description, xacro)
@@ -4,7 +4,7 @@
   <xacro:include filename="$(find onrobot_description)/urdf/inc/common_materials.xacro" />
   <xacro:macro name="onrobot_3fg15" params="prefix onrobot_type:='3fg15'">
-    <!-- ==================== Parámetros de escala visual/real ==================== -->
-    <xacro:property name="max_real_width"   value="0.150"/>   <!-- metros (ancho máximo real) -->
-    <xacro:property name="max_visual_angle" value="2.9"/>     <!-- radianes cuando está totalmente abierto -->
+    <!-- ==================== Visual/real scale parameters ==================== -->
+    <xacro:property name="max_real_width"   value="0.150"/>   <!-- meters (max real width) -->
+    <xacro:property name="max_visual_angle" value="2.9"/>     <!-- radians when fully open -->
     <xacro:property name="angle_multiplier" value="${-max_visual_angle / max_real_width}"/> <!-- ≈ -19.3333 -->
     <!-- ====================== Base Link ====================== -->
@@ -29,5 +29,5 @@
       </collision>
     </link>
-    <!-- ====================== Dedos ====================== -->
+    <!-- ====================== Fingers ====================== -->
     <link name="${prefix}left_finger_link">
       <inertial>
@@ -90,5 +90,5 @@
       </collision>
     </link>
-    <!-- ====================== Mock link (solo para el joint prismatic) ====================== -->
+    <!-- ====================== Mock link (only for prismatic joint) ====================== -->
     <link name="${prefix}finger_width_mock_link">
       <inertial>
@@ -97,5 +97,5 @@
       </inertial>
     </link>
-    <!-- ====================== Joint principal EN METROS (para el robot real) ====================== -->
+    <!-- ====================== Main joint IN METERS (for real robot) ====================== -->
     <joint name="${prefix}finger_width" type="prismatic">
       <parent link="${prefix}onrobot_base_link"/>
@@ -106,5 +106,5 @@
       <dynamics damping="5.0" friction="0.0"/>
     </joint>
-    <!-- ====================== Joints de dedos (revolute + mimic escalado) ====================== -->
+    <!-- ====================== Finger joints (revolute + scaled mimic) ====================== -->
     <joint name="${prefix}left_finger_joint" type="revolute">
       <parent link="${prefix}onrobot_base_link"/>
@@ -131,12 +131,12 @@
       <mimic joint="${prefix}finger_width" multiplier="${angle_multiplier}" offset="${max_visual_angle}"/>
     </joint>
-    <!-- ====================== TCP (punto de agarre) ====================== -->
+    <!-- ====================== TCP (grasp point) ====================== -->
     <link name="${prefix}gripper_tcp"/>
     <joint name="${prefix}tcp_joint" type="fixed">
       <parent link="${prefix}onrobot_base_link"/>
       <child link="${prefix}gripper_tcp"/>
-      <origin xyz="0 0 0.135" rpy="0 0 0"/> <!-- 135 mm desde la base según datasheet oficial -->
+      <origin xyz="0 0 0.135" rpy="0 0 0"/> <!-- 135 mm from the base according to official datasheet -->
     </joint>
-    <!-- ====================== Transmission para ros2_control ====================== -->
+    <!-- ====================== Transmission for ros2_control ====================== -->
     <xacro:transmission_macro prefix="${prefix}" joint_name="finger_width"/>
   </xacro:macro>

File: urdf/3fg15_macro_bk.xacro (robot description, xacro)
@@ -25,6 +25,6 @@
       </collision>
     </link>
-    <!-- ====================== Dedos individuales ====================== -->
-    <!-- Dedo izquierdo (120° a la izquierda) -->
+    <!-- ====================== Individual fingers ====================== -->
+    <!-- Left finger (120° to the left) -->
     <link name="${prefix}left_finger_link">
       <inertial>
@@ -47,5 +47,5 @@
       </collision>
     </link>
-    <!-- Dedo derecho (120° a la derecha) -->
+    <!-- Right finger (120° to the right) -->
     <link name="${prefix}right_finger_link">
       <inertial>
@@ -68,5 +68,5 @@
       </collision>
     </link>
-    <!-- Dedo central (hacia abajo) -->
+    <!-- Center finger (downward) -->
     <link name="${prefix}center_finger_link">
       <inertial>
@@ -89,5 +89,5 @@
       </collision>
     </link>
-    <!-- ====================== Mock link para el joint principal ====================== -->
+    <!-- ====================== Mock link for the main joint ====================== -->
     <link name="${prefix}finger_width_mock_link">
       <inertial>
@@ -96,5 +96,5 @@
       </inertial>
     </link>
-    <!-- ====================== Joint principal de control (0 a 150 mm) ====================== -->
+    <!-- ====================== Main control joint (0 to 150 mm) ====================== -->
     <joint name="${prefix}finger_width" type="revolute">
       <parent link="${prefix}onrobot_base_link"/>
@@ -104,5 +104,5 @@
       <limit lower="0.0" upper="2.8" effort="140" velocity="0.45"/>
     </joint>
-    <!-- ====================== Eje Z visual (debug) ====================== -->
+    <!-- ====================== Visual Z axis (debug) ====================== -->
     <!--
     <link name="${prefix}z_axis_visual_link2">
@@ -155,6 +155,6 @@
     </joint>
     -->
-    <!-- ====================== Joints de los dedos (mimic del principal) ====================== -->
-    <!-- Los tres dedos se mueven radialmente según el ancho (finger_width / 3 por dedo) -->
+    <!-- ====================== Finger joints (mimic from main) ====================== -->
+    <!-- The three fingers move radially according to the width (finger_width / 3 per finger) -->
     <joint name="${prefix}left_finger_joint" type="revolute">
       <origin xyz="-0.026 0.015 0" rpy = "0 0 0"/>
@@ -181,5 +181,5 @@
       <mimic joint="${prefix}finger_width"  offset="0"/>
     </joint>
-    <!-- ====================== TCP (punto de agarre) ====================== -->
+    <!-- ====================== TCP (grasp point) ====================== -->
     <link name="${prefix}gripper_tcp"/>
     <joint name="${prefix}tcp_joint" type="fixed">
@@ -188,5 +188,5 @@
       <child link="${prefix}gripper_tcp"/>
     </joint>
-    <!-- ====================== Transmission para ROS Control ====================== -->
+    <!-- ====================== Transmission for ROS Control ====================== -->
     <xacro:transmission_macro prefix="${prefix}" joint_name="finger_width"/>
   </xacro:macro>

File: urdf/onrobot_macro.xacro (robot description, xacro)
@@ -1,5 +1,5 @@
 <?xml version="1.0"?>
 <robot xmlns:xacro="http://wiki.ros.org/xacro">
-  <!-- Macro principal para todos los grippers OnRobot -->
+  <!-- Main macro for all OnRobot grippers -->
   <xacro:macro name="onrobot"
     params="
