Commit message: Refactor OnRobot URDF/XACRO files for improved structure and new model support
- Added new material definitions for "onrobot_black" in common_materials.xacro.
- Removed deprecated common_utils.xacro and rg_common.xacro files.
- Updated onrobot.urdf.xacro to change default onrobot_type to "2fg7" and added use_mock_hardware argument.
- Refactored onrobot_macro.xacro to streamline hardware interface definitions and removed unnecessary fake hardware configurations.
- Deleted outdated rg2_macro.xacro and rg6_macro.xacro files.
- Introduced new vgc10_macro.xacro for VGC10 model support with appropriate links and joints.

File: urdf/2fg7_macro.xacro (robot description, xacro)
@@ -80,5 +80,10 @@
     </link>
     <!-- Dummy link for the main control joint -->
-    <link name="${prefix}finger_width_mock_link"/>
+    <link name="${prefix}finger_width_mock_link">
+      <inertial>
+        <mass value="1e-9"/>
+        <inertia ixx="1e-9" ixy="0" ixz="0" iyy="1e-9" iyz="0" izz="1e-9"/>
+      </inertial>
+    </link>
     <!-- Main control joint (finger_width) -->
     <joint name="${prefix}finger_width" type="prismatic">
@@ -96,5 +101,5 @@
       <axis xyz="1 0 0"/>
       <limit lower="-0.0175" upper="0.0" effort="140" velocity="0.45"/>
-      <mimic joint="${prefix}finger_width" multiplier="0.5" offset="0"/>
+      <mimic joint="${prefix}finger_width" multiplier="-0.5" offset="0.0175"/>
     </joint>
     <!-- Right Finger Joint -->
@@ -105,5 +110,5 @@
       <axis xyz="-1 0 0"/>
       <limit lower="-0.0175" upper="0.0" effort="140" velocity="0.45"/>
-      <mimic joint="${prefix}finger_width" multiplier="0.5" offset="0"/>
+      <mimic joint="${prefix}finger_width" multiplier="-0.5" offset="0.0175"/>
     </joint>
     <!-- TCP Link -->
@@ -114,6 +119,4 @@
       <child link="${prefix}gripper_tcp"/>
     </joint>
-    <!-- Transmission for ROS Control -->
-    <xacro:transmission_macro prefix="${prefix}" joint_name="finger_width"/>
   </xacro:macro>
 </robot>

File: urdf/3fg15_macro.xacro (robot description, xacro)
@@ -138,6 +138,4 @@
       <origin xyz="0 0 0.135" rpy="0 0 0"/> <!-- 135 mm from the base according to official datasheet -->
     </joint>
-    <!-- ====================== Transmission for ros2_control ====================== -->
-    <xacro:transmission_macro prefix="${prefix}" joint_name="finger_width"/>
   </xacro:macro>
 </robot>

File: urdf/inc/common_materials.xacro (robot description, xacro)
@@ -8,3 +8,6 @@
     <color rgba="0.700 0.700 0.700 1.000"/>
   </material>
+  <material name="onrobot_black">
+    <color rgba="0.100 0.100 0.100 1.000"/>
+  </material>
 </robot>

File: urdf/inc/common_utils.xacro (robot description, xacro)
@@ -1,24 +1,4 @@
 <?xml version="1.0"?>
 <robot xmlns:xacro="http://www.ros.org/wiki/xacro">
-  <!-- Gazebo plugin macro (for ros2_control simulation) -->
-  <xacro:macro name="gazebo_plugin" params="prefix">
-    <gazebo>
-      <plugin filename="libgazebo_ros2_control.so" name="gazebo_ros2_control">
-        <!-- Add additional parameters as needed -->
-      </plugin>
-    </gazebo>
-  </xacro:macro>
-  <!-- Simple transmission macro for a joint -->
-  <xacro:macro name="transmission_macro" params="prefix joint_name">
-    <transmission name="${prefix}${joint_name}_trans">
-      <type>transmission_interface/SimpleTransmission</type>
-      <joint name="${prefix}${joint_name}">
-        <hardwareInterface>hardware_interface/PositionJointInterface</hardwareInterface>
-      </joint>
-      <actuator name="${prefix}${joint_name}_motor">
-        <hardwareInterface>hardware_interface/PositionJointInterface</hardwareInterface>
-        <mechanicalReduction>1</mechanicalReduction>
-      </actuator>
-    </transmission>
-  </xacro:macro>
+  <!-- Common utilities for OnRobot descriptions -->
 </robot>

File: urdf/onrobot.urdf.xacro (robot description, xacro)
@@ -1,10 +1,9 @@
 <?xml version="1.0"?>
-<robot xmlns:xacro="http://wiki.ros.org/xacro" name="$(arg name)">
+<robot xmlns:xacro="http://wiki.ros.org/xacro" name="onrobot">
     <!-- Arguments -->
-    <xacro:arg name="onrobot_type" default="rg2"/>
+    <xacro:arg name="onrobot_type" default="2fg7"/>
     <xacro:arg name="prefix" default=""/>
-    <xacro:arg name="name" default="onrobot"/>
-    <xacro:arg name="sim_gazebo" default="false"/>
     <xacro:arg name="use_fake_hardware" default="false"/>
+    <xacro:arg name="use_mock_hardware" default="false"/>
     <xacro:arg name="connection_type" default="serial"/>
     <xacro:arg name="device" default="/tmp/ttyUR"/>
@@ -17,6 +16,6 @@
         onrobot_type="$(arg onrobot_type)"
         prefix="$(arg prefix)"
-        sim_gazebo="$(arg sim_gazebo)"
         use_fake_hardware="$(arg use_fake_hardware)"
+        use_mock_hardware="$(arg use_mock_hardware)"
         connection_type="$(arg connection_type)"
         device="$(arg device)"

File: urdf/onrobot_macro.xacro (robot description, xacro)
@@ -6,6 +6,6 @@
       onrobot_type
       prefix:=''
-      sim_gazebo:=false
       use_fake_hardware:=false
+      use_mock_hardware:=false
       connection_type:=tcp
       device:=/tmp/ttyUR
@@ -14,16 +14,6 @@
       device_address:=65
     ">
-    <!-- ====================== RG2 ====================== -->
-    <xacro:if value="${onrobot_type == 'rg2'}">
-      <xacro:include filename="$(find onrobot_description)/urdf/rg2_macro.xacro"/>
-      <xacro:onrobot_rg2 prefix="${prefix}"/>
-    </xacro:if>
-    <!-- ====================== RG6 ====================== -->
-    <xacro:if value="${onrobot_type == 'rg6'}">
-      <xacro:include filename="$(find onrobot_description)/urdf/rg6_macro.xacro"/>
-      <xacro:onrobot_rg6 prefix="${prefix}"/>
-    </xacro:if>
-    <!-- ====================== 2FG7 / 2FG14 ====================== -->
-    <xacro:if value="${onrobot_type == '2fg7' or onrobot_type == '2fg14'}">
+    <!-- ====================== 2FG7 ====================== -->
+    <xacro:if value="${onrobot_type == '2fg7'}">
       <xacro:include filename="$(find onrobot_description)/urdf/2fg7_macro.xacro"/>
       <xacro:onrobot_2fg7 prefix="${prefix}" onrobot_type="${onrobot_type}"/>
@@ -34,126 +24,49 @@
       <xacro:onrobot_3fg15 prefix="${prefix}"/>
     </xacro:if>
-    <!-- ====================== Gazebo Simulation ====================== -->
-    <xacro:if value="${sim_gazebo}">
-      <gazebo>
-        <plugin filename="libgazebo_ros2_control.so" name="gazebo_ros2_control">
-          <parameters>$(find onrobot_description)/config/onrobot_controllers.yaml</parameters>
-        </plugin>
-      </gazebo>
+    <!-- ====================== VGC10 ====================== -->
+    <xacro:if value="${onrobot_type == 'vgc10'}">
+      <xacro:include filename="$(find onrobot_description)/urdf/vgc10_macro.xacro"/>
+      <xacro:onrobot_vgc10 prefix="${prefix}"/>
     </xacro:if>
-    <!-- ====================== ROS2 Control ====================== -->
-    <xacro:unless value="${use_fake_hardware}">
+    <!-- ====================== ROS2 Control (Humble) ====================== -->
+    <xacro:if value="${onrobot_type in ['2fg7', '3fg15']}">
       <ros2_control name="OnRobotGripper" type="actuator">
         <hardware>
-          <!-- 2FG7 / 2FG14 - TwoFG Hardware Interface -->
-          <xacro:if value="${onrobot_type == '2fg7' or onrobot_type == '2fg14'}">
-            <plugin>onrobot_driver::TwoFGHardwareInterface</plugin>
-            <param name="onrobot_type">${onrobot_type}</param>
-            <param name="prefix">${prefix}</param>
-            <param name="connection_type">${connection_type}</param>
-            <param name="device">${device}</param>
-            <param name="ip_address">${ip_address}</param>
-            <param name="port">${port}</param>
-            <param name="device_address">${device_address}</param>
-            <param name="use_fake_hardware">false</param>
+          <xacro:if value="${use_mock_hardware}">
+            <plugin>mock_components/GenericSystem</plugin>
           </xacro:if>
-          <!-- 3FG15 - ThreeFG Hardware Interface -->
-          <xacro:if value="${onrobot_type == '3fg15'}">
-            <plugin>onrobot_driver::ThreeFGHardwareInterface</plugin>
-            <param name="onrobot_type">${onrobot_type}</param>
-            <param name="prefix">${prefix}</param>
-            <param name="connection_type">${connection_type}</param>
-            <param name="device">${device}</param>
-            <param name="ip_address">${ip_address}</param>
-            <param name="port">${port}</param>
-            <param name="device_address">${device_address}</param>
-            <param name="use_fake_hardware">false</param>
-          </xacro:if>
-          <!-- RG2 / RG6 - RG Hardware Interface -->
-          <xacro:if value="${onrobot_type == 'rg2' or onrobot_type == 'rg6'}">
-            <plugin>onrobot_driver::RGHardwareInterface</plugin>
-            <param name="onrobot_type">${onrobot_type}</param>
-            <param name="prefix">${prefix}</param>
-            <param name="connection_type">${connection_type}</param>
-            <param name="device">${device}</param>
-            <param name="ip_address">${ip_address}</param>
-            <param name="port">${port}</param>
-            <param name="device_address">${device_address}</param>
-            <param name="use_fake_hardware">false</param>
-          </xacro:if>
+          <xacro:unless value="${use_mock_hardware}">
+            <!-- 2FG7 - TwoFG Hardware Interface -->
+            <xacro:if value="${onrobot_type == '2fg7'}">
+              <plugin>onrobot_driver::TwoFGHardwareInterface</plugin>
+              <param name="onrobot_type">${onrobot_type}</param>
+              <param name="prefix">${prefix}</param>
+              <param name="connection_type">${connection_type}</param>
+              <param name="device">${device}</param>
+              <param name="ip_address">${ip_address}</param>
+              <param name="port">${port}</param>
+              <param name="device_address">${device_address}</param>
+              <param name="use_fake_hardware">${use_fake_hardware}</param>
+            </xacro:if>
+            <!-- 3FG15 - ThreeFG Hardware Interface -->
+            <xacro:if value="${onrobot_type == '3fg15'}">
+              <plugin>onrobot_driver::ThreeFGHardwareInterface</plugin>
+              <param name="onrobot_type">${onrobot_type}</param>
+              <param name="prefix">${prefix}</param>
+              <param name="connection_type">${connection_type}</param>
+              <param name="device">${device}</param>
+              <param name="ip_address">${ip_address}</param>
+              <param name="port">${port}</param>
+              <param name="device_address">${device_address}</param>
+              <param name="use_fake_hardware">${use_fake_hardware}</param>
+            </xacro:if>
+          </xacro:unless>
         </hardware>
-        <!-- Joint configuration for all gripper types -->
-        <xacro:if value="${onrobot_type == '2fg7' or onrobot_type == '2fg14' or onrobot_type == '3fg15'}">
-          <joint name="${prefix}finger_width">
-            <command_interface name="position"/>
-            <state_interface name="position"/>
-            <state_interface name="velocity"/>
-          </joint>
-        </xacro:if>
-        <xacro:if value="${onrobot_type == 'rg2' or onrobot_type == 'rg6'}">
-          <joint name="${prefix}gripper_finger_joint">
-            <command_interface name="position"/>
-            <state_interface name="position"/>
-            <state_interface name="velocity"/>
-          </joint>
-        </xacro:if>
-      </ros2_control>
-    </xacro:unless>
-    <!-- ====================== Fake Hardware (for testing) ====================== -->
-    <xacro:if value="${use_fake_hardware}">
-      <ros2_control name="OnRobotGripper" type="actuator">
-        <hardware>
-          <!-- 2FG7 / 2FG14 - TwoFG Hardware Interface with fake hardware -->
-          <xacro:if value="${onrobot_type == '2fg7' or onrobot_type == '2fg14'}">
-            <plugin>onrobot_driver::TwoFGHardwareInterface</plugin>
-            <param name="onrobot_type">${onrobot_type}</param>
-            <param name="prefix">${prefix}</param>
-            <param name="connection_type">${connection_type}</param>
-            <param name="device">${device}</param>
-            <param name="ip_address">${ip_address}</param>
-            <param name="port">${port}</param>
-            <param name="device_address">${device_address}</param>
-            <param name="use_fake_hardware">true</param>
-          </xacro:if>
-          <!-- 3FG15 - ThreeFG Hardware Interface with fake hardware -->
-          <xacro:if value="${onrobot_type == '3fg15'}">
-            <plugin>onrobot_driver::ThreeFGHardwareInterface</plugin>
-            <param name="onrobot_type">${onrobot_type}</param>
-            <param name="prefix">${prefix}</param>
-            <param name="connection_type">${connection_type}</param>
-            <param name="device">${device}</param>
-            <param name="ip_address">${ip_address}</param>
-            <param name="port">${port}</param>
-            <param name="device_address">${device_address}</param>
-            <param name="use_fake_hardware">true</param>
-          </xacro:if>
-          <!-- RG2 / RG6 - RG Hardware Interface with fake hardware -->
-          <xacro:if value="${onrobot_type == 'rg2' or onrobot_type == 'rg6'}">
-            <plugin>onrobot_driver::RGHardwareInterface</plugin>
-            <param name="onrobot_type">${onrobot_type}</param>
-            <param name="prefix">${prefix}</param>
-            <param name="connection_type">${connection_type}</param>
-            <param name="device">${device}</param>
-            <param name="ip_address">${ip_address}</param>
-            <param name="port">${port}</param>
-            <param name="device_address">${device_address}</param>
-            <param name="use_fake_hardware">true</param>
-          </xacro:if>
-        </hardware>
-        <!-- Joint configuration for all gripper types -->
-        <xacro:if value="${onrobot_type == '2fg7' or onrobot_type == '2fg14' or onrobot_type == '3fg15'}">
-          <joint name="${prefix}finger_width">
-            <command_interface name="position"/>
-            <state_interface name="position"/>
-            <state_interface name="velocity"/>
-          </joint>
-        </xacro:if>
-        <xacro:if value="${onrobot_type == 'rg2' or onrobot_type == 'rg6'}">
-          <joint name="${prefix}gripper_finger_joint">
-            <command_interface name="position"/>
-            <state_interface name="position"/>
-            <state_interface name="velocity"/>
-          </joint>
-        </xacro:if>
+        <!-- Joint configuration for actuated grippers -->
+        <joint name="${prefix}finger_width">
+          <command_interface name="position"/>
+          <state_interface name="position"/>
+          <state_interface name="velocity"/>
+        </joint>
       </ros2_control>
     </xacro:if>

Commit message: Update 2FG7 joint configurations: adjust limits and origins for left and right finger joints

File: urdf/2fg7_macro.xacro (robot description, xacro)
@@ -92,23 +92,23 @@
       <child link="${prefix}finger_width_mock_link"/>
       <axis xyz="0 0 1"/>
-      <limit lower="0.035" upper="0.07" velocity="0.45" effort="140"/>
+      <limit lower="0.035" upper="0.073" velocity="0.45" effort="140"/>
     </joint>
     <!-- Left Finger Joint -->
     <joint name="${prefix}left_finger_joint" type="prismatic">
-      <origin xyz="-0.0302 0 0" rpy="0 0 0"/>
+      <origin xyz="0 0 0" rpy="0 0 3.141593"/>
       <parent link="${prefix}onrobot_base_link"/>
       <child link="${prefix}left_finger_link"/>
       <axis xyz="1 0 0"/>
-      <limit lower="-0.0175" upper="0.0" effort="140" velocity="0.45"/>
-      <mimic joint="${prefix}finger_width" multiplier="-0.5" offset="0.0175"/>
+      <limit lower="-0.0154" upper="0.0036" effort="140" velocity="0.45"/>
+      <mimic joint="${prefix}finger_width" multiplier="0.5" offset="-0.0329"/>
     </joint>
     <!-- Right Finger Joint -->
     <joint name="${prefix}right_finger_joint" type="prismatic">
-      <origin xyz="0.0302 0 0" rpy="0 0 0"/>
+      <origin xyz="0 0 0" rpy="0 0 3.141593"/>
       <parent link="${prefix}onrobot_base_link"/>
       <child link="${prefix}right_finger_link"/>
       <axis xyz="-1 0 0"/>
-      <limit lower="-0.0175" upper="0.0" effort="140" velocity="0.45"/>
-      <mimic joint="${prefix}finger_width" multiplier="-0.5" offset="0.0175"/>
+      <limit lower="-0.0154" upper="0.0036" effort="140" velocity="0.45"/>
+      <mimic joint="${prefix}finger_width" multiplier="0.5" offset="-0.0329"/>
     </joint>
     <!-- TCP Link -->
